File: BREAKOUT_BOARDS/Boostconverter.kicad_sch (KiCad schematic)
At the start: 37 parts, among them J1 POWERIN, J2 POWEROUT, Q1 TBD_N, Q2 TBD_N, Q3 TBD_N, Q4 TBD_N, U1 LM5175RHF

Commit message: Routing 1
Completed all footprint and part sourcing. Completed half of the routing.
Parts:
- added C16: 82u, MyFootprintLibrary:CAP_35SVPF82M, symbol Device:C_Polarized
- added U2: LM5175PWP, Package_SO:HTSSOP-28-1EP_4.4x9.7mm_P0.65mm_EP3.4x9.5mm_ThermalVias, symbol Regulator_Switching:LM5175PWP
- C1: footprint Capacitor_SMD:CP_Elec_6.3x5.4 -> MyFootprintLibrary:PCAP_SVP_F12_PAN-M
- C12, C13, C14, C2: footprint Capacitor_SMD:C_0603_1608Metric -> Capacitor_SMD:C_1210_3225Metric
- C5: value 22n -> 68n
- C7: value 47p -> 33p
- D1, D5: value SS54 -> SS14
- D2, D3: value B5819W SL -> SS14; footprint Diode_SMD:D_SOD-123 -> Diode_SMD:D_SMA
- D4: value SS54 -> SK104B; footprint Diode_SMD:D_SMA -> Diode_SMD:D_SMB
- L1: value 3.3u -> 2.2u; footprint Inductor_SMD:L_Panasonic_PCC-M0850M -> Inductor_SMD:L_Coilcraft_XAL1010-XXX
- Q1, Q2, Q3, Q4: value TBD_N -> NCEP60T15G; footprint Package_TO_SOT_SMD:SOT-23 -> MyFootprintLibrary:AO_DFN-8-1EP_5.55x5.2mm_P1.27mm_EP4.12x4.6mm
- R4: value 21k -> 26.7k
- R7: value 8m -> 5m
- U1: value LM5175RHF -> LM5175PWP
Connections:
- net +12V: now also U1.3 (VISNS); no longer U1.28 (VISNS)
- net +24V: now also J2.2 (Pin_2), U1.24 (BIAS), C16.1; no longer J2.1 (Pin_1), U1.21 (BIAS)
- net AGND: now also U1.5 (DITH); no longer U1.2 (DITH)
- net GNDREF: now also J2.1 (Pin_1), U1.10 (AGND), U1.15 (CSG), U1.22 (PGND), C16.2; no longer J2.2 (Pin_2), U1.12 (CSG), U1.19 (PGND), U1.7 (AGND)
- net HDRV1: now also U1.27 (HDRV1); no longer U1.24 (HDRV1)
- net HDRV2: now also U1.19 (HDRV2); no longer U1.16 (HDRV2)
- net LDRV2: now also U1.21 (LDRV2); no longer U1.18 (LDRV2)
- net SW2: now also D5.2 (A), L1.2, Q3.2 (S), Q4.3 (D), U1.18 (SW2); no longer U1.15 (SW2)
- net VCC: now also U1.23 (VCC); no longer U1.20 (VCC)
- net at R8.2, R9.1: now also U1.11 (FB); no longer U1.8 (FB)
- net at C10.1, D2.1 (K): now also U1.26 (BOOT1); no longer U1.23 (BOOT1)
- net at R1.2, R2.1: now also U1.1 (EN/UVLO); no longer U1.26 (EN/UVLO)
- net at D1.1 (K): now also R6.2; no longer R6.1
- net at R3.2: now also U1.6 (RT/SYNC); no longer U1.3 (RT/SYNC)
- net at C7.2, R4.2: now also U1.9 (COMP); no longer U1.6 (COMP)
- net at C6.2: now also U1.7 (SLOPE); no longer U1.4 (SLOPE)
- net at C11.1, D4.2 (A), Q2.2 (S)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: now also U1.16 (CS); no longer U1.13 (CS)
- net at C15.2: now also U1.12 (VOSNS); no longer U1.9 (VOSNS)
- net at C10.2, D4.1 (K), L1.1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: now also U1.28 (SW1); no longer U1.25 (SW1)
- net at R5.2: now also U1.4 (MODE); no longer U1.1 (MODE)
- net at Q2.1 (G): now also U1.25 (LDRV1); no longer U1.22 (LDRV1)
- net at C5.2: now also U1.8 (SS); no longer U1.5 (SS)
- net at C9.2, D3.1 (K): now also U1.20 (BOOT2); no longer U1.17 (BOOT2)
- net at U1.14 (ISNS(+)): now also U1.13 (ISNS(-))
- new net: C8.1, R6.1, U1.2 (VIN)
Other:
- moved on the sheet: J2, R6

Commit message: Add files via upload
Parts:
- removed U2: LM5175PWP, Package_SO:HTSSOP-28-1EP_4.4x9.7mm_P0.65mm_EP3.4x9.5mm_ThermalVias, symbol Regulator_Switching:LM5175PWP
- R7: footprint Resistor_SMD:R_0603_1608Metric -> Resistor_SMD:R_1206_3216Metric
Changed lines of the file:
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@@
 	(wire
 		(pts
-			(xy 121.92 57.15) (xy 125.73 57.15)
-		)
-		(stroke
-			(width 0)
-			(type default)
-		)
-	)
-	(wire
-		(pts
 			(xy 83.82 102.87) (xy 86.36 102.87)
 		)
@@
 	(wire
 		(pts
+			(xy 121.92 57.15) (xy 125.73 57.15)
+		)
+		(stroke
+			(width 0)
+			(type default)
+		)
+	)
+	(wire
+		(pts
 			(xy 259.08 58.42) (xy 259.08 60.96)
 		)
@@
 	)
 	(symbol
-		(lib_id "Regulator_Switching:LM5175PWP")
-		(at 30.48 104.14 0)
-		(unit 1)
-		(body_style 1)
-		(exclude_from_sim no)
-		(in_bom yes)
-		(on_board yes)
-		(in_pos_files yes)
-		(dnp no)
-		(fields_autoplaced yes)
-		(property "Reference" "U2"
-			(at 37.7033 78.74 0)
-			(show_name no)
-			(do_not_autoplace no)
-			(effects
-				(font
-					(size 1.27 1.27)
-				)
-				(justify left)
-			)
-		)
-		(property "Value" "LM5175PWP"
-			(at 37.7033 81.28 0)
-			(show_name no)
-			(do_not_autoplace no)
-			(effects
-				(font
-					(size 1.27 1.27)
-				)
-				(justify left)
-			)
-		)
-		(property "Footprint" "Package_SO:HTSSOP-28-1EP_4.4x9.7mm_P0.65mm_EP3.4x9.5mm_ThermalVias"
-			(at 48.26 82.55 0)
-			(hide yes)
-			(show_name no)
-			(do_not_autoplace no)
-			(effects
-				(font
-					(size 1.27 1.27)
-				)
-				(justify left)
-			)
-		)
-		(property "Datasheet" "http://www.ti.com/lit/ds/symlink/lm5175.pdf"
-			(at 81.28 115.57 0)
-			(hide yes)
-			(show_name no)
-			(do_not_autoplace no)
-			(effects
-				(font
-					(size 1.27 1.27)
-				)
-			)
-		)
-		(property "Description" "42-V wide Vin synchronous 4-switch Buck-Boost controller, HTSSOP-28 package"
-			(at 30.48 104.14 0)
-			(hide yes)
-			(show_name no)
-			(do_not_autoplace no)
-			(effects
-				(font
-					(size 1.27 1.27)
-				)
-			)
-		)
-		(pin "5"
-		)
-		(pin "13"
-		)
-		(pin "9"
-		)
-		(pin "16"
-		)
-		(pin "12"
-		)
-		(pin "11"
-		)
-		(pin "7"
-		)
-		(pin "4"
-		)
-		(pin "1"
-		)
-		(pin "2"
-		)
-		(pin "3"
-		)
-		(pin "6"
-		)
-		(pin "8"
-		)
-		(pin "10"
-		)
-		(pin "14"
-		)
-		(pin "15"
-		)
-		(pin "18"
-		)
-		(pin "21"
-		)
-		(pin "20"
-		)
-		(pin "23"
-		)
-		(pin "25"
-		)
-		(pin "28"
-		)
-		(pin "24"
-		)
-		(pin "26"
-		)
-		(pin "27"
-		)
-		(pin "29"
-		)
-		(pin "22"
-		)
-		(pin "17"
-		)
-		(pin "19"
-		)
-		(instances
-			(project "Boostconverter"
-				(path "/55e1af9e-0ce6-427e-8a3b-d9517e87da9c"
-					(reference "U2")
-					(unit 1)
-				)
-			)
-		)
-	)
-	(symbol
 		(lib_id "power:+12V")
 		(at 224.79 29.21 0)
@@
 			)
 		)
-		(property "Footprint" "Resistor_SMD:R_0603_1608Metric"
+		(property "Footprint" "Resistor_SMD:R_1206_3216Metric"
 			(at 170.942 101.6 90)
 			(hide yes)
