File: ELECTRONICS/ANCHOR/AutoBot.kicad_sch (KiCad schematic)
At the start: 33 parts, among them IC1 DW3210, J1 USB_C_Receptacle_USB2.0_16P, U1 BQ24075RGT, U2 NRF52840-QFAA-R7, U3 AP7370-33FDC

Commit message: Add files via upload
Parts:
- added C17: 4.7u, symbol Device:C
- C1: value 47u -> 4.7u
- C15, C16: value 100n -> 1u
Connections:
- net BQ_OUT: now also C17.1
- net GNDREF: now also C17.2; no longer J1.A8 (SBU1), J1.B8 (SBU2)
- net D+: no longer names the net of J1.A6 (D+)
- net D+: no longer J1.B6 (D+)
- net D-: no longer names the net of J1.A7 (D-)
- net D-: no longer J1.B7 (D-)
- no-connect marks 1 -> 7
Changed lines of the file:
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@@
 	)
 	(junction
-		(at 54.61 44.45)
+		(at 189.23 161.29)
 		(diameter 0)
 		(color 0 0 0 0)
 	)
 	(junction
-		(at 189.23 161.29)
+		(at 163.83 58.42)
 		(diameter 0)
 		(color 0 0 0 0)
@@
 	)
 	(junction
-		(at 57.15 66.04)
-		(diameter 0)
-		(color 0 0 0 0)
-	)
-	(junction
-		(at 54.61 66.04)
-		(diameter 0)
-		(color 0 0 0 0)
-	)
-	(junction
 		(at 237.49 119.38)
 		(diameter 0)
@@
 	)
 	(junction
-		(at 163.83 58.42)
+		(at 163.83 67.31)
 		(diameter 0)
 		(color 0 0 0 0)
@@
 	)
 	(junction
+		(at 156.21 58.42)
+		(diameter 0)
+		(color 0 0 0 0)
+	)
+	(junction
 		(at 222.25 130.81)
 		(diameter 0)
@@
 		(color 0 0 0 0)
 	)
-	(junction
-		(at 54.61 39.37)
-		(diameter 0)
-		(color 0 0 0 0)
+	(no_connect
+		(at 54.61 40.64)
+	)
+	(no_connect
+		(at 54.61 45.72)
+	)
+	(no_connect
+		(at 54.61 43.18)
+	)
+	(no_connect
+		(at 54.61 55.88)
 	)
 	(no_connect
 		(at 113.03 35.56)
 	)
+	(no_connect
+		(at 54.61 38.1)
+	)
+	(no_connect
+		(at 54.61 53.34)
+	)
 	(wire
 		(pts
@@
 	(wire
 		(pts
-			(xy 54.61 39.37) (xy 59.69 39.37)
-		)
-		(stroke
-			(width 0)
-			(type default)
-		)
-	)
-	(wire
-		(pts
 			(xy 147.32 133.35) (xy 158.75 133.35)
 		)
@@
 	(wire
 		(pts
-			(xy 147.32 125.73) (xy 158.75 125.73)
-		)
-		(stroke
-			(width 0)
-			(type default)
-		)
-	)
-	(wire
-		(pts
-			(xy 179.07 161.29) (xy 179.07 160.02)
+			(xy 163.83 67.31) (xy 175.26 67.31)
 		)
 		(stroke
@@
 	(wire
 		(pts
-			(xy 68.58 50.8) (xy 68.58 66.04)
+			(xy 147.32 125.73) (xy 158.75 125.73)
 		)
 		(stroke
@@
 	(wire
 		(pts
-			(xy 57.15 66.04) (xy 68.58 66.04)
+			(xy 179.07 161.29) (xy 179.07 160.02)
 		)
 		(stroke
@@
 	(wire
 		(pts
-			(xy 163.83 67.31) (xy 175.26 67.31)
+			(xy 68.58 50.8) (xy 68.58 66.04)
 		)
 		(stroke
@@
 	(wire
 		(pts
-			(xy 54.61 38.1) (xy 54.61 39.37)
+			(xy 181.61 161.29) (xy 182.88 161.29)
 		)
 		(stroke
@@
 	(wire
 		(pts
-			(xy 181.61 161.29) (xy 182.88 161.29)
+			(xy 156.21 67.31) (xy 156.21 66.04)
 		)
 		(stroke
@@
 	(wire
 		(pts
-			(xy 39.37 66.04) (xy 54.61 66.04)
+			(xy 39.37 66.04) (xy 68.58 66.04)
 		)
 		(stroke
@@
 	(wire
 		(pts
-			(xy 54.61 55.88) (xy 54.61 66.04)
-		)
-		(stroke
-			(width 0)
-			(type default)
-		)
-	)
-	(wire
-		(pts
 			(xy 243.84 95.25) (xy 243.84 106.68)
 		)
@@
 	(wire
 		(pts
-			(xy 54.61 53.34) (xy 57.15 53.34)
-		)
-		(stroke
-			(width 0)
-			(type default)
-		)
-	)
-	(wire
-		(pts
 			(xy 168.91 161.29) (xy 171.45 161.29)
 		)
@@
 	(wire
 		(pts
-			(xy 57.15 53.34) (xy 57.15 66.04)
-		)
-		(stroke
-			(width 0)
-			(type default)
-		)
-	)
-	(wire
-		(pts
 			(xy 138.43 40.64) (xy 152.4 40.64)
 		)
@@
 	(wire
 		(pts
-			(xy 54.61 44.45) (xy 54.61 45.72)
-		)
-		(stroke
-			(width 0)
-			(type default)
-		)
-	)
-	(wire
-		(pts
 			(xy 218.44 35.56) (xy 218.44 38.1)
 		)
@@
 	(wire
 		(pts
-			(xy 171.45 161.29) (xy 171.45 160.02)
+			(xy 156.21 67.31) (xy 163.83 67.31)
 		)
 		(stroke
@@
 	(wire
 		(pts
-			(xy 147.32 128.27) (xy 158.75 128.27)
+			(xy 171.45 161.29) (xy 171.45 160.02)
 		)
 		(stroke
@@
 	(wire
 		(pts
-			(xy 74.93 30.48) (xy 74.93 39.37)
+			(xy 147.32 128.27) (xy 158.75 128.27)
 		)
 		(stroke
@@
 	(wire
 		(pts
-			(xy 212.09 95.25) (xy 237.49 95.25)
+			(xy 74.93 30.48) (xy 74.93 39.37)
 		)
 		(stroke
@@
 	(wire
 		(pts
-			(xy 54.61 43.18) (xy 54.61 44.45)
+			(xy 212.09 95.25) (xy 237.49 95.25)
 		)
 		(stroke
@@
 	(wire
 		(pts
-			(xy 54.61 39.37) (xy 54.61 40.64)
-		)
-		(stroke
-			(width 0)
-			(type default)
-		)
-	)
-	(wire
-		(pts
 			(xy 218.44 45.72) (xy 218.44 38.1)
 		)
@@
 	(wire
 		(pts
-			(xy 54.61 66.04) (xy 57.15 66.04)
-		)
-		(stroke
-			(width 0)
-			(type default)
-		)
-	)
-	(wire
-		(pts
 			(xy 212.09 148.59) (xy 226.06 148.59)
 		)
@@
 	(wire
 		(pts
-			(xy 54.61 44.45) (xy 59.69 44.45)
+			(xy 212.09 119.38) (xy 222.25 119.38)
 		)
 		(stroke
@@
 	(wire
 		(pts
-			(xy 212.09 119.38) (xy 222.25 119.38)
+			(xy 156.21 58.42) (xy 163.83 58.42)
 		)
 		(stroke
@@
 	(wire
 		(pts
-			(xy 158.75 58.42) (xy 163.83 58.42)
+			(xy 144.78 58.42) (xy 156.21 58.42)
 		)
 		(stroke
@@
 	)
 	(label "BQ_OUT"
-		(at 158.75 58.42 0)
+		(at 144.78 58.42 0)
 		(effects
 			(font
@@
 		)
 	)
-	(label "D-"
-		(at 59.69 39.37 180)
-		(effects
-			(font
-				(size 1.27 1.27)
-			)
-			(justify right bottom)
-		)
-	)
 	(label "DW_RST"
 		(at 149.86 97.79 0)
@@
 		)
 	)
-	(label "D+"
-		(at 59.69 44.45 180)
-		(effects
-			(font
-				(size 1.27 1.27)
-			)
-			(justify right bottom)
-		)
-	)
 	(label "SPIMOSI"
 		(at 149.86 102.87 0)
@@
 	(symbol
 		(lib_id "Device:C")
+		(at 156.21 62.23 0)
+		(unit 1)
+		(body_style 1)
+		(exclude_from_sim no)
+		(in_bom yes)
+		(on_board yes)
+		(in_pos_files yes)
+		(dnp no)
+		(property "Reference" "C17"
+			(at 156.718 60.452 0)
+			(show_name no)
+			(do_not_autoplace no)
+			(effects
+				(font
+					(size 1.27 1.27)
+				)
+				(justify left)
+			)
+		)
+		(property "Value" "4.7u"
+			(at 156.972 64.516 0)
+			(show_name no)
+			(do_not_autoplace no)
+			(effects
+				(font
+					(size 1.27 1.27)
+				)
+				(justify left)
+			)
+		)
+		(property "Footprint" ""
+			(at 157.1752 66.04 0)
+			(hide yes)
+			(show_name no)
+			(do_not_autoplace no)
+			(effects
+				(font
+					(size 1.27 1.27)
+				)
+			)
+		)
+		(property "Datasheet" ""
+			(at 156.21 62.23 0)
+			(hide yes)
+			(show_name no)
+			(do_not_autoplace no)
+			(effects
+				(font
+					(size 1.27 1.27)
+				)
+			)
+		)
+		(property "Description" "Unpolarized capacitor"
+			(at 156.21 62.23 0)
+			(hide yes)
+			(show_name no)
+			(do_not_autoplace no)
+			(effects
+				(font
+					(size 1.27 1.27)
+				)
+			)
+		)
+		(pin "2"
+		)
+		(pin "1"
+		)
+		(instances
+			(project "AutoBot"
+				(path "/f0c1f634-c0f3-4bd1-ace6-074b146b57fe"
+					(reference "C17")
+					(unit 1)
+				)
+			)
+		)
+	)
+	(symbol
+		(lib_id "Device:C")
 		(at 237.49 134.62 0)
 		(unit 1)
@@
 			)
 		)
-		(property "Value" "100n"
+		(property "Value" "1u"
 			(at 187.452 64.262 0)
 			(show_name no)
@@
 			)
 		)
-		(property "Value" "47u"
+		(property "Value" "4.7u"
 			(at 158.242 41.656 0)
 			(show_name no)
@@
 			)
 		)
-		(property "Value" "100n"
+		(property "Value" "1u"
 			(at 164.592 64.262 0)
 			(show_name no)

Commit message: Add files via upload
Parts:
- C11: value 100n -> 220n
Changed lines of the file:
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@@
 			)
 		)
-		(property "Value" "100n"
+		(property "Value" "220n"
 			(at 226.822 154.432 0)
 			(show_name no)

Commit message: Add files via upload
Parts:
- removed C14: 2p, symbol Device:C
Connections:
- net CHG: now also D2.1 (K); no longer D2.2 (A)
- net PGOOD: now also D1.1 (K); no longer D1.2 (A)
- net at IC1.13 (RF2): now also R8.2
- net at R6.1: now also D1.2 (A); no longer D1.1 (K)
- net at R7.1: now also D2.2 (A); no longer D2.1 (K)
Other:
- moved on the sheet: D1, D2, R8
Changed lines of the file:
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@@
 	)
 	(junction
-		(at 168.91 161.29)
+		(at 156.21 58.42)
 		(diameter 0)
 		(color 0 0 0 0)
 	)
 	(junction
-		(at 140.97 115.57)
+		(at 168.91 161.29)
 		(diameter 0)
 		(color 0 0 0 0)
 	)
 	(junction
-		(at 222.25 119.38)
+		(at 140.97 115.57)
 		(diameter 0)
 		(color 0 0 0 0)
 	)
 	(junction
-		(at 156.21 58.42)
+		(at 222.25 119.38)
 		(diameter 0)
 		(color 0 0 0 0)
@@
 	(wire
 		(pts
-			(xy 134.62 147.32) (xy 137.16 147.32)
+			(xy 138.43 147.32) (xy 147.32 147.32)
 		)
 		(stroke
@@
 	(wire
 		(pts
-			(xy 134.62 147.32) (xy 134.62 148.59)
+			(xy 138.43 147.32) (xy 138.43 148.59)
 		)
 		(stroke
@@
 	(wire
 		(pts
-			(xy 144.78 147.32) (xy 147.32 147.32)
+			(xy 154.94 147.32) (xy 158.75 147.32)
 		)
 		(stroke
@@
 	(wire
 		(pts
+			(xy 144.78 58.42) (xy 156.21 58.42)
+		)
+		(stroke
+			(width 0)
+			(type default)
+		)
+	)
+	(wire
+		(pts
 			(xy 176.53 161.29) (xy 179.07 161.29)
 		)
@@
 	(wire
 		(pts
-			(xy 154.94 147.32) (xy 158.75 147.32)
-		)
-		(stroke
-			(width 0)
-			(type default)
-		)
-	)
-	(wire
-		(pts
 			(xy 90.17 125.73) (xy 101.6 125.73)
 		)
@@
 	(wire
 		(pts
-			(xy 144.78 58.42) (xy 156.21 58.42)
-		)
-		(stroke
-			(width 0)
-			(type default)
-		)
-	)
-	(wire
-		(pts
 			(xy 186.69 66.04) (xy 186.69 67.31)
 		)
@@
 	(symbol
 		(lib_id "Device:C")
-		(at 151.13 147.32 90)
-		(unit 1)
-		(body_style 1)
-		(exclude_from_sim no)
-		(in_bom yes)
-		(on_board yes)
-		(in_pos_files yes)
-		(dnp no)
-		(property "Reference" "C14"
-			(at 153.924 148.844 90)
-			(show_name no)
-			(do_not_autoplace no)
-			(effects
-				(font
-					(size 1.27 1.27)
-				)
-			)
-		)
-		(property "Value" "2p"
-			(at 153.924 146.05 90)
-			(show_name no)
-			(do_not_autoplace no)
-			(effects
-				(font
-					(size 1.27 1.27)
-				)
-			)
-		)
-		(property "Footprint" ""
-			(at 154.94 146.3548 0)
-			(hide yes)
-			(show_name no)
-			(do_not_autoplace no)
-			(effects
-				(font
-					(size 1.27 1.27)
-				)
-			)
-		)
-		(property "Datasheet" ""
-			(at 151.13 147.32 0)
-			(hide yes)
-			(show_name no)
-			(do_not_autoplace no)
-			(effects
-				(font
-					(size 1.27 1.27)
-				)
-			)
-		)
-		(property "Description" "Unpolarized capacitor"
-			(at 151.13 147.32 0)
-			(hide yes)
-			(show_name no)
-			(do_not_autoplace no)
-			(effects
-				(font
-					(size 1.27 1.27)
-				)
-			)
-		)
-		(pin "2"
-		)
-		(pin "1"
-		)
-		(instances
-			(project "AutoBot"
-				(path "/f0c1f634-c0f3-4bd1-ace6-074b146b57fe"
-					(reference "C14")
-					(unit 1)
-				)
-			)
-		)
-	)
-	(symbol
-		(lib_id "Device:C")
 		(at 222.25 110.49 0)
 		(unit 1)
@@
 	(symbol
 		(lib_id "Device:LED")
-		(at 201.93 45.72 180)
+		(at 201.93 45.72 0)
 		(unit 1)
 		(body_style 1)
@@
 		(dnp no)
 		(property "Reference" "D2"
-			(at 201.676 43.18 0)
+			(at 202.184 48.26 0)
 			(show_name no)
 			(do_not_autoplace no)
@@
 		)
 		(property "Value" "LED"
-			(at 201.93 48.006 0)
+			(at 201.93 43.434 0)
 			(show_name no)
 			(do_not_autoplace no)
@@
 	(symbol
 		(lib_id "Device:R")
-		(at 140.97 147.32 90)
+		(at 151.13 147.32 90)
 		(unit 1)
 		(body_style 1)
@@
 		(dnp no)
 		(property "Reference" "R8"
-			(at 140.97 149.606 90)
+			(at 151.13 149.606 90)
 			(show_name no)
 			(do_not_autoplace no)
@@
 		)
 		(property "Value" "50"
-			(at 140.97 147.32 90)
+			(at 151.13 147.32 90)
 			(show_name no)
 			(do_not_autoplace no)
@@
 		)
 		(property "Footprint" ""
-			(at 140.97 149.098 90)
+			(at 151.13 149.098 90)
 			(hide yes)
 			(show_name no)
@@
 		)
 		(property "Datasheet" ""
-			(at 140.97 147.32 0)
+			(at 151.13 147.32 0)
 			(hide yes)
 			(show_name no)
@@
 		)
 		(property "Description" "Resistor"
-			(at 140.97 147.32 0)
+			(at 151.13 147.32 0)
 			(hide yes)
 			(show_name no)
@@
 	(symbol
 		(lib_id "Device:LED")
-		(at 201.93 38.1 180)
+		(at 201.93 38.1 0)
 		(unit 1)
 		(body_style 1)
@@
 		(dnp no)
 		(property "Reference" "D1"
-			(at 201.93 35.814 0)
+			(at 201.93 40.386 0)
 			(show_name no)
 			(do_not_autoplace no)
@@
 		)
 		(property "Value" "LED"
-			(at 201.93 40.132 0)
+			(at 201.93 36.068 0)
 			(show_name no)
 			(do_not_autoplace no)
@@
 	(symbol
 		(lib_id "power:GNDREF")
-		(at 134.62 148.59 0)
+		(at 138.43 148.59 0)
 		(unit 1)
 		(body_style 1)
@@
 		(fields_autoplaced yes)
 		(property "Reference" "#PWR016"
-			(at 134.62 154.94 0)
+			(at 138.43 154.94 0)
 			(hide yes)
 			(show_name no)
@@
 		)
 		(property "Value" "GNDREF"
-			(at 134.62 153.67 0)
+			(at 138.43 153.67 0)
 			(hide yes)
 			(show_name no)
@@
 		)
 		(property "Footprint" ""
-			(at 134.62 148.59 0)
+			(at 138.43 148.59 0)
 			(hide yes)
 			(show_name no)
@@
 		)
 		(property "Datasheet" ""
-			(at 134.62 148.59 0)
+			(at 138.43 148.59 0)
 			(hide yes)
 			(show_name no)
@@
 		)
 		(property "Description" "Power symbol creates a global label with name \"GNDREF\" , reference supply ground"
-			(at 134.62 148.59 0)
+			(at 138.43 148.59 0)
 			(hide yes)
 			(show_name no)

Commit message: Add files via upload
Parts:
- added C14: 1p, symbol Device:C
- added C18: 1u, symbol Device:C
- added C19: 100n, symbol Device:C
- added C20: 100p, symbol Device:C
- added D3, D4, D5: LED, symbol Device:LED
- added J2, J4: Conn_01x05_Pin, symbol Connector:Conn_01x05_Pin
- added J3: Conn_01x07_Pin, symbol Connector:Conn_01x07_Pin
- added J5: Conn_01x02_Pin, symbol Connector:Conn_01x02_Pin
- added L1: 3.9n, symbol Device:L
- added L2: 4.7n, symbol Device:L
- added Q1, Q2, Q3: DMG1012T, Package_TO_SOT_SMD:SOT-523, symbol Transistor_FET:DMG1012T
- added R11, R12, R9: R, symbol Device:R
- added R13, R14, R15, R16, R17, R18, R19: 10k, symbol Device:R
- added SW1: reset, symbol Switch:SW_Push
- added SW3: SW_DIP_x05, symbol Switch:SW_DIP_x05
- IC1: footprint QFN40P500X500X80-40N-D -> AutoBotfootprintlibrary:QFN40P500X500X80-40N-D
- R1, R2: value R -> 5.1k
- R3, R4: value R -> 2.2k
Connections:
- net +3V3: now also U2.12 (VDD), U2.17 (VDD), U2.25 (VDD), U2.37 (VDD), U2.48 (VDD), D3.2 (A), D4.2 (A), D5.2 (A), R13.2, R14.2, R15.2, R16.2, R17.2
- net DW_GPIO0: now also J2.2 (Pin_2)
- net DW_GPIO4: now also J2.4 (Pin_4)
- net DW_GPIO5: now also J2.3 (Pin_3)
- net DW_GPIO6: now also J2.1 (Pin_1)
- net DW_GPIO7: now also J2.5 (Pin_5)
- net DW_RST: now also U2.21 (P0.22/QSPI)
- net GNDREF: now also U2.32 (VSS_PA), U2.45 (VSS), U2.47 (DCC), U2.49 (VSS), C14.2, C18.2, C19.2, C20.2, Q1.2 (S), Q2.2 (S), Q3.2 (S), R18.1, R19.1, SW1.1
- net IRQ: now also U2.13 (P0.13)
- net RXLED: now also Q2.1 (G)
- net RX_OK_LED: now also Q1.1 (G)
- net SPICLK: now also U2.18 (P0.19/QSPI/SCK)
- net SPICSN: now also U2.14 (P0.14)
- net SPIMISO: now also U2.20 (P0.21/QSPI)
- net SPIMOSI: now also U2.19 (P0.20)
- net TRACECLK: now also J4.1 (Pin_1)
- net TRACEDATA1: now also J4.3 (Pin_3)
- net TRACEDATA2: now also J4.4 (Pin_4)
- net TRACEDATA3: now also J4.5 (Pin_5)
- net TXLED: now also Q3.1 (G)
- net WAKEUP: now also U2.22 (P0.23/QSPI)
- net at U2.1 (DEC1): now also C19.1
- net at U2.16 (P0.18/RESET/QSPI/CSN): now also SW1.2
- net TRACEDATA0: now reaches U2.24 (P1.00/TRACEDATA0/QSPI)
- net TRACEDATA0: now also J4.2 (Pin_2)
- net SWDIO: now reaches U2.26 (SWDIO)
- net SWDCLK: now reaches U2.27 (SWDCLK)
- net P0.09/NFC1: now reaches U2.29 (P0.09/NFC1)
- net P0.09/NFC1: now also J5.2 (Pin_2)
- net P0.10/NFC2: now reaches U2.30 (P0.10/NFC2)
- net P0.10/NFC2: now also J5.1 (Pin_1)
- net at U2.31 (ANT): now also L1.2
- net at U2.33 (DEC6): now also U2.46 (DEC4), C18.1
- net at U2.34 (DEC3): now also C20.1
- net XC1: now reaches U2.35 (XC1)
- net XC2: now reaches U2.36 (XC2)
- net P1.15: now reaches U2.38 (P1.15)
- net P1.15: now also J3.1 (Pin_1)
- net P0.03/AIN1: now reaches U2.39 (P0.03/AIN1)
- net P0.03/AIN1: now also J3.2 (Pin_2)
- net MODE__SEL: now reaches U2.4 (P0.04/AIN2)
- net P0.02/AIN0: now reaches U2.40 (P0.02/AIN0)
- net P0.02/AIN0: now also J3.3 (Pin_3)
- net P0.28/AIN4: now reaches U2.41 (P0.28/AIN4)
- net P0.28/AIN4: now also J3.4 (Pin_4)
- net P0.29/AIN5: now reaches U2.42 (P0.29/AIN5)
- net P0.29/AIN5: now also J3.5 (Pin_5)
- net P0.30/AIN6: now reaches U2.43 (P0.30/AIN6)
- net P0.30/AIN6: now also J3.6 (Pin_6)
- net P0.31/AIN7: now reaches U2.44 (P0.31/AIN7)
- net P0.31/AIN7: now also J3.7 (Pin_7)
- net ID_SEL: now reaches U2.5 (P0.05/AIN3)
- net ID_SEL: now also R18.2, SW3.2, SW3.3, SW3.4, SW3.5
- new net: R13.1, SW3.10
- new net: R17.1, SW3.6
- new net: R16.1, SW3.7
- new net: R15.1, SW3.8
- new net: R14.1, SW3.9
- new net: Q1.3 (D), R9.2
- new net: C14.1, L1.1, L2.2
- new net: Q2.3 (D), R11.2
- new net: Q3.3 (D), R12.2
- new net: D5.1 (K), R12.1
- new net: D3.1 (K), R9.1
- new net: D4.1 (K), R11.1
- new net MODE_SEL: R19.2, SW3.1
- new net NRF_ANT: L2.1
- no-connect marks 7 -> 11
Other:
- note added: "MAYBE PLACE CAPACITOR FOR DCC"
- note added: "USE DW3220 FOR PDOA SUPPORT"
- note added: "decoup cap prolly not req"
- note added: "might use the antenna for wireless flashing"
- note added: "resistor value shall be determined by whats already on the schematic"
- moved on the sheet: C10, C11, C12, C13, C2, C3, C4, C5, C6, C7, C8, C9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

Commit message: Add files via upload
Parts:
- added C21: NC, symbol Device:C
- added C22: 1p, symbol Device:C
- C14: value 1p -> 1.2p
Connections:
- net GNDREF: now also C21.2, C22.2
- net at C18.1, U2.33 (DEC6), U2.46 (DEC4): now also C21.1
- net at L1.2, U2.31 (ANT): now also C22.1
Other:
- note added: "GET CRYSTALS LATER"
- moved on the sheet: C14, L1, L2, R13, R14, R15, R16, R17, R18, R19

Commit message: Add files via upload
Parts:
- removed J3: Conn_01x07_Pin, symbol Connector:Conn_01x07_Pin
- removed R8: 50, symbol Device:R
- added C23: 1u, Capacitor_SMD:C_0402_1005Metric, symbol Device:C
- added C24: 1p, Capacitor_SMD:C_0402_1005Metric, symbol Device:C
- added C25, C26, C27, C28, C29, C30: 12p, Capacitor_SMD:C_0402_1005Metric, symbol Device:C
- added C31: 2p, Capacitor_SMD:C_0402_1005Metric, symbol Device:C
- added C32, C33, C34, C35: 100n, symbol Device:C
- added C36: 1u, symbol Device:C
- added J3, J6: Conn_01x04_Pin, Connector_PinHeader_2.54mm:PinHeader_1x04_P2.54mm_Vertical, symbol Connector:Conn_01x04_Pin
- added J7, J8: Conn_Coaxial, Connector_Coaxial:U.FL_Hirose_U.FL-R-SMT-1_Vertical, symbol Connector:Conn_Coaxial
- added J9: Conn_01x02_Pin, Connector_JST:JST_PH_B2B-PH-K_1x02_P2.00mm_Vertical, symbol Connector:Conn_01x02_Pin
- added L3: 10u, Inductor_SMD:L_0603_1608Metric, symbol Device:L
- added L4: 15u, Inductor_SMD:L_0603_1608Metric, symbol Device:L
- added Y1: TXC 8Y38472012, Crystal:Crystal_SMD_2016-4Pin_2.0x1.6mm, symbol Device:Crystal_GND24
- added Y2: ECS-320-8-37B-CKY-TR, Crystal:Crystal_SMD_2016-4Pin_2.0x1.6mm, symbol Device:Crystal_GND24
- added Y3: ECS-.327-6-1210B-N-TR, Crystal:Crystal_SMD_2016-4Pin_2.0x1.6mm, symbol Device:Crystal_GND24
- C1, C10, C11, C12, C13, C14, C15, C16, C17, C19, C2, C20, C21, C22, C3, C4, C5, C6, C7, C8, C9: footprint (none) -> Capacitor_SMD:C_0402_1005Metric
- C18: value 1u -> 47n; footprint (none) -> Capacitor_SMD:C_0402_1005Metric
- D1, D2, D3, D4, D5: footprint (none) -> LED_SMD:LED_0402_1005Metric
- FB1: footprint (none) -> Resistor_SMD:R_0603_1608Metric
- J1: footprint (none) -> Connector_USB:USB_C_Receptacle_GCT_USB4105-xx-A_16P_TopMnt_Horizontal
- J2, J4: footprint (none) -> Connector_PinHeader_2.54mm:PinHeader_1x05_P2.54mm_Vertical
- J5: footprint (none) -> Connector_PinHeader_2.54mm:PinHeader_1x02_P2.54mm_Vertical
- L1: value 3.9n -> 2.2n; footprint (none) -> Inductor_SMD:L_0402_1005Metric
- L2: footprint (none) -> Inductor_SMD:L_0402_1005Metric
- R1, R10, R11, R12, R13, R14, R15, R16, R17, R18, R19, R2, R5, R6, R7, R9: footprint (none) -> Resistor_SMD:R_0402_1005Metric
- R3, R4: value 2.2k -> 2.2K; footprint (none) -> Resistor_SMD:R_0402_1005Metric
- U2: footprint QFN48_NRF52840-QFAA-R7_NOR -> AutoBotfootprintlibrary:QFN48_NRF52840-QFAA-R7_NOR
Connections:
- net P0.02/AIN0 is gone; now on net CHG: U2.40 (P0.02/AIN0)
- net P0.03/AIN1 is gone; now on net PGOOD: U2.39 (P0.03/AIN1)
- net P1.15 is gone; now on net CE: U2.38 (P1.15)
- net +3V3: now also C32.1, C33.1, C34.1, C35.1, C36.1, J3.1 (Pin_1)
- net BAT+: now also J9.1 (Pin_1)
- net GNDREF: now also C24.2, C25.2, C26.2, C27.2, C28.2, C29.2, C30.2, C32.2, C33.2, C34.2, C35.2, C36.2, J3.4 (Pin_4), J7.2 (Ext), J8.2 (Ext), J9.2 (Pin_2), Y1.2 (G), Y1.4 (G), Y2.2 (G), Y2.4 (G), Y3.2 (G), Y3.4 (G); no longer U2.47 (DCC)
- net NRF_ANT: now also L1.1; no longer L2.1
- net P0.28/AIN4: now also J6.1 (Pin_1)
- net P0.29/AIN5: now also J6.2 (Pin_2)
- net P0.30/AIN6: now also J6.3 (Pin_3)
- net P0.31/AIN7: now also J6.4 (Pin_4)
- net SWDCLK: now also J3.2 (Pin_2)
- net SWDIO: now also J3.3 (Pin_3)
- net XC1: now also C27.1, C29.1, Y2.1, Y3.1
- net XC2: now also C28.1, C30.1, Y2.3, Y3.3
- net XTI: now also C26.1, Y1.3
- net XTO: now also C24.1, C25.1, Y1.1
- net at IC1.13 (RF2): now also C31.2
- net at C18.1, C21.1, U2.33 (DEC6)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: now also C23.2
- net at C22.1, U2.31 (ANT): now also L2.2; no longer L1.2
- net DW_RF renamed DW_RF1
- net DW_RF1: now also J7.1 (In)
- new net: C14.1, L1.2, L2.1
- new net: C23.1, L4.1
- new net: L3.2, U2.47 (DCC)
- new net: L3.1, L4.2
- new net DW_RF2: C31.1, J8.1 (In)
Other:
- note added: "1u for pin 48"
- note added: "32.768KHZ"
- note added: "32MHZ"
- note added: "ANCHOR ID, MASTER/SLAVE SEL"
- note added: "ANTENNAS"
- note added: "BATTERY"
- note added: "BLUE"
- note added: "C24 IS NOT A LOAD CAPACITOR C25 C26 VALUE NOT CONFIRMED TARGET 10 PF"
- note added: "CHARGING IC LEDS"
- note added: "CRYSTAL"
- note added: "CRYSTALS"
- note added: "DEBUGGING"
- note added: "DECOUPLING CAPS"
- note added: "DW3210 GPIO"
- note added: "DW3220 UWB TRANSCEIVER"
- note added: "GREEN"
- note added: "LED INDICATORS"
- note added: "NRF 52840 QFAA R7"
- note added: "NRF GPIO"
- note added: "POWER"
- note added: "RED"
- note added: "TEMP VALUES, TARGET 6 PF"
- note added: "TEMP VALUES, TARGET 8 PF"
- note added: "USBC"
- note removed: "GET CRYSTALS LATER"
- moved on the sheet: C1, C10, C11, C12, C13, C14, C15, C16, C17, C18, C19, C2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

Commit message: Add files via upload
Parts:
- removed J9: Conn_01x02_Pin, Connector_JST:JST_PH_B2B-PH-K_1x02_P2.00mm_Vertical, symbol Connector:Conn_01x02_Pin
- added BT1: LiPo, symbol Device:Battery_Cell
- R14: value 10k -> 1k
- R15: value 10k -> 2.2k
- R16: value 10k -> 5.1k
Connections:
- net BAT+: now also BT1.1 (+)
- net GNDREF: now also BT1.2 (-)
