File: ELECTRONICS/ANCHOR/AutoBot.kicad_sch (KiCad schematic)
At the start: 85 parts, among them IC1 DW3210, J1 USB_C_Receptacle_USB2.0_16P, J2 Conn_01x05_Pin, J3 Conn_01x04_Pin, J4 Conn_01x05_Pin, J5 Conn_01x02_Pin, J6 Conn_01x04_Pin, J7 Conn_Coaxial, J8 Conn_Coaxial, Q1 DMG1012T, Q2 DMG1012T, Q3 DMG1012T, SW1 reset, SW3 SW_DIP_x05, U1 BQ24075RGT, U2 NRF52840-QFAA-R7, U3 AP7370-33FDC, Y1 TXC 8Y38472012, Y2 ECS-320-8-37B-CKY-TR, Y3 ECS-.327-6-1210B-N-TR

Commit message: Add files via upload
Parts:
- removed BT1: LiPo, symbol Device:Battery_Cell
- removed C1, C17, C3: 4.7u, Capacitor_SMD:C_0402_1005Metric, symbol Device:C
- removed C10, C7: 10u, Capacitor_SMD:C_0402_1005Metric, symbol Device:C
- removed C11: 220n, Capacitor_SMD:C_0402_1005Metric, symbol Device:C
- removed C12, C19, C2, C6, C9: 100n, Capacitor_SMD:C_0402_1005Metric, symbol Device:C
- removed C13, C31: 2p, Capacitor_SMD:C_0402_1005Metric, symbol Device:C
- removed C14: 1.2p, Capacitor_SMD:C_0402_1005Metric, symbol Device:C
- removed C15, C16, C23: 1u, Capacitor_SMD:C_0402_1005Metric, symbol Device:C
- removed C18: 47n, Capacitor_SMD:C_0402_1005Metric, symbol Device:C
- removed C20: 100p, Capacitor_SMD:C_0402_1005Metric, symbol Device:C
- removed C21: NC, Capacitor_SMD:C_0402_1005Metric, symbol Device:C
- removed C22, C24: 1p, Capacitor_SMD:C_0402_1005Metric, symbol Device:C
- removed C25, C26, C27, C28, C29, C30: 12p, Capacitor_SMD:C_0402_1005Metric, symbol Device:C
- removed C32, C33, C34, C35: 100n, symbol Device:C
- removed C36: 1u, symbol Device:C
- removed C4, C5, C8: 4.7n, Capacitor_SMD:C_0402_1005Metric, symbol Device:C
- removed D1, D2, D3, D4, D5: LED, LED_SMD:LED_0402_1005Metric, symbol Device:LED
- removed FB1: fb, Resistor_SMD:R_0603_1608Metric, symbol Device:FerriteBead_Small
- removed IC1: DW3210, AutoBotfootprintlibrary:QFN40P500X500X80-40N-D, symbol AutoBotLibrary:DW3210
- removed J1: USB_C_Receptacle_USB2.0_16P, Connector_USB:USB_C_Receptacle_GCT_USB4105-xx-A_16P_TopMnt_Horizontal, symbol Connector:USB_C_Receptacle_USB2.0_16P
- removed J2, J4: Conn_01x05_Pin, Connector_PinHeader_2.54mm:PinHeader_1x05_P2.54mm_Vertical, symbol Connector:Conn_01x05_Pin
- removed J3, J6: Conn_01x04_Pin, Connector_PinHeader_2.54mm:PinHeader_1x04_P2.54mm_Vertical, symbol Connector:Conn_01x04_Pin
- removed J5: Conn_01x02_Pin, Connector_PinHeader_2.54mm:PinHeader_1x02_P2.54mm_Vertical, symbol Connector:Conn_01x02_Pin
- removed J7, J8: Conn_Coaxial, Connector_Coaxial:U.FL_Hirose_U.FL-R-SMT-1_Vertical, symbol Connector:Conn_Coaxial
- removed L1: 2.2n, Inductor_SMD:L_0402_1005Metric, symbol Device:L
- removed L2: 4.7n, Inductor_SMD:L_0402_1005Metric, symbol Device:L
- removed L3: 10u, Inductor_SMD:L_0603_1608Metric, symbol Device:L
- removed L4: 15u, Inductor_SMD:L_0603_1608Metric, symbol Device:L
- removed Q1, Q2, Q3: DMG1012T, Package_TO_SOT_SMD:SOT-523, symbol Transistor_FET:DMG1012T
- removed R1, R16, R2: 5.1k, Resistor_SMD:R_0402_1005Metric, symbol Device:R
- removed R10: 100K, Resistor_SMD:R_0402_1005Metric, symbol Device:R
- removed R11, R12, R6, R7, R9: R, Resistor_SMD:R_0402_1005Metric, symbol Device:R
- removed R13, R17, R18, R19, R5: 10k, Resistor_SMD:R_0402_1005Metric, symbol Device:R
- removed R14: 1k, Resistor_SMD:R_0402_1005Metric, symbol Device:R
- removed R15: 2.2k, Resistor_SMD:R_0402_1005Metric, symbol Device:R
- removed R3, R4: 2.2K, Resistor_SMD:R_0402_1005Metric, symbol Device:R
- removed SW1: reset, symbol Switch:SW_Push
- removed SW3: SW_DIP_x05, symbol Switch:SW_DIP_x05
- removed U1: BQ24075RGT, Package_DFN_QFN:VQFN-16-1EP_3x3mm_P0.5mm_EP1.6x1.6mm, symbol Battery_Management:BQ24075RGT
- removed U2: NRF52840-QFAA-R7, AutoBotfootprintlibrary:QFN48_NRF52840-QFAA-R7_NOR, symbol AutoBotLibrary:NRF52840-QFAA-R7
- removed U3: AP7370-33FDC, Package_DFN_QFN:DFN-6-1EP_2x2mm_P0.65mm_EP1.01x1.7mm, symbol Regulator_Linear:AP7370-33FDC
- removed Y1: TXC 8Y38472012, Crystal:Crystal_SMD_2016-4Pin_2.0x1.6mm, symbol Device:Crystal_GND24
- removed Y2: ECS-320-8-37B-CKY-TR, Crystal:Crystal_SMD_2016-4Pin_2.0x1.6mm, symbol Device:Crystal_GND24
- removed Y3: ECS-.327-6-1210B-N-TR, Crystal:Crystal_SMD_2016-4Pin_2.0x1.6mm, symbol Device:Crystal_GND24
Connections:
- no-connect marks 11 -> 0
Other:
- note removed: "1u for pin 48"
- note removed: "32.768KHZ"
- note removed: "32MHZ"
- note removed: "ANCHOR"
- note removed: "ANCHOR ID, MASTER/SLAVE SEL"
- note removed: "ANTENNAS"
- note removed: "BATTERY"
- note removed: "BLUE"
- note removed: "C24 IS NOT A LOAD CAPACITOR C25 C26 VALUE NOT CONFIRMED TARGET 10 PF"
- note removed: "CHARGING IC LEDS"
- note removed: "CRYSTAL"
- note removed: "CRYSTALS"
- note removed: "DEBUGGING"
- note removed: "DECOUPLING CAPS"
- note removed: "DW3210 GPIO"
- note removed: "DW3220 UWB TRANSCEIVER"
- note removed: "GREEN"
- note removed: "LED INDICATORS"
- note removed: "MAYBE PLACE CAPACITOR FOR DCC"
- note removed: "NRF 52840 QFAA R7"
- note removed: "NRF GPIO"
- note removed: "POWER"
- note removed: "RED"
- note removed: "TEMP VALUES, TARGET 6 PF"
- note removed: "TEMP VALUES, TARGET 8 PF"
- note removed: "USBC"
- note removed: "USE DW3220 FOR PDOA SUPPORT"
- note removed: "decoup cap prolly not req"
- note removed: "might use the antenna for wireless flashing"
- note removed: "resistor value shall be determined by whats already on the schematic"
