File: ELECTRONICS/ANCHOR/robot.kicad_sch (KiCad schematic)
At the start: 83 parts, among them IC2 DW3210, IC3 DW3210, J9 USB_C_Receptacle_USB2.0_16P, Q4 TBD_N, Q5 TBD_N, Q6 TBD_P, U4 STM32H7A3ZITx, U5 HUSB238_xxxDD, U6 BQ24170RGYR, U7 LM5175RHF

Commit message: Add files via upload
Parts:
- removed C79: C, symbol Device:C
- removed U4: STM32H7A3ZITx, Package_QFP:LQFP-144_20x20mm_P0.5mm, symbol MCU_ST_STM32H7:STM32H7A3ZITx
- added C107, C108, C109, C110, C111, C112, C113, C114, C115, C116, C118, C119, C120, C121, C80, C81: 100n, symbol Device:C
- added C117: 4u7, symbol Device:C
- added C122, C127: 100uF, Capacitor_Tantalum_SMD:CP_EIA-6032-28_Kemet-C, symbol Device:C_Polarized
- added C123, C125, C126, C128, C130, C131: 100nF, Capacitor_SMD:C_0402_1005Metric, symbol Device:C_Small
- added C124, C129: 22nF, Capacitor_SMD:C_0402_1005Metric, symbol Device:C_Small
- added C79: 68u, symbol Device:C_Polarized
- added C82: 22u, symbol Device:C
- added C83: 47p, symbol Device:C
- added C84, C85, C86: 10u, symbol Device:C
- added C87: 220n, symbol Device:C
- added C88: 220u, symbol Device:C
- added C89: 680u, symbol Device:C
- added C90, C91, C92, C93, C94, C95: 1u, symbol Device:C
- added D10, D7, D9: good diode fr, Diode_SMD:D_SOD-123, symbol Diode:1N4148W
- added D11, D12: D, symbol Device:D
- added D8: CDBK0520L-HF/EQ, Diode_SMD:D_SOD-123, symbol Diode:1N4148W
- added J10: MA, TerminalBlock_Phoenix:TerminalBlock_Phoenix_PT-1,5-4-3.5-H_1x04_P3.50mm_Horizontal, symbol Connector:Screw_Terminal_01x04
- added J11: MB, TerminalBlock_Phoenix:TerminalBlock_Phoenix_PT-1,5-4-3.5-H_1x04_P3.50mm_Horizontal, symbol Connector:Screw_Terminal_01x04
- added L6: 2.6u, symbol Device:L
- added L7: 33u, symbol Device:L
- added Q10, Q7, Q8, Q9: TBD_N, Package_TO_SOT_SMD:SOT-23, symbol Transistor_FET:DMG2302U
- added R43: 249k, symbol Device:R
- added R44: 5m, symbol Device:R
- added R45: 576k, symbol Device:R
- added R46: 20k, symbol Device:R
- added R47: 68.1k, symbol Device:R
- added R48: 10, symbol Device:R
- added R49, R50, R51, R58: 10k, symbol Device:R
- added R59, R60, R65, R66: 0.1, Resistor_SMD:R_1206_3216Metric, symbol Device:R
- added R61, R62: 1K, Resistor_SMD:R_0402_1005Metric, symbol Device:R
- added R63, R64: 10k, Resistor_SMD:R_0402_1005Metric, symbol Device:R
- added SW2, SW4: RESET, symbol Switch:SW_Push
- added U10, U11, U12: LP5907MFX-3.3, Package_TO_SOT_SMD:SOT-23-5, symbol Regulator_Linear:LP5907MFX-3.3
- added U13: STM32H7A3ZITx, Package_QFP:LQFP-144_20x20mm_P0.5mm, symbol AutoBotLibrary:STM32H7A3ZITx
- added U14, U4: BMI270, BMI270_BOS, symbol AutoBotLibrary:BMI270
- added U15, U16: (no value), MyFootprintLibrary:tmc2209, symbol My-Kicad-Library:TMC2209
- added U17: TVS1400DRV, Package_SON:WSON-6-1EP_2x2mm_P0.65mm_EP1x1.6mm, symbol Power_Protection:TVS1400DRV
- added U8: LM2596S-5, Package_TO_SOT_SMD:TO-263-5_TabPin3, symbol Regulator_Switching:LM2596S-5
- C74: value 1u-4u7 -> 1u
- C75: value C -> 68n
- C76: value C -> 120p
- C77: value C -> 10n
- C78: value C -> 47p
- R40: value R -> 86.6k
- R41: value R -> 23.7k
- R42: value R -> 93.1k
- U6: now not fitted
Connections:
- net +3V3: now also C107.1, C108.1, C109.1, C110.1, C111.1, C112.1, C113.1, C114.1, C115.1, C116.1, C117.1, C118.1, C119.1, C120.1, C121.1, C126.1, C131.1, C91.1, C93.1, C95.1, R49.1, R50.1, R51.1, R58.1, R63.2, R64.2, U10.5 (OUT), U11.5 (OUT), U12.5 (OUT), U13.108 (VDD), U13.121 (VDDMMC), U13.131 (VDD), U13.143 (PDR_ON), U13.144 (VDD), U13.17 (VDD), U13.30 (VDD), U13.33 (VDDA), U13.39 (VDD), U13.52 (VDD), U13.6 (VBAT), U13.62 (VDD), U13.72 (VDD), U13.84 (VDD), U13.95 (VDD33_USB), U14.5 (VDDIO), U14.8 (VDD), U15.10 (MS2_AD1), U15.15 (VCC_IO), U16.10 (MS2_AD1), U16.15 (VCC_IO), U4.5 (VDDIO), U4.8 (VDD)
- net AGND: now also C77.1, U7.2 (DITH); no longer R41.1
- net GNDREF: now also U7.12 (CSG), U7.19 (PGND), U7.29 (PowerPAD), U7.7 (AGND), C107.2, C108.2, C109.2, C110.2, C111.2, C112.2, C113.2, C114.2, C115.2, C116.2, C117.2, C118.2, C119.2, C120.2, C121.2, C122.2, C123.2, C126.2, C127.2, C128.2, C131.2, C79.2, C82.2, C83.2, C84.2, C85.2, C86.2, C87.2, C88.2, C89.2, C90.2, C91.2, C92.2, C93.2, C94.2, C95.2, D12.2 (A), R44.2, R46.2, R47.2, R59.2, R60.2, R65.2, R66.2, SW2.1, SW4.1, U10.2 (GND), U11.2 (GND), U12.2 (GND), U13.138 (BOOT0), U14.6 (GNDIO), U14.7 (GND), U15.13 (CLK), U15.18 (GND), U15.25 (GND), U15.29 (GND), U15.3 (GND), U15.9 (MS1_AD0), U16.13 (CLK), U16.18 (GND), U16.25 (GND), U16.29 (GND), U16.3 (GND), U16.9 (MS1_AD0), U17.1 (GND), U17.2 (GND), U17.3 (GND), U17.7 (GND), U4.6 (GNDIO), U4.7 (GND), U8.3 (GND), U8.5 (~{ON}/OFF)
- net VBAT: now also C79.1, C82.1, C89.1, D11.2 (A), Q7.3 (D), R43.1, U8.1 (VIN); no longer U7.26 (EN/UVLO), U7.27 (VIN)
- net VBUS: now also U17.4 (IN), U17.5 (IN), U17.6 (IN)
- net CC1: now reaches J9.A5 (CC1), U5.4 (CC1)
- net CC2: now reaches J9.B5 (CC2), U5.5 (CC2)
- net at R41.2: now also C78.2, U7.6 (COMP); no longer C77.1
- net VCC: now reaches C74.2, U7.20 (VCC)
- net VCC: now also D7.2 (A), D8.2 (A)
- net at U7.10 (ISNS(-)): now also U7.11 (ISNS(+))
- net at U7.13 (CS): now also C83.1, D9.2 (A), Q10.2 (S), Q8.2 (S), R44.1
- net SW2: now reaches U7.15 (SW2)
- net SW2: now also C81.1
- net HDRV2: now reaches U7.16 (HDRV2)
- net HDRV2: now also Q9.1 (G)
- net at U7.17 (BOOT2): now also C81.2, D8.1 (K)
- net LDRV2: now reaches U7.18 (LDRV2)
- net LDRV2: now also Q10.1 (G)
- net +24V: now reaches U7.21 (BIAS)
- net +24V: now also U7.9 (VOSNS), C122.1, C123.1, C124.1, C127.1, C128.1, C129.1, C84.1, C85.1, C86.1, D10.1 (K), Q9.3 (D), R45.1, U15.22 (VS), U15.28 (VS), U16.22 (VS), U16.28 (VS)
- net at U7.22 (LDRV1): now also Q8.1 (G)
- net at U7.23 (BOOT1): now also C80.1, D7.1 (K)
- net HDRV1: now reaches U7.24 (HDRV1)
- net HDRV1: now also Q7.1 (G)
- net at U7.25 (SW1): now also C80.2, D9.1 (K), L6.1, Q7.2 (S), Q8.3 (D)
- net at U7.8 (FB): now also R45.2, R46.1
- new net: R66.1, U16.23 (BRA)
- new net: C129.2, U16.6 (VCP)
- new net: C77.2, R41.1
- new net: D12.1 (K), L7.1, U8.2 (OUT)
- new net: C124.2, U15.6 (VCP)
- new net: R60.1, U15.23 (BRA)
- new net: R59.1, U15.27 (BRB)
- new net: C125.2, U15.4 (CP0)
- new net: C125.1, U15.5 (CPI)
- new net: D10.2 (A), L6.2, Q10.3 (D), Q9.2 (S)
- new net: R43.2, R47.1, U7.26 (EN/UVLO)
- new net: C87.1, R48.2, U7.27 (VIN)
- new net: C130.1, U16.5 (CPI)
- new net: C130.2, U16.4 (CP0)
- new net: R65.1, U16.27 (BRB)
- new net: R50.2, SW4.2
- new net: D11.1 (K), R48.1
- new net: U13.107 (VSS), U13.120 (VSS), U13.130 (VSS), U13.16 (VSS), U13.38 (VSS), U13.51 (VSS), U13.61 (VSS), U13.83 (VSS), U13.94 (VSS)
- new net +5V: C88.1, C90.1, C92.1, C94.1, L7.2, U10.1 (IN), U10.3 (EN), U11.1 (IN), U11.3 (EN), U12.1 (IN), U12.3 (EN), U8.4 (FB)
- new net BMI_CS_1: U4.12 (CSB)
- new net BMI_CS_2: U14.12 (CSB)
- new net BMI_INT_1: R51.2, U4.4 (INT1)
- new net BMI_INT_2: R58.2, U14.4 (INT1)
- new net BMI_MISO_1: U14.1 (SDO), U4.1 (SDO)
- new net BMI_MOSI_1: U4.14 (SDX)
- new net BMI_MOSI_2: U14.14 (SDX)
- new net BMI_SCK_1: U4.13 (SCX)
- new net BMI_SCK_2: U14.13 (SCX)
- new net DIAG_1: U15.11 (DIAG)
- new net DIAG_2: U16.11 (DIAG)
- new net DIR_1: U15.19 (DIR)
- new net DIR_2: U16.19 (DIR)
- new net ENN: U15.2 (ENN), U16.2 (ENN)
- new net INDEX_1: U15.12 (INDEX)
- new net INDEX_2: U16.12 (INDEX)
- new net NRST: R49.2, SW2.2, U13.25 (NRST)
- new net OA1-A: J10.2 (Pin_2), U15.24 (OA1)
- new net OA1-B: J11.2 (Pin_2), U16.24 (OA1)
- new net OA2-A: J10.1 (Pin_1), U15.21 (OA2)
- new net OA2-B: J11.1 (Pin_1), U16.21 (OA2)
- new net OB1-A: J10.3 (Pin_3), U15.26 (OB1)
- new net OB1-B: J11.3 (Pin_3), U16.26 (OB1)
- new net OB2-A: J10.4 (Pin_4), U15.1 (OB2)
- new net OB2-B: J11.4 (Pin_4), U16.1 (OB2)
- new net RXD0: R62.2, R64.1, U15.14 (PDN_UART)
- new net RXD1: R61.2, R63.1, U16.14 (PDN_UART)
- new net STEP_1: U15.16 (STEP)
- new net STEP_2: U16.16 (STEP)
- new net TXD0: R62.1
- new net TXD1: R61.1
- no-connect marks 4 -> 20
Other:
- note added: "avg current monitoring disabled"
- note added: "dw3220 gets separate ldos"
- note added: "prolly not gon use dith so maybe tie to gnd"
- moved on the sheet: C74, C75, C76, C77, C78, R23, R24, R40, R41, R42, U5, U7

Commit message: Add files via upload
Parts:
- removed R50: 10k, symbol Device:R
- removed SW2, SW4: RESET, symbol Switch:SW_Push
- removed U13: STM32H7A3ZITx, Package_QFP:LQFP-144_20x20mm_P0.5mm, symbol AutoBotLibrary:STM32H7A3ZITx
- added C96: 100n, symbol Device:C
- added R53: 10k, symbol Device:R
- added SW6: BOOT, symbol Switch:SW_Push
- added SW7: RESET, symbol Switch:SW_Push
- added U13: INA226, Package_SO:TSSOP-10_3x3mm_P0.5mm, symbol Sensor_Energy:INA226
- added U18, U19, U20, U21: (no value), symbol AutoBotLibrary:ADAFRUIT_VL53L1X_MODULE
- added U9: STM32H743ZITx, Package_QFP:LQFP-144_20x20mm_P0.5mm, symbol MCU_ST_STM32H7:STM32H743ZITx
- BT2: value Battery_Cell -> 3C
- R49: value 10k -> 5m
- U5: now not fitted
Connections:
- net BMI_MOSI_2 is gone; now on net BMI_MOSI: U14.14 (SDX)
- net BMI_SCK_2 is gone; now on net BMI_SCK: U14.13 (SCX)
- net +3V3: now also R53.1, U13.6 (VS), U18.1 (VIN), U19.1 (VIN), U20.1 (VIN), U21.1 (VIN), U9.108 (VDD), U9.121 (VDD), U9.131 (VDD), U9.143 (PDR_ON), U9.144 (VDD), U9.17 (VDD), U9.30 (VDD), U9.33 (VDDA), U9.39 (VDD), U9.52 (VDD), U9.6 (VBAT), U9.62 (VDD), U9.72 (VDD), U9.84 (VDD), U9.95 (VDD33_USB); no longer R49.1
- net BMI_CS_1: now also U9.92 (PG7)
- net BMI_CS_2: now also U9.93 (PG8)
- net BMI_INT_1: now also U9.125 (PG10)
- net BMI_INT_2: now also U9.126 (PG11)
- net D+: now also U9.104 (PA12)
- net D-: now also U9.103 (PA11)
- net DIAG_1: now also U9.88 (PG3)
- net DIAG_2: now also U9.90 (PG5)
- net DIR_1: now also U9.57 (PG1)
- net DIR_2: now also U9.91 (PG6)
- net DW_RST_1: now also U9.69 (PB10)
- net DW_RST_2: now also U9.115 (PD1)
- net GNDREF: now also C96.2, SW6.1, SW7.1, U13.1 (A1), U13.2 (A0), U13.7 (GND), U18.2 (GND), U19.2 (GND), U20.2 (GND), U21.2 (GND), U9.138 (BOOT0)
- net INDEX_1: now also U9.87 (PG2)
- net INDEX_2: now also U9.89 (PG4)
- net IRQ_1: now also U9.128 (PG13); no longer IC3.1 (IRQ/_GPIO8), R21.1
- net NRST: now also C96.1, SW7.2, U9.25 (NRST); no longer R49.2
- net RXD0: now also U9.18 (PF6)
- net RXD1: now also U9.141 (PE0)
- net STEP_1: now also U9.60 (PE9)
- net STEP_2: now also U9.64 (PE11)
- net TXD0: now also U9.19 (PF7)
- net TXD1: now also U9.142 (PE1)
- net WAKEUP_1: now also U9.70 (PB11)
- net WAKEUP_2: now also U9.116 (PD2)
- net BMI_MISO_1 renamed BMI_MISO
- net BMI_MISO: now also U9.42 (PA6)
- net BMI_MOSI_1 renamed BMI_MOSI
- net BMI_MOSI: now also U9.43 (PA7)
- net BMI_SCK_1 renamed BMI_SCK
- net BMI_SCK: now also U9.41 (PA5)
- net ENN renamed TMC_EN
- net TMC_EN: now also U9.56 (PG0)
- net EXTON_1: no longer names the net of IC2.31 (EXTON)
- net EXTON_2: no longer names the net of IC3.31 (EXTON)
- net SPICLK_1 renamed DW_CLK_1
- net DW_CLK_1: now also U9.74 (PB13)
- net SPICLK_2 renamed DW_CLK_2
- net DW_CLK_2: now also U9.111 (PC10)
- net SPICSN_1 renamed DW_CSN_1
- net DW_CSN_1: now also U9.114 (PD0), U9.73 (PB12)
- net SPICSN_2 renamed DW_CSN_2
- net SPIMISO_1 renamed DW_MISO_1
- net DW_MISO_1: now also U9.75 (PB14)
- net SPIMISO_2 renamed DW_MISO_2
- net DW_MISO_2: now also U9.112 (PC11)
- net SPIMOSI_1 renamed DW_MOSI_1
- net DW_MOSI_1: now also U9.76 (PB15)
- net SPIMOSI_2 renamed DW_MOSI_2
- net DW_MOSI_2: now also U9.113 (PC12)
- net VBAT renamed INA_VIN-
- net INA_VIN-: now also R49.2, U13.8 (Vbus), U13.9 (Vin-); no longer BT2.1 (+)
- new net: U9.107 (VSS), U9.120 (VSS), U9.130 (VSS), U9.16 (VSS), U9.38 (VSS), U9.51 (VSS), U9.61 (VSS), U9.83 (VSS), U9.94 (VSS)
- new net: R53.2, SW6.2
- new net ALERT: U13.3 (~{Alert}), U9.124 (PG9)
- new net INA_SCL: U13.5 (SCL)
- new net INA_SDA: U13.4 (SDA)
- new net INA_VIN+: BT2.1 (+), R49.1, U13.10 (Vin+)
- new net IRQ_2: IC3.1 (IRQ/_GPIO8), R21.1, U9.129 (PG14)
- new net VL_IO1: U18.5 (GPIO)
- new net VL_IO2: U19.5 (GPIO)
- new net VL_IO3: U20.5 (GPIO)
- new net VL_IO4: U21.5 (GPIO)
- new net VL_SCL1: U18.3 (SCL)
- new net VL_SCL2: U19.3 (SCL)
- new net VL_SCL3: U20.3 (SCL)
- new net VL_SCL4: U21.3 (SCL)
- new net VL_SDA1: U18.4 (SDA)
- new net VL_SDA2: U19.4 (SDA)
- new net VL_SDA3: U20.4 (SDA)
- new net VL_SDA4: U21.4 (SDA)
- new net VL_XSHUT1: U18. (XSHUT)
- new net VL_XSHUT2: U19. (XSHUT)
- new net VL_XSHUT3: U20. (XSHUT)
- new net VL_XSHUT4: U21. (XSHUT)
- no-connect marks 20 -> 22
Other:
- note added: "ADDRESS: 1000000"
- note added: "OMIT FOR V1 USE BMS INSTEAD"
- note added: "PROBABLY JUST GROUND GPIO5 AND GPIO 6"
- note added: "PROLLY OMIT THIS TOO FOR V1"
- note added: "PWM"
- note added: "THIS IS TEMPORARY PLACEMENT"
- note added: "maybe something smaller"
- moved on the sheet: C107, C108, C109, C110, C111, C112, C113, C114, C115, C116, C117
