File: ELECTRONICS/ANCHOR/AutoBot.kicad_pcb (KiCad board)
At the start: 4 copper layers, 78 parts, among them IC1 DW3210, J1 USB_C_Receptacle_USB2.0_16P, J2 Conn_01x05_Pin, J3 Conn_01x04_Pin, J4 Conn_01x05_Pin, J5 Conn_01x02_Pin, J6 Conn_01x04_Pin, J7 Conn_Coaxial, J8 Conn_Coaxial, J9 Conn_01x02_Pin, Q1 DMG1012T, Q2 DMG1012T, Q3 DMG1012T, U1 BQ24075RGT, U2 NRF52840-QFAA-R7, U3 AP7370-33FDC, Y1 TXC 8Y38472012, Y2 ECS-320-8-37B-CKY-TR, Y3 ECS-.327-6-1210B-N-TR

Commit message: Add files via upload
Parts:
- added C122: 100uF, Capacitor_Tantalum_SMD:CP_EIA-6032-28_Kemet-C, F.Cu at (216.7, 80.3)
- added C123: 100nF, Capacitor_SMD:C_0402_1005Metric, F.Cu at (219.5, 76.9)
- added C124: 22nF, Capacitor_SMD:C_0402_1005Metric, F.Cu at (222.4, 61.1)
- added C125: 100nF, Capacitor_SMD:C_0402_1005Metric, F.Cu at (222.4, 63.1)
- added C126: 100nF, Capacitor_SMD:C_0402_1005Metric, F.Cu at (222.4, 65.1)
- added C127: 100uF, Capacitor_Tantalum_SMD:CP_EIA-6032-28_Kemet-C, F.Cu at (216.7, 85.0)
- added C128: 100nF, Capacitor_SMD:C_0402_1005Metric, F.Cu at (222.4, 67.0)
- added C129: 22nF, Capacitor_SMD:C_0402_1005Metric, F.Cu at (222.4, 69.0)
- added C130: 100nF, Capacitor_SMD:C_0402_1005Metric, F.Cu at (222.4, 71.0)
- added C131: 100nF, Capacitor_SMD:C_0402_1005Metric, F.Cu at (222.4, 73.0)
- added C37: 2p, Capacitor_SMD:C_0402_1005Metric, F.Cu at (213.8, 61.1)
- added C38: 2p, Capacitor_SMD:C_0402_1005Metric, F.Cu at (213.8, 63.1)
- added C39: 100n, Capacitor_SMD:C_0402_1005Metric, F.Cu at (213.8, 65.1)
- added C40: 4.7n, Capacitor_SMD:C_0402_1005Metric, F.Cu at (213.8, 67.0)
- added C41: 4.7n, Capacitor_SMD:C_0402_1005Metric, F.Cu at (213.8, 69.0)
- added C42: 4.7n, Capacitor_SMD:C_0402_1005Metric, F.Cu at (213.8, 71.0)
- added C43: 220n, Capacitor_SMD:C_0402_1005Metric, F.Cu at (213.8, 73.0)
- added C44: 100n, Capacitor_SMD:C_0402_1005Metric, F.Cu at (213.8, 74.9)
- added C45: 100n, Capacitor_SMD:C_0402_1005Metric, F.Cu at (213.8, 76.9)
- added C46: 100n, Capacitor_SMD:C_0402_1005Metric, F.Cu at (216.7, 61.1)
- added C47: 4.7u, Capacitor_SMD:C_0402_1005Metric, F.Cu at (216.7, 63.1)
- added C48: 10u, Capacitor_SMD:C_0402_1005Metric, F.Cu at (216.7, 65.1)
- added C49: 10u, Capacitor_SMD:C_0402_1005Metric, F.Cu at (216.7, 67.0)
- added C50: 2p, Capacitor_SMD:C_0402_1005Metric, F.Cu at (216.7, 69.0)
- added C51: 2p, Capacitor_SMD:C_0402_1005Metric, F.Cu at (216.7, 71.0)
- added C52: 100n, Capacitor_SMD:C_0402_1005Metric, F.Cu at (216.7, 73.0)
- added C53: 4.7n, Capacitor_SMD:C_0402_1005Metric, F.Cu at (216.7, 74.9)
- added C54: 4.7n, Capacitor_SMD:C_0402_1005Metric, F.Cu at (216.7, 76.9)
- added C55: 4.7n, Capacitor_SMD:C_0402_1005Metric, F.Cu at (219.5, 61.1)
- added C56: 220n, Capacitor_SMD:C_0402_1005Metric, F.Cu at (219.5, 63.1)
- added C57: 100n, Capacitor_SMD:C_0402_1005Metric, F.Cu at (219.5, 65.1)
- added C58: 100n, Capacitor_SMD:C_0402_1005Metric, F.Cu at (219.5, 67.0)
- added C59: 100n, Capacitor_SMD:C_0402_1005Metric, F.Cu at (219.5, 69.0)
- added C60: 4.7u, Capacitor_SMD:C_0402_1005Metric, F.Cu at (219.5, 71.0)
- added C61: 10u, Capacitor_SMD:C_0402_1005Metric, F.Cu at (219.5, 73.0)
- added C62: 10u, Capacitor_SMD:C_0402_1005Metric, F.Cu at (219.5, 74.9)
- added D10: good diode fr, Diode_SMD:D_SOD-123, F.Cu at (194.8, 47.5)
- added D15: CDBK0520L-HF/EQ, Diode_SMD:D_SOD-123, F.Cu at (194.8, 50.9)
- added D16: CDBK0520L-HF/EQ, Diode_SMD:D_SOD-123, F.Cu at (194.8, 54.2)
- added D17: CDBK0520L-HF/EQ, Diode_SMD:D_SOD-123, F.Cu at (194.8, 57.6)
- added D18: CDBK0520L-HF/EQ, Diode_SMD:D_SOD-123, F.Cu at (194.8, 60.9)
- added D7: good diode fr, Diode_SMD:D_SOD-123, F.Cu at (194.8, 37.5)
- added D8: CDBK0520L-HF/EQ, Diode_SMD:D_SOD-123, F.Cu at (194.8, 40.8)
- added D9: good diode fr, Diode_SMD:D_SOD-123, F.Cu at (194.8, 44.2)
- added FB2: fb, Resistor_SMD:R_0603_1608Metric, F.Cu at (193.9, 80.3)
- added FB3: fb, Resistor_SMD:R_0603_1608Metric, F.Cu at (193.9, 82.9)
- added IC2: DW3210, AutoBotfootprintlibrary:QFN40P500X500X80-40N-D, F.Cu at (234.9, 76.2)
- added IC3: DW3210, AutoBotfootprintlibrary:QFN40P500X500X80-40N-D, F.Cu at (234.9, 83.5)
- added J10: MA, TerminalBlock_Phoenix:TerminalBlock_Phoenix_PT-1,5-4-3.5-H_1x04_P3.50mm_Horizontal, F.Cu at (224.8, 39.9)
- added J11: MB, TerminalBlock_Phoenix:TerminalBlock_Phoenix_PT-1,5-4-3.5-H_1x04_P3.50mm_Horizontal, F.Cu at (224.8, 49.8)
- added Q10: TBD_N, Package_TO_SOT_SMD:SOT-23, F.Cu at (205.0, 71.3)
- added Q15: TBD_N, Package_TO_SOT_SMD:SOT-23, F.Cu at (205.0, 75.7)
- added Q16: TBD_N, Package_TO_SOT_SMD:SOT-23, F.Cu at (209.9, 62.4)
- added Q17: TBD_N, Package_TO_SOT_SMD:SOT-23, F.Cu at (209.9, 66.8)
- added Q18: TBD_N, Package_TO_SOT_SMD:SOT-23, F.Cu at (209.9, 71.3)
- added Q4: TBD_N, Package_TO_SOT_SMD:SOT-23, F.Cu at (200.1, 62.4)
- added Q5: TBD_N, Package_TO_SOT_SMD:SOT-23, F.Cu at (200.1, 66.8)
- added Q6: TBD_P, Package_TO_SOT_SMD:SOT-23, F.Cu at (200.1, 71.3)
- added Q7: TBD_N, Package_TO_SOT_SMD:SOT-23, F.Cu at (200.1, 75.7)
- added Q8: TBD_N, Package_TO_SOT_SMD:SOT-23, F.Cu at (205.0, 62.4)
- added Q9: TBD_N, Package_TO_SOT_SMD:SOT-23, F.Cu at (205.0, 66.8)
- added R20: 100K, Resistor_SMD:R_0402_1005Metric, F.Cu at (193.3, 63.6)
- added R21: 100K, Resistor_SMD:R_0402_1005Metric, F.Cu at (193.3, 65.6)
- added R59: 0.1, Resistor_SMD:R_1206_3216Metric, F.Cu at (240.8, 37.5)
- added R60: 0.1, Resistor_SMD:R_1206_3216Metric, F.Cu at (240.8, 40.8)
- added R61: 1K, Resistor_SMD:R_0402_1005Metric, F.Cu at (193.3, 67.6)
- added R62: 1K, Resistor_SMD:R_0402_1005Metric, F.Cu at (193.3, 69.6)
- added R63: 10k, Resistor_SMD:R_0402_1005Metric, F.Cu at (193.3, 71.6)
- added R64: 10k, Resistor_SMD:R_0402_1005Metric, F.Cu at (193.3, 73.5)
- added R65: 0.1, Resistor_SMD:R_1206_3216Metric, F.Cu at (240.8, 44.1)
- added R66: 0.1, Resistor_SMD:R_1206_3216Metric, F.Cu at (240.8, 47.4)
- added U10: LP5907MFX-3.3, Package_TO_SOT_SMD:SOT-23-5, F.Cu at (241.2, 74.9)
- added U11: LP5907MFX-3.3, Package_TO_SOT_SMD:SOT-23-5, F.Cu at (241.2, 79.5)
- added U12: LP5907MFX-3.3, Package_TO_SOT_SMD:SOT-23-5, F.Cu at (241.2, 84.2)
- added U13: STM32H7A3ZITx, Package_QFP:LQFP-144_20x20mm_P0.5mm, F.Cu at (184.0, 119.2)
- added U15: ~, MyFootprintLibrary:tmc2209, F.Cu at (227.5, 76.1)
- added U16: ~, MyFootprintLibrary:tmc2209, F.Cu at (227.5, 83.6)
- added U17: TVS1400DRV, Package_SON:WSON-6-1EP_2x2mm_P0.65mm_EP1x1.6mm, F.Cu at (223.8, 57.5)
- added U5: HUSB238_xxxDD, Package_DFN_QFN:WDFN-10-1EP_3x3mm_P0.5mm_EP1.8x2.5mm, F.Cu at (194.9, 76.8)
- added U6: BQ24170RGYR, AutoBotfootprintlibrary:RGY24_2P05X3P1, F.Cu at (241.2, 53.0)
- added U7: LM5175RHF, Package_DFN_QFN:VQFN-28-1EP_4x5mm_P0.5mm_EP2.55x3.55mm, F.Cu at (201.2, 81.6)
- added U8: LM2596S-5, Package_TO_SOT_SMD:TO-263-5_TabPin3, F.Cu at (234.6, 66.3)
- added U9: LM5175RHF, Package_DFN_QFN:VQFN-28-1EP_4x5mm_P0.5mm_EP2.55x3.55mm, F.Cu at (207.9, 81.6)
- R14: value 10k -> 1k
- R15: value 10k -> 2.2k
- R16: value 10k -> 5.1k

Commit message: Add files via upload
Parts:
- moved U13 10.0 mm to (180.2, 109.8)
Changed lines of the file:
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@@
 	(footprint "Package_QFP:LQFP-144_20x20mm_P0.5mm"
 		(layer "F.Cu")
-		(at 184 119.15 180)
+		(at 180.25 109.85 180)
 		(descr "LQFP, 144 Pin (JEDEC MS-026 variation BFB, 1.40mm body thickness, https://www.jedec.org/document_search?search_api_views_fulltext=MS-026, https://ww1.microchip.com/downloads/en/PackagingSpec/00000049BQ.pdf#page=425)")
 		(tags "LQFP QFP Microchip_144-Lead-Plastic-Low-Profile-Quad-Flatpack-(PL) Microsemi_TQ144")

Commit message: Add files via upload
Parts:
- removed C122, C127: 100uF, Capacitor_Tantalum_SMD:CP_EIA-6032-28_Kemet-C
- removed C123, C125, C126, C128, C130, C131: 100nF, Capacitor_SMD:C_0402_1005Metric
- removed C124, C129: 22nF, Capacitor_SMD:C_0402_1005Metric
- removed C37, C38, C50, C51: 2p, Capacitor_SMD:C_0402_1005Metric
- removed C39, C44, C45, C46, C52, C57, C58, C59: 100n, Capacitor_SMD:C_0402_1005Metric
- removed C40, C41, C42, C53, C54, C55: 4.7n, Capacitor_SMD:C_0402_1005Metric
- removed C43, C56: 220n, Capacitor_SMD:C_0402_1005Metric
- removed C47, C60: 4.7u, Capacitor_SMD:C_0402_1005Metric
- removed C48, C49, C61, C62: 10u, Capacitor_SMD:C_0402_1005Metric
- removed D10, D7, D9: good diode fr, Diode_SMD:D_SOD-123
- removed D15, D16, D17, D18, D8: CDBK0520L-HF/EQ, Diode_SMD:D_SOD-123
- removed FB2, FB3: fb, Resistor_SMD:R_0603_1608Metric
- removed IC2, IC3: DW3210, AutoBotfootprintlibrary:QFN40P500X500X80-40N-D
- removed J10: MA, TerminalBlock_Phoenix:TerminalBlock_Phoenix_PT-1,5-4-3.5-H_1x04_P3.50mm_Horizontal
- removed J11: MB, TerminalBlock_Phoenix:TerminalBlock_Phoenix_PT-1,5-4-3.5-H_1x04_P3.50mm_Horizontal
- removed J9: Conn_01x02_Pin, Connector_JST:JST_PH_B2B-PH-K_1x02_P2.00mm_Vertical
- removed Q10, Q15, Q16, Q17, Q18, Q4, Q5, Q7, Q8, Q9: TBD_N, Package_TO_SOT_SMD:SOT-23
- removed Q6: TBD_P, Package_TO_SOT_SMD:SOT-23
- removed R20, R21: 100K, Resistor_SMD:R_0402_1005Metric
- removed R59, R60, R65, R66: 0.1, Resistor_SMD:R_1206_3216Metric
- removed R61, R62: 1K, Resistor_SMD:R_0402_1005Metric
- removed R63, R64: 10k, Resistor_SMD:R_0402_1005Metric
- removed U10, U11, U12: LP5907MFX-3.3, Package_TO_SOT_SMD:SOT-23-5
- removed U13: STM32H7A3ZITx, Package_QFP:LQFP-144_20x20mm_P0.5mm
- removed U15, U16: ~, MyFootprintLibrary:tmc2209
- removed U17: TVS1400DRV, Package_SON:WSON-6-1EP_2x2mm_P0.65mm_EP1x1.6mm
- removed U5: HUSB238_xxxDD, Package_DFN_QFN:WDFN-10-1EP_3x3mm_P0.5mm_EP1.8x2.5mm
- removed U6: BQ24170RGYR, AutoBotfootprintlibrary:RGY24_2P05X3P1
- removed U7, U9: LM5175RHF, Package_DFN_QFN:VQFN-28-1EP_4x5mm_P0.5mm_EP2.55x3.55mm
- removed U8: LM2596S-5, Package_TO_SOT_SMD:TO-263-5_TabPin3
- added C32: 100n, Capacitor_SMD:C_0402_1005Metric, F.Cu at (47.0, 65.9)
- added C33: 100n, Capacitor_SMD:C_0402_1005Metric, F.Cu at (40.9, 69.5)
- added C34: 100n, Capacitor_SMD:C_0402_1005Metric, F.Cu at (51.0, 69.6)
- added C35: 100n, Capacitor_SMD:C_0402_1005Metric, F.Cu at (42.4, 76.4)
- added C36: 1u, Capacitor_SMD:C_0402_1005Metric, F.Cu at (50.2, 76.5)
- C13, C31: footprint Capacitor_SMD:C_0402_1005Metric -> Capacitor_SMD:C_0201_0603Metric
- moved J7 117.6 mm to (36.0, 24.7)
- moved U1 115.4 mm to (40.4, 83.7), turned to 0 degrees
- moved U2 109.9 mm to (46.0, 72.5)
- moved J1 109.5 mm to (46.0, 92.5)
- moved IC1 109.3 mm to (46.0, 47.5)
- moved FB1 104.8 mm to (4.76, 28.4)
- moved J8 103.2 mm to (56.0, 24.7)
- moved C31 90.6 mm to (47.0, 42.8), turned to -90 degrees
- moved L1 89.2 mm to (6.33, 37.3)
- moved L2 89.2 mm to (6.33, 39.3)
- moved R10 88.5 mm to (12.8, 37.9)
- moved R13 88.5 mm to (12.8, 43.9)
- moved R14 88.5 mm to (12.8, 45.9)
- moved R15 88.5 mm to (15.7, 37.9)
- moved R16 88.5 mm to (15.7, 39.9)
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Connections:
- C27 pad 1: /XC1 -> /XL1
- C28 pad 1: /XC2 -> /XL2
- J4 pad 1: /TRACECLK -> /TRACEDATA0
- J4 pad 2: /TRACEDATA0 -> /TRACEDATA1
- J4 pad 3: /TRACEDATA1 -> /TRACEDATA2
- J4 pad 4: /TRACEDATA2 -> /TRACEDATA3
- J4 pad 5: /TRACEDATA3 -> /TRACECLK
- U2 pad 18: /SPICLK -> /SPIMISO
- U2 pad 20: /SPIMISO -> /SPICLK
- Y2 pad 1: /XC1 -> /XL1
- Y2 pad 3: /XC2 -> /XL2
Routing:
- net /P0.28/AIN4: track 0.00 -> 25.3 mm
- net /P0.29/AIN5: track 0.00 -> 23.7 mm
- net /P0.30/AIN6: track 0.00 -> 22.2 mm
- net /TRACEDATA0: track 0.00 -> 21.8 mm, vias 0 -> 1
- net /P0.31/AIN7: track 0.00 -> 20.6 mm
- net /SPICSN: track 0.00 -> 20.1 mm
- net /DW_RF2: track 0.00 -> 19.7 mm
- net /DW_RF1: track 0.00 -> 19.7 mm
- net /DW_RST: track 0.00 -> 19.6 mm
- net /SPICLK: track 0.00 -> 19.6 mm
- net /SPIMISO: track 0.00 -> 19.6 mm
- net /SPIMOSI: track 0.00 -> 19.6 mm
- net /WAKEUP: track 0.00 -> 19.6 mm
- net /DW_GPIO7: track 0.00 -> 17.6 mm
- net /PGOOD: track 0.00 -> 17.5 mm, vias 0 -> 2
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Other:
- board outline added: 40 x 75 mm

Commit message: Add files via upload
Parts:
- FB1: footprint Resistor_SMD:R_0603_1608Metric -> Inductor_SMD:L_0402_1005Metric
- moved FB1 41.7 mm to (39.9, 50.9), turned to 180 degrees
- moved C24 36.0 mm to (38.2, 45.2), turned to 180 degrees
- moved C27 34.9 mm to (54.7, 73.3)
- moved C28 31.7 mm to (51.5, 74.8), turned to 90 degrees
- moved C26 29.9 mm to (42.9, 43.0), turned to 90 degrees
- moved C11 29.0 mm to (39.6, 49.7), turned to 180 degrees
- moved C25 24.9 mm to (40.3, 45.8), turned to 180 degrees
- moved C21 21.6 mm to (39.4, 70.6), turned to 180 degrees
- moved C30 21.1 mm to (41.0, 76.7), turned to -90 degrees
- moved C29 18.1 mm to (38.2, 73.7), turned to 180 degrees
- moved L3 17.8 mm to (49.1, 78.8), turned to 0 degrees
- moved Y2 14.7 mm to (53.5, 75.2), turned to 180 degrees
- moved C8 14.2 mm to (40.5, 47.6), turned to -90 degrees
- moved R18 12.9 mm to (18.0, 56.6)
- moved C2 12.0 mm to (41.9, 51.4)
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Routing:
- net GNDREF: track 0.00 -> 41.2 mm, vias 0 -> 41
- net +3V3: track 13.7 -> 42.3 mm, vias 2 -> 29
- net /SWDCLK: track 0.00 -> 17.2 mm, vias 0 -> 1
- net /SWDIO: track 0.00 -> 16.4 mm, vias 0 -> 1
- net /CHG: track 6.40 -> 17.7 mm, vias 0 -> 2
- net Net-(U2-DEC4): track 3.92 -> 13.3 mm, vias 0 -> 2
- net VBUS: track 10.2 -> 19.4 mm
- net /XL1: track 0.00 -> 6.69 mm
- net /XC1: track 0.00 -> 5.75 mm
- net Net-(IC1-VDD2A): track 0.00 -> 5.28 mm
- net /XL2: track 0.00 -> 4.33 mm
- net /XTO: track 0.00 -> 4.21 mm
- net Net-(IC1-VTX_D): track 0.00 -> 4.04 mm
- net /XC2: track 0.00 -> 3.89 mm
- net /XTI: track 0.00 -> 3.76 mm
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- added copper zone on F.Cu, net +3V3
- added copper zone on In2.Cu, net +3V3
- added copper zone on In1.Cu, net GNDREF

Commit message: Add files via upload
Parts:
- removed C14: 1.2p, Capacitor_SMD:C_0402_1005Metric
- removed C22: 1p, Capacitor_SMD:C_0402_1005Metric
- removed L1: 2.2n, Inductor_SMD:L_0402_1005Metric
- removed L2: 4.7n, Inductor_SMD:L_0402_1005Metric
- added SW3: SW_DIP_x05, MyFootprintLibrary:SW-SMD_2.54-5P-TPGT, F.Cu at (33.0, 59.2)
- moved R10 46.6 mm to (49.4, 66.8)
- moved C12 37.9 mm to (49.5, 51.4)
- moved C23 29.8 mm to (47.3, 77.9), turned to 90 degrees
- moved R17 24.4 mm to (37.5, 52.8), turned to 180 degrees
- moved R18 23.5 mm to (40.5, 63.7), turned to 180 degrees
- moved R16 23.2 mm to (35.0, 52.8), turned to 180 degrees
- moved R19 22.9 mm to (27.4, 65.6)
- moved R15 21.9 mm to (33.0, 51.4), turned to 90 degrees
- moved L4 18.5 mm to (48.2, 79.8), turned to 0 degrees
- moved R14 18.5 mm to (30.4, 51.4), turned to 90 degrees
- moved J5 17.4 mm to (27.7, 81.6), turned to 180 degrees
- moved R13 16.8 mm to (27.9, 51.4), turned to 90 degrees
- moved J3 2.47 mm to (27.7, 75.5)
- moved L3 1.40 mm to (50.5, 79.1), turned to 90 degrees
- moved C19 1.01 mm to (50.4, 75.8)
Connections:
- U2 pad 18: /SPIMISO -> /SPICLK
- U2 pad 20: /SPICLK -> /SPIMISO
- U2 pad 4: /MODE__SEL -> /MODE_SEL
Routing:
- net /MODE_SEL: track 0.00 -> 30.2 mm, vias 0 -> 2
- net /ID_SEL: track 1.26 -> 25.8 mm, vias 1 -> 2
- net /IRQ: track 0.00 -> 20.7 mm
- net /P0.09/NFC1: track 0.91 -> 18.4 mm
- net /P0.10/NFC2: track 1.91 -> 19.4 mm
- net Net-(U2-DCC): track 0.00 -> 5.04 mm
- net +3V3: track 42.3 -> 46.3 mm, vias 29 -> 34
- net /MODE__SEL: track 2.87 -> 0.00 mm, vias 1 -> 0
- net Net-(R13-Pad1): track 0.00 -> 2.85 mm
- net Net-(R14-Pad1): track 0.00 -> 2.79 mm
- net Net-(R15-Pad1): track 0.00 -> 2.75 mm
- net Net-(R16-Pad1): track 0.00 -> 1.96 mm
- net Net-(R17-Pad1): track 0.00 -> 1.91 mm
- net Net-(IC1-VIO_D): track 0.00 -> 1.87 mm
- net Net-(L3-Pad1): track 0.00 -> 1.52 mm
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