File: ELECTRONICS/MAINBOARD/MOTOR_CONNECTOR.kicad_sch (KiCad schematic)
At the start: 1 part, among them J4 MA

Commit message: Add files via upload
Parts:
- renumbered J4 to J2
Changed lines of the file:
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@@
 		(in_pos_files yes)
 		(dnp no)
-		(property "Reference" "J4"
+		(property "Reference" "J2"
 			(at 21.59 20.32 0)
 			(show_name no)
@@
 				)
 				(path "/f053f1d0-b1f5-4f80-9758-8ee1a2d3659d/8f5b1df0-1690-439e-a60a-46a43198f202"
-					(reference "J4")
+					(reference "J2")
 					(unit 1)
 				)
