File: ELECTRONICS/MAINBOARD/TMC2209.kicad_sch (KiCad schematic)
At the start: 11 parts, among them U3 TVS1400DRV

Commit message: 9/4
Parts:
- added C42: 100nF, Capacitor_SMD:C_0402_1005Metric, symbol Device:C_Small
Connections:
- net 24V: now also C42.1
- net GNDREF: now also C42.2
Other:
- moved on the sheet: C6, C8, U3

Commit message: Add files via upload
Parts:
- renumbered C11 to C10, C12 to C11, C16 to C12, C6 to C7, C42 to C9, R11 to R10, R5 to R7, R6 to R8, R13 to R9, U3 to U5, U8 to U6
Changed lines of the file:
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@@
 		(dnp no)
 		(fields_autoplaced yes)
-		(property "Reference" "U3"
+		(property "Reference" "U5"
 			(at 52.07 57.1499 0)
 			(show_name no)
@@
 			(project "autobot_mainboard"
 				(path "/f053f1d0-b1f5-4f80-9758-8ee1a2d3659d/33095814-6a92-4caa-8704-b20bd44a0045"
-					(reference "U4")
-					(unit 1)
-				)
-				(path "/f053f1d0-b1f5-4f80-9758-8ee1a2d3659d/39e7d174-ffe7-4b4e-a983-e2abb212b9b6"
-					(reference "U3")
+					(reference "U7")
+					(unit 1)
+				)
+				(path "/f053f1d0-b1f5-4f80-9758-8ee1a2d3659d/39e7d174-ffe7-4b4e-a983-e2abb212b9b6"
+					(reference "U5")
 					(unit 1)
 				)
@@
 		(in_pos_files yes)
 		(dnp no)
-		(property "Reference" "R5"
+		(property "Reference" "R7"
 			(at 125.222 92.964 0)
 			(show_name no)
@@
 			(project "autobot_mainboard"
 				(path "/f053f1d0-b1f5-4f80-9758-8ee1a2d3659d/33095814-6a92-4caa-8704-b20bd44a0045"
+					(reference "R11")
+					(unit 1)
+				)
+				(path "/f053f1d0-b1f5-4f80-9758-8ee1a2d3659d/39e7d174-ffe7-4b4e-a983-e2abb212b9b6"
 					(reference "R7")
-					(unit 1)
-				)
-				(path "/f053f1d0-b1f5-4f80-9758-8ee1a2d3659d/39e7d174-ffe7-4b4e-a983-e2abb212b9b6"
-					(reference "R5")
 					(unit 1)
 				)
@@
 		(in_pos_files yes)
 		(dnp no)
-		(property "Reference" "#PWR017"
+		(property "Reference" "#PWR025"
 			(at 170.18 35.56 0)
 			(hide yes)
@@
 			(project "autobot_mainboard"
 				(path "/f053f1d0-b1f5-4f80-9758-8ee1a2d3659d/33095814-6a92-4caa-8704-b20bd44a0045"
-					(reference "#PWR020")
-					(unit 1)
-				)
-				(path "/f053f1d0-b1f5-4f80-9758-8ee1a2d3659d/39e7d174-ffe7-4b4e-a983-e2abb212b9b6"
-					(reference "#PWR017")
+					(reference "#PWR030")
+					(unit 1)
+				)
+				(path "/f053f1d0-b1f5-4f80-9758-8ee1a2d3659d/39e7d174-ffe7-4b4e-a983-e2abb212b9b6"
+					(reference "#PWR025")
 					(unit 1)
 				)
@@
 		(in_pos_files yes)
 		(dnp no)
-		(property "Reference" "C11"
+		(property "Reference" "C10"
 			(at 91.186 46.736 0)
 			(show_name no)
@@
 			(project "autobot_mainboard"
 				(path "/f053f1d0-b1f5-4f80-9758-8ee1a2d3659d/33095814-6a92-4caa-8704-b20bd44a0045"
-					(reference "C13")
-					(unit 1)
-				)
-				(path "/f053f1d0-b1f5-4f80-9758-8ee1a2d3659d/39e7d174-ffe7-4b4e-a983-e2abb212b9b6"
-					(reference "C11")
+					(reference "C16")
+					(unit 1)
+				)
+				(path "/f053f1d0-b1f5-4f80-9758-8ee1a2d3659d/39e7d174-ffe7-4b4e-a983-e2abb212b9b6"
+					(reference "C10")
 					(unit 1)
 				)
@@
 		(dnp no)
 		(fields_autoplaced yes)
-		(property "Reference" "U8"
+		(property "Reference" "U6"
 			(at 116.4433 90.17 0)
 			(show_name no)
@@
 			(project "autobot_mainboard"
 				(path "/f053f1d0-b1f5-4f80-9758-8ee1a2d3659d/33095814-6a92-4caa-8704-b20bd44a0045"
-					(reference "U9")
-					(unit 1)
-				)
-				(path "/f053f1d0-b1f5-4f80-9758-8ee1a2d3659d/39e7d174-ffe7-4b4e-a983-e2abb212b9b6"
 					(reference "U8")
+					(unit 1)
+				)
+				(path "/f053f1d0-b1f5-4f80-9758-8ee1a2d3659d/39e7d174-ffe7-4b4e-a983-e2abb212b9b6"
+					(reference "U6")
 					(unit 1)
 				)
@@
 		(dnp no)
 		(fields_autoplaced yes)
-		(property "Reference" "#PWR08"
+		(property "Reference" "#PWR021"
 			(at 48.26 72.39 0)
 			(hide yes)
@@
 			(project "autobot_mainboard"
 				(path "/f053f1d0-b1f5-4f80-9758-8ee1a2d3659d/33095814-6a92-4caa-8704-b20bd44a0045"
-					(reference "#PWR09")
-					(unit 1)
-				)
-				(path "/f053f1d0-b1f5-4f80-9758-8ee1a2d3659d/39e7d174-ffe7-4b4e-a983-e2abb212b9b6"
-					(reference "#PWR08")
+					(reference "#PWR026")
+					(unit 1)
+				)
+				(path "/f053f1d0-b1f5-4f80-9758-8ee1a2d3659d/39e7d174-ffe7-4b4e-a983-e2abb212b9b6"
+					(reference "#PWR021")
 					(unit 1)
 				)
@@
 		(in_pos_files yes)
 		(dnp no)
-		(property "Reference" "R6"
+		(property "Reference" "R8"
 			(at 134.112 90.424 0)
 			(show_name no)
@@
 			(project "autobot_mainboard"
 				(path "/f053f1d0-b1f5-4f80-9758-8ee1a2d3659d/33095814-6a92-4caa-8704-b20bd44a0045"
+					(reference "R12")
+					(unit 1)
+				)
+				(path "/f053f1d0-b1f5-4f80-9758-8ee1a2d3659d/39e7d174-ffe7-4b4e-a983-e2abb212b9b6"
 					(reference "R8")
-					(unit 1)
-				)
-				(path "/f053f1d0-b1f5-4f80-9758-8ee1a2d3659d/39e7d174-ffe7-4b4e-a983-e2abb212b9b6"
-					(reference "R6")
 					(unit 1)
 				)
@@
 		(dnp no)
 		(fields_autoplaced yes)
-		(property "Reference" "#PWR016"
+		(property "Reference" "#PWR023"
 			(at 83.82 71.12 0)
 			(hide yes)
@@
 			(project "autobot_mainboard"
 				(path "/f053f1d0-b1f5-4f80-9758-8ee1a2d3659d/33095814-6a92-4caa-8704-b20bd44a0045"
-					(reference "#PWR019")
-					(unit 1)
-				)
-				(path "/f053f1d0-b1f5-4f80-9758-8ee1a2d3659d/39e7d174-ffe7-4b4e-a983-e2abb212b9b6"
-					(reference "#PWR016")
+					(reference "#PWR028")
+					(unit 1)
+				)
+				(path "/f053f1d0-b1f5-4f80-9758-8ee1a2d3659d/39e7d174-ffe7-4b4e-a983-e2abb212b9b6"
+					(reference "#PWR023")
 					(unit 1)
 				)
@@
 		(in_pos_files yes)
 		(dnp no)
-		(property "Reference" "#PWR015"
+		(property "Reference" "#PWR022"
 			(at 80.01 64.77 0)
 			(hide yes)
@@
 			(project "autobot_mainboard"
 				(path "/f053f1d0-b1f5-4f80-9758-8ee1a2d3659d/33095814-6a92-4caa-8704-b20bd44a0045"
-					(reference "#PWR018")
-					(unit 1)
-				)
-				(path "/f053f1d0-b1f5-4f80-9758-8ee1a2d3659d/39e7d174-ffe7-4b4e-a983-e2abb212b9b6"
-					(reference "#PWR015")
+					(reference "#PWR027")
+					(unit 1)
+				)
+				(path "/f053f1d0-b1f5-4f80-9758-8ee1a2d3659d/39e7d174-ffe7-4b4e-a983-e2abb212b9b6"
+					(reference "#PWR022")
 					(unit 1)
 				)
@@
 		(in_pos_files yes)
 		(dnp no)
-		(property "Reference" "C16"
+		(property "Reference" "C12"
 			(at 146.05 67.056 0)
 			(show_name no)
@@
 			(project "autobot_mainboard"
 				(path "/f053f1d0-b1f5-4f80-9758-8ee1a2d3659d/33095814-6a92-4caa-8704-b20bd44a0045"
-					(reference "C17")
-					(unit 1)
-				)
-				(path "/f053f1d0-b1f5-4f80-9758-8ee1a2d3659d/39e7d174-ffe7-4b4e-a983-e2abb212b9b6"
-					(reference "C16")
+					(reference "C18")
+					(unit 1)
+				)
+				(path "/f053f1d0-b1f5-4f80-9758-8ee1a2d3659d/39e7d174-ffe7-4b4e-a983-e2abb212b9b6"
+					(reference "C12")
 					(unit 1)
 				)
@@
 		(in_pos_files yes)
 		(dnp no)
-		(property "Reference" "R13"
+		(property "Reference" "R9"
 			(at 175.006 50.546 0)
 			(show_name no)
@@
 			(project "autobot_mainboard"
 				(path "/f053f1d0-b1f5-4f80-9758-8ee1a2d3659d/33095814-6a92-4caa-8704-b20bd44a0045"
-					(reference "R14")
-					(unit 1)
-				)
-				(path "/f053f1d0-b1f5-4f80-9758-8ee1a2d3659d/39e7d174-ffe7-4b4e-a983-e2abb212b9b6"
 					(reference "R13")
+					(unit 1)
+				)
+				(path "/f053f1d0-b1f5-4f80-9758-8ee1a2d3659d/39e7d174-ffe7-4b4e-a983-e2abb212b9b6"
+					(reference "R9")
 					(unit 1)
 				)
@@
 			(project "autobot_mainboard"
 				(path "/f053f1d0-b1f5-4f80-9758-8ee1a2d3659d/33095814-6a92-4caa-8704-b20bd44a0045"
-					(reference "C9")
+					(reference "C14")
 					(unit 1)
 				)
@@
 		(dnp no)
 		(fields_autoplaced yes)
-		(property "Reference" "#PWR022"
+		(property "Reference" "#PWR024"
 			(at 110.49 102.87 0)
 			(hide yes)
@@
 			(project "autobot_mainboard"
 				(path "/f053f1d0-b1f5-4f80-9758-8ee1a2d3659d/33095814-6a92-4caa-8704-b20bd44a0045"
-					(reference "#PWR023")
-					(unit 1)
-				)
-				(path "/f053f1d0-b1f5-4f80-9758-8ee1a2d3659d/39e7d174-ffe7-4b4e-a983-e2abb212b9b6"
-					(reference "#PWR022")
+					(reference "#PWR029")
+					(unit 1)
+				)
+				(path "/f053f1d0-b1f5-4f80-9758-8ee1a2d3659d/39e7d174-ffe7-4b4e-a983-e2abb212b9b6"
+					(reference "#PWR024")
 					(unit 1)
 				)
@@
 		(in_pos_files yes)
 		(dnp no)
-		(property "Reference" "C6"
+		(property "Reference" "C7"
 			(at 59.69 66.548 0)
 			(show_name no)
@@
 			(project "autobot_mainboard"
 				(path "/f053f1d0-b1f5-4f80-9758-8ee1a2d3659d/33095814-6a92-4caa-8704-b20bd44a0045"
+					(reference "C13")
+					(unit 1)
+				)
+				(path "/f053f1d0-b1f5-4f80-9758-8ee1a2d3659d/39e7d174-ffe7-4b4e-a983-e2abb212b9b6"
 					(reference "C7")
-					(unit 1)
-				)
-				(path "/f053f1d0-b1f5-4f80-9758-8ee1a2d3659d/39e7d174-ffe7-4b4e-a983-e2abb212b9b6"
-					(reference "C6")
 					(unit 1)
 				)
@@
 		(in_pos_files yes)
 		(dnp no)
-		(property "Reference" "C12"
+		(property "Reference" "C11"
 			(at 87.122 73.152 0)
 			(show_name no)
@@
 			(project "autobot_mainboard"
 				(path "/f053f1d0-b1f5-4f80-9758-8ee1a2d3659d/33095814-6a92-4caa-8704-b20bd44a0045"
-					(reference "C14")
-					(unit 1)
-				)
-				(path "/f053f1d0-b1f5-4f80-9758-8ee1a2d3659d/39e7d174-ffe7-4b4e-a983-e2abb212b9b6"
-					(reference "C12")
+					(reference "C17")
+					(unit 1)
+				)
+				(path "/f053f1d0-b1f5-4f80-9758-8ee1a2d3659d/39e7d174-ffe7-4b4e-a983-e2abb212b9b6"
+					(reference "C11")
 					(unit 1)
 				)
@@
 		(in_pos_files yes)
 		(dnp no)
-		(property "Reference" "R11"
+		(property "Reference" "R10"
 			(at 175.26 60.96 90)
 			(show_name no)
@@
 			(project "autobot_mainboard"
 				(path "/f053f1d0-b1f5-4f80-9758-8ee1a2d3659d/33095814-6a92-4caa-8704-b20bd44a0045"
-					(reference "R12")
-					(unit 1)
-				)
-				(path "/f053f1d0-b1f5-4f80-9758-8ee1a2d3659d/39e7d174-ffe7-4b4e-a983-e2abb212b9b6"
-					(reference "R11")
+					(reference "R14")
+					(unit 1)
+				)
+				(path "/f053f1d0-b1f5-4f80-9758-8ee1a2d3659d/39e7d174-ffe7-4b4e-a983-e2abb212b9b6"
+					(reference "R10")
 					(unit 1)
 				)
@@
 		(in_pos_files yes)
 		(dnp no)
-		(property "Reference" "C42"
+		(property "Reference" "C9"
 			(at 76.454 67.056 0)
 			(show_name no)
@@
 			(project "autobot_mainboard"
 				(path "/f053f1d0-b1f5-4f80-9758-8ee1a2d3659d/33095814-6a92-4caa-8704-b20bd44a0045"
-					(reference "C43")
-					(unit 1)
-				)
-				(path "/f053f1d0-b1f5-4f80-9758-8ee1a2d3659d/39e7d174-ffe7-4b4e-a983-e2abb212b9b6"
-					(reference "C42")
-					(unit 1)
-				)
+					(reference "C15")
+					(unit 1)
+				)
+				(path "/f053f1d0-b1f5-4f80-9758-8ee1a2d3659d/39e7d174-ffe7-4b4e-a983-e2abb212b9b6"
+					(reference "C9")
+					(unit 1)
+				)
