File: ELECTRONICS/MAINBOARD/autobot_mainboard.kicad_sch (KiCad schematic)
At the start: 173 parts, among them IC2 DW3210, IC3 DW3210, J10 MA, J11 MB, J9 USB_C_Receptacle_USB2.0_16P, Q10 TBD_N, Q4 TBD_N, Q5 TBD_N, Q6 TBD_P, Q7 TBD_N, Q8 TBD_N, Q9 TBD_N, SW6 BOOT, SW7 RESET, U10 LP5907MFX-3.3, U11 LP5907MFX-3.3, U12 LP5907MFX-3.3, U13 INA226, U14 BMI270, U17 TVS1400DRV, U4 BMI270, U5 HUSB238_xxxDD, U6 BQ24170RGYR, U7 LM5175RHF, U8 LM2596S-5, U9 STM32H743ZITx

Commit message: Add files via upload
Parts:
- removed BT2: 3C, symbol Device:Battery_Cell
- removed C63, C64, C67, C70, C71, C80, C81: 100n, symbol Device:C
- removed C65, C66, C68, C74: 1u, symbol Device:C
- removed C69: 4.7n, symbol Device:C
- removed C72, C73, C84, C85, C86: 10u, symbol Device:C
- removed C75: 68n, symbol Device:C
- removed C76: 120p, symbol Device:C
- removed C77: 10n, symbol Device:C
- removed C78, C83: 47p, symbol Device:C
- removed C79: 68u, symbol Device:C_Polarized
- removed C82: 22u, symbol Device:C
- removed C87: 220n, symbol Device:C
- removed D10, D7, D9: good diode fr, Diode_SMD:D_SOD-123, symbol Diode:1N4148W
- removed D11: D, symbol Device:D
- removed D6: LED, symbol Device:LED
- removed D8: CDBK0520L-HF/EQ, Diode_SMD:D_SOD-123, symbol Diode:1N4148W
- removed L5: 3.3m, symbol Device:L
- removed L6: 2.6u, symbol Device:L
- removed Q10, Q4, Q5, Q7, Q8, Q9: TBD_N, Package_TO_SOT_SMD:SOT-23, symbol Transistor_FET:DMG2302U
- removed Q6: TBD_P, Package_TO_SOT_SMD:SOT-23, symbol Transistor_FET:DMP3099L
- removed R23: 10k, symbol Device:R
- removed R24, R26, R27, R28, R29, R32: TBD, symbol Device:R
- removed R25, R48: 10, symbol Device:R
- removed R30: 1M, symbol Device:R
- removed R31: 100K, symbol Device:R
- removed R33: 5.23K, symbol Device:R
- removed R34: 30.1K, symbol Device:R
- removed R35, R36: 4k, symbol Device:R
- removed R37: 1k, symbol Device:R
- removed R38, R39: 10m, symbol Device:R
- removed R40: 86.6k, symbol Device:R
- removed R41: 23.7k, symbol Device:R
- removed R42: 93.1k, symbol Device:R
- removed R43: 249k, symbol Device:R
- removed R44, R49: 5m, symbol Device:R
- removed R45: 576k, symbol Device:R
- removed R46: 20k, symbol Device:R
- removed R47: 68.1k, symbol Device:R
- removed TH1: 103AT, symbol Device:Thermistor
- removed U5: HUSB238_xxxDD, Package_DFN_QFN:WDFN-10-1EP_3x3mm_P0.5mm_EP1.8x2.5mm, symbol Interface_USB:HUSB238_xxxDD
- removed U6: BQ24170RGYR, AutoBotfootprintlibrary:RGY24_2P05X3P1, symbol AutoBotLibrary:BQ24170RGYR
- removed U7: LM5175RHF, Package_DFN_QFN:VQFN-28-1EP_4x5mm_P0.5mm_EP2.55x3.55mm, symbol AutoBotLibrary:LM5175RHF
- added R10, R9: 5.1k, symbol Device:R
- added U22: TVS1400DRV, Package_SON:WSON-6-1EP_2x2mm_P0.65mm_EP1x1.6mm, symbol Power_Protection:TVS1400DRV
- U18, U19, U20, U21: value (none) -> VL53L1X; footprint (none) -> Connector_JST:JST_PH_S6B-PH-K_1x06_P2.00mm_Horizontal
Connections:
- net DW_GPIO5_1 is gone; now on net GNDREF: IC2.5 (GPIO5_/_EXTTXE_/_SPIPOL)
- net DW_GPIO5_2 is gone; now on net GNDREF: IC3.5 (GPIO5_/_EXTTXE_/_SPIPOL)
- net DW_GPIO6_1 is gone; now on net GNDREF: IC2.2 (GPIO6_/_EXTRXE_/_SPIPHA)
- net DW_GPIO6_2 is gone; now on net GNDREF: IC3.2 (GPIO6_/_EXTRXE_/_SPIPHA)
- net +12V: now also C89.1, U8.1 (VIN), U22.4 (IN), U22.5 (IN), U22.6 (IN)
- net +3V3: no longer U16.10 (MS2_AD1)
- net GNDREF: now also U16.10 (MS2_AD1), U9.107 (VSS), U9.120 (VSS), U9.130 (VSS), U9.16 (VSS), U9.31 (VSSA), U9.38 (VSS), U9.51 (VSS), U9.61 (VSS), U9.83 (VSS), U9.94 (VSS), R10.1, R9.1, U22.1 (GND), U22.2 (GND), U22.3 (GND), U22.7 (GND)
- net INA_VIN-: no longer U13.8 (Vbus)
- net CC1: no longer names the net of J9.A5 (CC1)
- net CC1: now also R10.2
- net CC2: no longer names the net of J9.B5 (CC2)
- net CC2: now also R9.2
- new net VBAT: U13.8 (Vbus)
- no-connect marks 22 -> 20
Other:
- note added: "IMU"
- note added: "TMC2209"
- note added: "USB"
- note added: "VL53L1X"
- note added: "just do the rest of the decoup later, prolly add more bulk capacitors add ferrite bead"
- note removed: "CELL 1 CELL LOW 2 CELL FLOAT 3 CELL HIGH LOWK JS ADD A DIPSWITCH OR SMTH"
- note removed: "DO MATH LATER YOURSELF, THIS IS REFERENCE CIRCUIT"
- note removed: "EPAD IS AGND, DEAL WITH THIS LATER"
- note removed: "OMIT FOR V1 USE BMS INSTEAD"
- note removed: "PROLLY OMIT THIS TOO FOR V1"
- note removed: "SET R VALUE TO LIMIT CURRENT, LEAVE FLOATING FOR 3.25A"
- note removed: "avg current monitoring disabled"
- note removed: "maybe something smaller"
- note removed: "prolly not gon use dith so maybe tie to gnd"
- moved on the sheet: C118, C119, C120, C121, C122, C123, C124, C125, C126, C127, C128, C129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

Commit message: Add files via upload
Parts:
- removed C88: 220u, symbol Device:C
- removed C89: 680u, symbol Device:C
- removed D12: D, symbol Device:D
- removed L7: 33u, symbol Device:L
- removed U22: TVS1400DRV, Package_SON:WSON-6-1EP_2x2mm_P0.65mm_EP1x1.6mm, symbol Power_Protection:TVS1400DRV
- removed U8: LM2596S-5, Package_TO_SOT_SMD:TO-263-5_TabPin3, symbol Regulator_Switching:LM2596S-5
- added C61: 1u, Capacitor_SMD:C_0603_1608Metric, symbol Device:C
- added C62, C63: 100n, Capacitor_SMD:C_0603_1608Metric, symbol Device:C
- added C64: 47u, Capacitor_SMD:C_0603_1608Metric, symbol Device:C
- added L2: 5.6u, Inductor_SMD:L_APV_APH0840, symbol Device:L
- added R18: 162k, Resistor_SMD:R_0603_1608Metric, symbol Device:R
- added R19: 22.1k, Resistor_SMD:R_0603_1608Metric, symbol Device:R
- added U17: LMR51430XDDCR, MyFootprintLibrary:SOT-23-THIN-6_DDC_TEX, symbol AutoBotLibrary:LMR51430XDDCR
- added U6: TVS1400DRV, Package_SON:WSON-6-1EP_2x2mm_P0.65mm_EP1x1.6mm, symbol Power_Protection:TVS1400DRV
- C1: renamed from C122; footprint Capacitor_Tantalum_SMD:CP_EIA-6032-28_Kemet-C -> MyFootprintLibrary:PCAP_SVP_F12_PAN-M
- C10: renamed from C118; footprint (none) -> Capacitor_SMD:C_0402_1005Metric
- C14: renamed from C90; footprint (none) -> Capacitor_SMD:C_0402_1005Metric
- C16: renamed from C91; footprint (none) -> Capacitor_SMD:C_0402_1005Metric
- C17: renamed from C120; footprint (none) -> Capacitor_SMD:C_0402_1005Metric
- C18: renamed from C96; footprint (none) -> Capacitor_SMD:C_0402_1005Metric
- C19: renamed from C121; footprint (none) -> Capacitor_SMD:C_0402_1005Metric
- C22: renamed from C92; footprint (none) -> Capacitor_SMD:C_0402_1005Metric
- C23: renamed from C93; footprint (none) -> Capacitor_SMD:C_0402_1005Metric
- C35: renamed from C107; footprint (none) -> Capacitor_SMD:C_0402_1005Metric
- C36: renamed from C108; footprint (none) -> Capacitor_SMD:C_0402_1005Metric
- C39: renamed from C109; footprint (none) -> Capacitor_SMD:C_0402_1005Metric
- C40: renamed from C110; footprint (none) -> Capacitor_SMD:C_0402_1005Metric
- C41: renamed from C94; footprint (none) -> Capacitor_SMD:C_0402_1005Metric
- C42: renamed from C111; footprint (none) -> Capacitor_SMD:C_0402_1005Metric
- C43: renamed from C112; footprint (none) -> Capacitor_SMD:C_0402_1005Metric
- C44: renamed from C113; footprint (none) -> Capacitor_SMD:C_0402_1005Metric
- C45: renamed from C114; footprint (none) -> Capacitor_SMD:C_0402_1005Metric
- C46: renamed from C95; footprint (none) -> Capacitor_SMD:C_0402_1005Metric
- C47: renamed from C115; footprint (none) -> Capacitor_SMD:C_0402_1005Metric
- C48: renamed from C116; footprint (none) -> Capacitor_SMD:C_0402_1005Metric
- C49: renamed from C117; footprint (none) -> Capacitor_SMD:C_0402_1005Metric
- C7: renamed from C127; footprint Capacitor_Tantalum_SMD:CP_EIA-6032-28_Kemet-C -> MyFootprintLibrary:PCAP_SVP_F12_PAN-M
- C9: renamed from C119; footprint (none) -> Capacitor_SMD:C_0402_1005Metric
- IC1: renamed from IC2; footprint AutoBotfootprintlibrary:QFN40P500X500X80-40N-D -> MyFootprintLibrary:qfn_DW3220_QOR-M
- IC2: renamed from IC3; footprint AutoBotfootprintlibrary:QFN40P500X500X80-40N-D -> MyFootprintLibrary:qfn_DW3220_QOR-M
- J1: renamed from J9; footprint (none) -> Connector_USB:USB_C_Receptacle_GCT_USB4105-xx-A_16P_TopMnt_Horizontal
- R1: renamed from R8; footprint (none) -> Capacitor_SMD:C_0402_1005Metric
- R14: renamed from R58; footprint (none) -> Resistor_SMD:R_0402_1005Metric
- R15: renamed from R53; footprint (none) -> Resistor_SMD:R_0402_1005Metric
- R2: renamed from R22; footprint (none) -> Capacitor_SMD:C_0402_1005Metric
- R3: renamed from R9; footprint (none) -> Capacitor_SMD:C_0402_1005Metric
- R4: renamed from R10; footprint (none) -> Capacitor_SMD:C_0402_1005Metric
- R5: renamed from R59; footprint Resistor_SMD:R_1206_3216Metric -> Resistor_SMD:R_0402_1005Metric
- R6: renamed from R60; footprint Resistor_SMD:R_1206_3216Metric -> Resistor_SMD:R_0402_1005Metric
- R7: renamed from R65; footprint Resistor_SMD:R_1206_3216Metric -> Resistor_SMD:R_0402_1005Metric
- R8: renamed from R66; footprint Resistor_SMD:R_1206_3216Metric -> Resistor_SMD:R_0402_1005Metric
- R9: renamed from R51; footprint (none) -> Resistor_SMD:R_0402_1005Metric
- SW1: renamed from SW7; footprint (none) -> Button_Switch_THT:SW_PUSH_6mm
- SW2: renamed from SW6; footprint (none) -> Button_Switch_THT:SW_PUSH_6mm
- U10: renamed from U4; footprint BMI270_BOS -> (none)
- U13: renamed from U14; footprint BMI270_BOS -> (none)
- renumbered C129 to C11, C130 to C12, C131 to C15, C123 to C2, C37 to C20, C38 to C21, C39 to C24, C40 to C25, C41 to C26, C42 to C27, C43 to C28, C44 to C29, C124 to C3, C45 to C30, C46 to C31, C47 to C32, C48 to C33, C49 to C34, C50 to C37, C51 to C38, C125 to C4, C126 to C5, C52 to C50, C53 to C51, C54 to C52, C55 to C53, C56 to C54, C57 to C55, C58 to C56, C59 to C57, C60 to C58, C61 to C59, C62 to C60, C128 to C8, FB2 to FB1, FB3 to FB2, J10 to J2, J11 to J3, R61 to R10, R62 to R11, R63 to R12, R64 to R13, R20 to R16, R21 to R17, U18 to U1, U16 to U11, U10 to U12, U9 to U14, U11 to U15, U12 to U16, U13 to U2, U19 to U3, U15 to U4, U20 to U5, U17 to U7, U21 to U8
Connections:
- net +12V: now also C61.1, C62.1, U17.3 (VIN), U17.5 (EN), U6.4 (IN), U6.5 (IN), U6.6 (IN)
- net +5V: now also C64.1, L2.2, R18.1
- net GNDREF: now also C61.2, C62.2, C64.2, R19.2, U17.1 (GND), U6.1 (GND), U6.2 (GND), U6.3 (GND), U6.7 (GND)
- net VL_XSHUT1: now also U1.6 (XSHUT); no longer U1. (XSHUT)
- net VL_XSHUT2: now also U3.6 (XSHUT); no longer U3. (XSHUT)
- net VL_XSHUT3: now also U5.6 (XSHUT); no longer U5. (XSHUT)
- net VL_XSHUT4: now also U8.6 (XSHUT); no longer U8. (XSHUT)
- new net: C63.2, L2.1, U17.2 (SW)
- new net: R18.2, R19.1, U17.4 (FB)
- new net: C63.1, U17.6 (CB)
Other:
- moved on the sheet: C10, C14, C16, C17, C19, C9, J1, R1, R14, R2, R3, R4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

Commit message: Add files via upload
Parts:
- removed C18: 100n, Capacitor_SMD:C_0402_1005Metric, symbol Device:C
- removed C61: 1u, Capacitor_SMD:C_0603_1608Metric, symbol Device:C
- removed C63: 100n, Capacitor_SMD:C_0603_1608Metric, symbol Device:C
- removed C64: 47u, Capacitor_SMD:C_0603_1608Metric, symbol Device:C
- removed R1, R2: 22, Capacitor_SMD:C_0402_1005Metric, symbol Device:R
- removed U14: STM32H743ZITx, Package_QFP:LQFP-144_20x20mm_P0.5mm, symbol MCU_ST_STM32H7:STM32H743ZITx
- removed U17: LMR51430XDDCR, MyFootprintLibrary:SOT-23-THIN-6_DDC_TEX, symbol AutoBotLibrary:LMR51430XDDCR
- removed U6, U7: TVS1400DRV, Package_SON:WSON-6-1EP_2x2mm_P0.65mm_EP1x1.6mm, symbol Power_Protection:TVS1400DRV
- added C1, C26, C3, C5, C81, C83, C9: 100n, Capacitor_SMD:C_0402_1005Metric, symbol Device:C
- added C10, C2, C4, C7: 10u, Capacitor_SMD:C_0402_1005Metric, symbol Device:C
- added C13, C17: 2.2u, symbol Device:C
- added C44, C49, C59: C, Capacitor_SMD:C_0402_1005Metric, symbol Device:C
- added C53, C68: AMT-102-V, Connector_JST:JST_PH_S6B-PH-K_1x06_P2.00mm_Horizontal, symbol AutoBotLibrary:AMT102-V
- added C75: 1u, Capacitor_SMD:C_0603_1608Metric, symbol Device:C
- added C76, C77: 100n, Capacitor_SMD:C_0603_1608Metric, symbol Device:C
- added C78: 47u, Capacitor_SMD:C_0603_1608Metric, symbol Device:C
- added C79, C80: 12p, symbol Device:C
- added C82: 1u, Capacitor_SMD:C_0402_1005Metric, symbol Device:C
- added D1: SS24, Diode_SMD:D_SMA, symbol Diode:SS24
- added FB2, FB3, FB5: FerriteBead_Small, symbol Device:FerriteBead_Small
- added J4: Conn_01x03_Pin, symbol Connector:Conn_01x03_Pin
- added J6, J7: Conn_01x05_Socket, symbol Connector:Conn_01x05_Socket
- added R20: 10k, Resistor_SMD:R_0402_1005Metric, symbol Device:R
- added R3, R4: 22, Resistor_SMD:R_0402_1005Metric, symbol Device:R
- added U12, U21, U3: TVS1400DRV, Package_SON:WSON-6-1EP_2x2mm_P0.65mm_EP1x1.6mm, symbol Power_Protection:TVS1400DRV
- added U16: STM32H743ZITx, Package_QFP:LQFP-144_20x20mm_P0.5mm, symbol MCU_ST_STM32H7:STM32H743ZITx
- added U18, U20: TPD4E05U06DQA, Package_SON:USON-10_2.5x1.0mm_P0.5mm, symbol Power_Protection:TPD4E05U06DQA
- added U22: LMR51430XDDCR, MyFootprintLibrary:SOT-23-THIN-6_DDC_TEX, symbol AutoBotLibrary:LMR51430XDDCR
- added U5: TPD2EUSB30A, Package_TO_SOT_SMD:Texas_DRT-3, symbol Power_Protection:TPD2EUSB30A
- added Y1: 25mhz placeholder, Crystal:Crystal_SMD_2016-4Pin_2.0x1.6mm, symbol Device:Crystal_GND24
- C62: value 100n -> C; footprint Capacitor_SMD:C_0603_1608Metric -> Capacitor_SMD:C_0402_1005Metric
- R1: renamed from R3; footprint Capacitor_SMD:C_0402_1005Metric -> Resistor_SMD:R_0402_1005Metric
- R15: value 10k -> 47; footprint Resistor_SMD:R_0402_1005Metric -> (none)
- R2: renamed from R4; footprint Capacitor_SMD:C_0402_1005Metric -> Resistor_SMD:R_0402_1005Metric
- R5, R6: footprint Resistor_SMD:R_0402_1005Metric -> Resistor_SMD:R_1206_3216Metric
- R8: renamed from R7; footprint Resistor_SMD:R_0402_1005Metric -> Resistor_SMD:R_1206_3216Metric
- R9: renamed from R8; footprint Resistor_SMD:R_0402_1005Metric -> Resistor_SMD:R_1206_3216Metric
- U11: renamed from U10; footprint (none) -> MyFootprintLibrary:BMI270_BOS-M
- U14: renamed from U13; footprint (none) -> MyFootprintLibrary:BMI270_BOS-M
- renumbered C3 to C11, C4 to C12, C9 to C14, C10 to C15, C5 to C16, C7 to C18, C8 to C19, C11 to C20, C12 to C21, C14 to C22, C16 to C23, C15 to C24, C17 to C25, C19 to C27, C20 to C28, C21 to C29, C22 to C30, C23 to C31, C24 to C32, C25 to C33, C26 to C34, C27 to C35, C28 to C36, C29 to C37, C30 to C38, C31 to C39, C32 to C40, C33 to C41, C34 to C42, C35 to C43, C36 to C45, C37 to C46, C38 to C47, C39 to C48, C40 to C50, C41 to C51, C42 to C52, C43 to C54, C44 to C55, C45 to C56, C46 to C57, C47 to C58, C1 to C6, C48 to C60, C49 to C61, C50 to C63, C51 to C64, C52 to C65, C53 to C66, C54 to C67, C55 to C69, C56 to C70, C57 to C71, C58 to C72, C59 to C73, C60 to C74, C2 to C8, FB2 to FB4, J2 to J1, J1 to J2, R14 to R12, R12 to R13, R13 to R14, R9 to R7, U11 to U13, U12 to U15, U15 to U17, U16 to U19, U3 to U4, U5 to U6, U4 to U8, U8 to U9
Connections:
- net +12V: now also C75.1, C76.1, J4.1 (Pin_1), U21.4 (IN), U21.5 (IN), U21.6 (IN), U22.3 (VIN), U22.5 (EN); no longer C62.1
- net +24V: now also J4.2 (Pin_2), U12.4 (IN), U12.5 (IN), U12.6 (IN), U3.4 (IN), U3.5 (IN), U3.6 (IN)
- net +3V3: now also SW2.2, C1.1, C10.1, C2.1, C3.1, C4.1, C5.1, C7.1, C81.1, C9.1, FB5.1, J6.2 (Pin_2), J7.2 (Pin_2), U16.108 (VDD), U16.121 (VDD), U16.131 (VDD), U16.143 (PDR_ON), U16.144 (VDD), U16.17 (VDD), U16.30 (VDD), U16.39 (VDD), U16.52 (VDD), U16.6 (VBAT), U16.62 (VDD), U16.72 (VDD), U16.84 (VDD), U16.95 (VDD33_USB); no longer R15.1
- net +5V: now also C44.1, C59.1, C78.1, FB2.1, FB3.1, U18.4 (D2+), U20.4 (D2+)
- net ALERT: now also U16.124 (PG9)
- net BMI_CS_1: now also U16.92 (PG7)
- net BMI_CS_2: now also U16.93 (PG8)
- net BMI_INT_1: now also U16.125 (PG10)
- net BMI_INT_2: now also U16.126 (PG11)
- net BMI_MISO: now also U16.42 (PA6)
- net BMI_MOSI: now also U16.43 (PA7)
- net BMI_SCK: now also U16.41 (PA5)
- net D+: now also R4.2, U16.104 (PA12)
- net D-: now also R3.2, U16.103 (PA11)
- net DIAG_1: now also U16.88 (PG3)
- net DIAG_2: now also U16.90 (PG5)
- net DIR_1: now also U16.57 (PG1)
- net DIR_2: now also U16.91 (PG6)
- net DW_CLK_1: now also U16.74 (PB13)
- net DW_CLK_2: now also U16.111 (PC10)
- net DW_CSN_1: now also U16.114 (PD0), U16.73 (PB12)
- net DW_MISO_1: now also U16.75 (PB14)
- net DW_MISO_2: now also U16.112 (PC11)
- net DW_MOSI_1: now also U16.76 (PB15)
- net DW_MOSI_2: now also U16.113 (PC12)
- net DW_RST_1: now also U16.69 (PB10)
- net DW_RST_2: now also U16.115 (PD1)
- net GNDREF: now also C1.2, C10.2, C13.2, C17.2, C2.2, C26.2, C3.2, C4.2, C44.2, C49.2, C5.2, C53.1 (GND), C59.2, C68.1 (GND), C7.2, C75.2, C76.2, C78.2, C79.2, C80.2, C81.2, C82.2, C83.2, C9.2, J4.3 (Pin_3), J6.3 (Pin_3), J7.3 (Pin_3), R20.2, U12.1 (GND), U12.2 (GND), U12.3 (GND), U12.7 (GND), U16.107 (VSS), U16.120 (VSS), U16.130 (VSS), U16.16 (VSS), U16.31 (VSSA), U16.38 (VSS), U16.51 (VSS), U16.61 (VSS), U16.83 (VSS), U16.94 (VSS), U18.3 (GND), U18.8 (GND), U20.3 (GND), U20.8 (GND), U21.1 (GND), U21.2 (GND), U21.3 (GND), U21.7 (GND), U22.1 (GND), U3.1 (GND), U3.2 (GND), U3.3 (GND), U3.7 (GND), U5.3 (GND), Y1.2 (G), Y1.4 (G); no longer SW2.1
- net INDEX_1: now also U16.87 (PG2)
- net INDEX_2: now also U16.89 (PG4)
- net IRQ_1: now also U16.128 (PG13)
- net IRQ_2: now also U16.129 (PG14)
- net NRST: now also C26.1, U16.25 (NRST)
- net RXD0: now also U16.18 (PF6)
- net RXD1: now also U16.141 (PE0)
- net STEP_1: now also U16.60 (PE9)
- net STEP_2: now also U16.64 (PE11)
- net TMC_EN: now also U16.56 (PG0)
- net TXD0: now also U16.19 (PF7)
- net TXD1: now also U16.142 (PE1)
- net VBUS: now also D1.1 (K); no longer J2.A4 (VBUS), J2.A9 (VBUS), J2.B4 (VBUS), J2.B9 (VBUS)
- net WAKEUP_1: now also U16.70 (PB11)
- net WAKEUP_2: now also U16.116 (PD2)
- net at R15.2: now also C82.1, C83.1, FB5.2, U16.33 (VDDA); no longer SW2.2
- net DATA +: now reaches J2.A6 (D+), J2.B6 (D+)
- net DATA +: now also R4.1, U5.1 (D+)
- net DATA -: now reaches J2.A7 (D-), J2.B7 (D-)
- net DATA -: now also R3.1, U5.2 (D-)
- net at L2.1: now also C77.2, U22.2 (SW)
- net at R18.2, R19.1: now also U22.4 (FB)
- new net: D1.2 (A), J2.A4 (VBUS), J2.A9 (VBUS), J2.B4 (VBUS), J2.B9 (VBUS)
- new net: C17.1, U16.106 (VCAP)
- new net: C13.1, U16.71 (VCAP)
- new net: C77.1, U22.6 (CB)
- new net: C62.1, C68.2 (VIN), FB3.2
- new net: C49.1, C53.2 (VIN), FB2.2
- new net AMT_A_L: C53.3 (A), U18.1 (D1+)
- new net AMT_A_R: C68.3 (A), U20.1 (D1+)
- new net AMT_B_L: C53.4 (B), U18.2 (D1-)
- new net AMT_B_R: C68.4 (B), U20.2 (D1-)
- new net AMT_X_L: C53.5 (X), U18.5 (D2-)
- new net AMT_X_R: C68.5 (X), U20.5 (D2-)
- new net BOOT0: R20.1, SW2.1, U16.138 (BOOT0)
- new net NRESET: J6.5 (Pin_5)
- new net PH0: C79.1, U16.23 (PH0), Y1.1
- new net PH1: C80.1, U16.24 (PH1), Y1.3
- new net SWCLK: J7.5 (Pin_5), U16.109 (PA14)
- new net SWDIO: J7.4 (Pin_4), U16.105 (PA13)
- new net VREF: R15.1, U16.32 (VREF+)
- no-connect marks 20 -> 31
Other:
- note added: "D+ and D- is just I/O, so just cosmetic ig"
- note added: "LEFT"
- note added: "RIGHT"
- note added: "ROTARY ENCODER"
- note added: "SWIM NC"
- note added: "VL53L1X DECOUP"
- note added: "prolly get a coin battery? not required. (for vbat)"
- moved on the sheet: C11, C12, C14, C15, C16, C18, C19, C20, C21, C22, C23, C24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

Commit message: Add files via upload
Parts:
- removed C1, C14, C15, C25, C26, C27, C3, C32, C37, C38, C39, C43, C45, C48, C5, C50, C52, C54, C55, C56, C58, C60, C63, C69, C70, C71, C81, C83, C9: 100n, Capacitor_SMD:C_0402_1005Metric, symbol Device:C
- removed C10, C2, C4, C41, C42, C7, C73, C74: 10u, Capacitor_SMD:C_0402_1005Metric, symbol Device:C
- removed C11, C20: 22nF, Capacitor_SMD:C_0402_1005Metric, symbol Device:C_Small
- removed C12, C16, C19, C21, C24, C8: 100nF, Capacitor_SMD:C_0402_1005Metric, symbol Device:C_Small
- removed C13, C17: 2.2u, symbol Device:C
- removed C18, C6: 100uF, MyFootprintLibrary:PCAP_SVP_F12_PAN-M, symbol Device:C_Polarized
- removed C22, C23, C30, C31, C51, C57, C82: 1u, Capacitor_SMD:C_0402_1005Metric, symbol Device:C
- removed C28, C29, C46, C47: 2p, Capacitor_SMD:C_0402_1005Metric, symbol Device:C
- removed C33, C34, C35, C64, C65, C66: 4.7n, Capacitor_SMD:C_0402_1005Metric, symbol Device:C
- removed C36, C67: 220n, Capacitor_SMD:C_0402_1005Metric, symbol Device:C
- removed C40, C72: 4.7u, Capacitor_SMD:C_0402_1005Metric, symbol Device:C
- removed C44, C49, C59, C62: C, Capacitor_SMD:C_0402_1005Metric, symbol Device:C
- removed C53, C68: AMT-102-V, Connector_JST:JST_PH_S6B-PH-K_1x06_P2.00mm_Horizontal, symbol AutoBotLibrary:AMT102-V
- removed C61: 4u7, Capacitor_SMD:C_0402_1005Metric, symbol Device:C
- removed C75: 1u, Capacitor_SMD:C_0603_1608Metric, symbol Device:C
- removed C76, C77: 100n, Capacitor_SMD:C_0603_1608Metric, symbol Device:C
- removed C78: 47u, Capacitor_SMD:C_0603_1608Metric, symbol Device:C
- removed C79, C80: 12p, symbol Device:C
- removed D1: SS24, Diode_SMD:D_SMA, symbol Diode:SS24
- removed FB1, FB4: fb, Resistor_SMD:R_0603_1608Metric, symbol Device:FerriteBead_Small
- removed FB2, FB3, FB5: FerriteBead_Small, symbol Device:FerriteBead_Small
- removed IC1, IC2: DW3210, MyFootprintLibrary:qfn_DW3220_QOR-M, symbol AutoBotLibrary:DW3210
- removed J1: MA, TerminalBlock_Phoenix:TerminalBlock_Phoenix_PT-1,5-4-3.5-H_1x04_P3.50mm_Horizontal, symbol Connector:Screw_Terminal_01x04
- removed J2: USB_C_Receptacle_USB2.0_16P, Connector_USB:USB_C_Receptacle_GCT_USB4105-xx-A_16P_TopMnt_Horizontal, symbol Connector:USB_C_Receptacle_USB2.0_16P
- removed J3: MB, TerminalBlock_Phoenix:TerminalBlock_Phoenix_PT-1,5-4-3.5-H_1x04_P3.50mm_Horizontal, symbol Connector:Screw_Terminal_01x04
- removed J4: Conn_01x03_Pin, symbol Connector:Conn_01x03_Pin
- removed J6, J7: Conn_01x05_Socket, symbol Connector:Conn_01x05_Socket
- removed L2: 5.6u, Inductor_SMD:L_APV_APH0840, symbol Device:L
- removed R1, R2: 5.1k, Resistor_SMD:R_0402_1005Metric, symbol Device:R
- removed R10, R11: 1K, Resistor_SMD:R_0402_1005Metric, symbol Device:R
- removed R12, R13, R14, R20, R7: 10k, Resistor_SMD:R_0402_1005Metric, symbol Device:R
- removed R15: 47, symbol Device:R
- removed R16, R17: 100K, Resistor_SMD:R_0402_1005Metric, symbol Device:R
- removed R18: 162k, Resistor_SMD:R_0603_1608Metric, symbol Device:R
- removed R19: 22.1k, Resistor_SMD:R_0603_1608Metric, symbol Device:R
- removed R3, R4: 22, Resistor_SMD:R_0402_1005Metric, symbol Device:R
- removed R5, R6, R8, R9: 0.1, Resistor_SMD:R_1206_3216Metric, symbol Device:R
- removed SW1: RESET, Button_Switch_THT:SW_PUSH_6mm, symbol Switch:SW_Push
- removed SW2: BOOT, Button_Switch_THT:SW_PUSH_6mm, symbol Switch:SW_Push
- removed U1, U4, U6, U9: VL53L1X, Connector_JST:JST_PH_S6B-PH-K_1x06_P2.00mm_Horizontal, symbol AutoBotLibrary:ADAFRUIT_VL53L1X_MODULE
- removed U11, U14: BMI270, MyFootprintLibrary:BMI270_BOS-M, symbol AutoBotLibrary:BMI270
- removed U12, U21, U3: TVS1400DRV, Package_SON:WSON-6-1EP_2x2mm_P0.65mm_EP1x1.6mm, symbol Power_Protection:TVS1400DRV
- removed U13, U8: (no value), MyFootprintLibrary:tmc2209, symbol My-Kicad-Library:TMC2209
- removed U15, U17, U19: LP5907MFX-3.3, Package_TO_SOT_SMD:SOT-23-5, symbol Regulator_Linear:LP5907MFX-3.3
- removed U16: STM32H743ZITx, Package_QFP:LQFP-144_20x20mm_P0.5mm, symbol MCU_ST_STM32H7:STM32H743ZITx
- removed U18, U20: TPD4E05U06DQA, Package_SON:USON-10_2.5x1.0mm_P0.5mm, symbol Power_Protection:TPD4E05U06DQA
- removed U2: INA226, Package_SO:TSSOP-10_3x3mm_P0.5mm, symbol Sensor_Energy:INA226
- removed U22: LMR51430XDDCR, MyFootprintLibrary:SOT-23-THIN-6_DDC_TEX, symbol AutoBotLibrary:LMR51430XDDCR
- removed U5: TPD2EUSB30A, Package_TO_SOT_SMD:Texas_DRT-3, symbol Power_Protection:TPD2EUSB30A
- removed Y1: 25mhz placeholder, Crystal:Crystal_SMD_2016-4Pin_2.0x1.6mm, symbol Device:Crystal_GND24
Connections:
- no-connect marks 31 -> 1
Other:
- added sheet AMT102_L (AMT102.kicad_sch)
- added sheet AMT102_R (AMT102.kicad_sch)
- added sheet BMI270_L (BMI270.kicad_sch)
- added sheet BMI270_R (BMI270.kicad_sch)
- added sheet DW3220_B (DW3220.kicad_sch)
- added sheet DW3220_T (DW3220.kicad_sch)
- added sheet LDO (LDO.kicad_sch)
- added sheet LDO1 (LDO.kicad_sch)
- added sheet LDO2 (LDO.kicad_sch)
- added sheet LDO3 (LDO.kicad_sch)
- added sheet LMR51430XDDCR (Power.sch.kicad_sch)
- added sheet MOTOR_CONNECTOR_L (MOTOR_CONNECTOR.kicad_sch)
- added sheet MOTOR_CONNECTOR_R (MOTOR_CONNECTOR.kicad_sch)
- added sheet POWER_CONNECTOR (POWER_CONNECTOR.kicad_sch)
- added sheet STM32H743 (STM32H743.kicad_sch)
- added sheet TMC2209_L (TMC2209.kicad_sch)
- added sheet TMC2209_R (TMC2209.kicad_sch)
- added sheet USB (USB.kicad_sch)
- added sheet VL53L1X0 (VL53L1X.kicad_sch)
- added sheet VL53L1X1 (VL53L1X.kicad_sch)
- added sheet VL53L1X2 (VL53L1X.kicad_sch)
- added sheet VL53L1X3 (VL53L1X.kicad_sch)
- note removed: "ADDRESS: 1000000"
- note removed: "D+ and D- is just I/O, so just cosmetic ig"
- note removed: "IMU"
- note removed: "LEFT"
- note removed: "PROBABLY JUST GROUND GPIO5 AND GPIO 6"
- note removed: "PWM"
- note removed: "RIGHT"
- note removed: "ROTARY ENCODER"
- note removed: "SWIM NC"
- note removed: "THIS IS TEMPORARY PLACEMENT"
- note removed: "TMC2209"
- note removed: "USB"
- note removed: "VL53L1X"
- note removed: "VL53L1X DECOUP"
- note removed: "dw3220 gets separate ldos"
- note removed: "just do the rest of the decoup later, prolly add more bulk capacitors add ferrite bead"
- note removed: "prolly get a coin battery? not required. (for vbat)"
