File: ELECTRONICS/MAINBOARD/autobot_mainboard.kicad_sch (KiCad schematic)
At the start: 0 parts

Commit message: 9/4
Other:
- note added: "just do 1"
Changed lines of the file:
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@@
 	(generator_version "10.0")
 	(paper "A4")
+	(text "just do 1\n"
+		(exclude_from_sim no)
+		(at 86.106 45.72 0)
+		(effects
+			(font
+				(size 1.27 1.27)
+			)
+		)
+	)
 	(junction
 		(at 224.79 27.94)
@@
 		)
 		(instances
-			(project "betterschematicbotig"
+			(project "autobot_mainboard"
 				(path "/f053f1d0-b1f5-4f80-9758-8ee1a2d3659d"
 					(reference "#PWR02")
@@
 		)
 		(instances
-			(project "betterschematicbotig"
+			(project "autobot_mainboard"
 				(path "/f053f1d0-b1f5-4f80-9758-8ee1a2d3659d"
 					(reference "#PWR064")
@@
 		)
 		(instances
-			(project "betterschematicbotig"
+			(project "autobot_mainboard"
 				(path "/f053f1d0-b1f5-4f80-9758-8ee1a2d3659d"
 					(reference "#PWR065")
@@
 		)
 		(instances
-			(project "betterschematicbotig"
+			(project "autobot_mainboard"
 				(path "/f053f1d0-b1f5-4f80-9758-8ee1a2d3659d"
 					(reference "#PWR063")
@@
 		)
 		(instances
-			(project "betterschematicbotig"
+			(project "autobot_mainboard"
 				(path "/f053f1d0-b1f5-4f80-9758-8ee1a2d3659d"
 					(reference "#PWR069")
@@
 		)
 		(instances
-			(project "betterschematicbotig"
+			(project "autobot_mainboard"
 				(path "/f053f1d0-b1f5-4f80-9758-8ee1a2d3659d"
 					(reference "#PWR060")
@@
 		)
 		(instances
-			(project "betterschematicbotig"
+			(project "autobot_mainboard"
 				(path "/f053f1d0-b1f5-4f80-9758-8ee1a2d3659d"
 					(reference "#PWR061")
@@
 		)
 		(instances
-			(project "betterschematicbotig"
+			(project "autobot_mainboard"
 				(path "/f053f1d0-b1f5-4f80-9758-8ee1a2d3659d"
 					(page "10")
@@
 		)
 		(instances
-			(project "betterschematicbotig"
+			(project "autobot_mainboard"
 				(path "/f053f1d0-b1f5-4f80-9758-8ee1a2d3659d"
 					(page "20")
@@
 		)
 		(instances
-			(project "betterschematicbotig"
+			(project "autobot_mainboard"
 				(path "/f053f1d0-b1f5-4f80-9758-8ee1a2d3659d"
 					(page "9")
@@
 		)
 		(instances
-			(project "betterschematicbotig"
+			(project "autobot_mainboard"
 				(path "/f053f1d0-b1f5-4f80-9758-8ee1a2d3659d"
 					(page "22")
@@
 		)
 		(instances
-			(project "betterschematicbotig"
+			(project "autobot_mainboard"
 				(path "/f053f1d0-b1f5-4f80-9758-8ee1a2d3659d"
 					(page "23")
@@
 		)
 		(instances
-			(project "betterschematicbotig"
+			(project "autobot_mainboard"
 				(path "/f053f1d0-b1f5-4f80-9758-8ee1a2d3659d"
 					(page "8")
@@
 		)
 		(instances
-			(project "betterschematicbotig"
+			(project "autobot_mainboard"
 				(path "/f053f1d0-b1f5-4f80-9758-8ee1a2d3659d"
 					(page "5")
@@
 		)
 		(instances
-			(project "betterschematicbotig"
+			(project "autobot_mainboard"
 				(path "/f053f1d0-b1f5-4f80-9758-8ee1a2d3659d"
 					(page "2")
@@
 		)
 		(instances
-			(project "betterschematicbotig"
+			(project "autobot_mainboard"
 				(path "/f053f1d0-b1f5-4f80-9758-8ee1a2d3659d"
 					(page "17")
@@
 		)
 		(instances
-			(project "betterschematicbotig"
+			(project "autobot_mainboard"
 				(path "/f053f1d0-b1f5-4f80-9758-8ee1a2d3659d"
 					(page "4")
@@
 		)
 		(instances
-			(project "betterschematicbotig"
+			(project "autobot_mainboard"
 				(path "/f053f1d0-b1f5-4f80-9758-8ee1a2d3659d"
 					(page "7")
@@
 		)
 		(pin "RXD0" output
-			(at 121.92 129.54 180)
+			(at 121.92 158.75 180)
 			(effects
 				(font
@@
 		)
 		(pin "RXD1" output
-			(at 121.92 158.75 180)
+			(at 121.92 129.54 180)
 			(effects
 				(font
@@
 		)
 		(pin "TXD0" input
-			(at 121.92 132.08 180)
+			(at 121.92 161.29 180)
 			(effects
 				(font
@@
 		)
 		(pin "TXD1" input
-			(at 121.92 161.29 180)
+			(at 121.92 132.08 180)
 			(effects
 				(font
@@
 		)
 		(instances
-			(project "betterschematicbotig"
+			(project "autobot_mainboard"
 				(path "/f053f1d0-b1f5-4f80-9758-8ee1a2d3659d"
 					(page "21")
@@
 		)
 		(instances
-			(project "betterschematicbotig"
+			(project "autobot_mainboard"
 				(path "/f053f1d0-b1f5-4f80-9758-8ee1a2d3659d"
 					(page "6")
@@
 		)
 		(instances
-			(project "betterschematicbotig"
+			(project "autobot_mainboard"
 				(path "/f053f1d0-b1f5-4f80-9758-8ee1a2d3659d"
 					(page "13")
@@
 		)
 		(instances
-			(project "betterschematicbotig"
+			(project "autobot_mainboard"
 				(path "/f053f1d0-b1f5-4f80-9758-8ee1a2d3659d"
 					(page "15")
@@
 		)
 		(instances
-			(project "betterschematicbotig"
+			(project "autobot_mainboard"
 				(path "/f053f1d0-b1f5-4f80-9758-8ee1a2d3659d"
 					(page "25")
@@
 		)
 		(instances
-			(project "betterschematicbotig"
+			(project "autobot_mainboard"
 				(path "/f053f1d0-b1f5-4f80-9758-8ee1a2d3659d"
 					(page "24")
@@
 		)
 		(instances
-			(project "betterschematicbotig"
+			(project "autobot_mainboard"
 				(path "/f053f1d0-b1f5-4f80-9758-8ee1a2d3659d"
 					(page "19")
@@
 		)
 		(instances
-			(project "betterschematicbotig"
+			(project "autobot_mainboard"
 				(path "/f053f1d0-b1f5-4f80-9758-8ee1a2d3659d"
 					(page "12")
@@
 		)
 		(instances
-			(project "betterschematicbotig"
+			(project "autobot_mainboard"
 				(path "/f053f1d0-b1f5-4f80-9758-8ee1a2d3659d"
 					(page "14")
@@
 		)
 		(instances
-			(project "betterschematicbotig"
+			(project "autobot_mainboard"
 				(path "/f053f1d0-b1f5-4f80-9758-8ee1a2d3659d"
 					(page "3")
@@
 		)
 		(instances
-			(project "betterschematicbotig"
+			(project "autobot_mainboard"
 				(path "/f053f1d0-b1f5-4f80-9758-8ee1a2d3659d"
 					(page "11")

Commit message: Add files via upload
Other:
- removed sheet DW3220_B
- removed sheet LDO2
- added sheet ESC (ESC.kicad_sch)
- note removed: "just do 1"

Commit message: Add files via upload
Other:
- sheet ESC renamed STM32G0
- sheet POWER_CONNECTOR ports: added none; removed 24V
- sheet STM32H743 ports: added none; removed AMT_A_L, AMT_A_R, AMT_B_L, AMT_B_R, AMT_X_L, AMT_X_R, CSN_B, IRQ_B, MISO_B, MOSI_B, RESET_B, SPICLK_B, WAKEUP_B

Commit message: Add files via upload
Other:
- added sheet LDO2 (LDO.kicad_sch)
- added sheet Power_connector_g0 (Power_connector_g0.kicad_sch)
- sheet STM32G0 ports: added 24V, 3V3, AMT_A_L, AMT_A_R, AMT_B_L, AMT_B_R, AMT_X_L, AMT_X_R, USART_RX, USART_TX; removed none
- sheet STM32H743 ports: added USART_RX, USART_TX; removed none
