File: ELECTRONICS/MAINBOARD/autobot_mainboard.kicad_sch (KiCad schematic)
At the start: 0 parts

Commit message: Add files via upload
Other:
- removed sheet MOTOR_CONNECTOR_L
- removed sheet MOTOR_CONNECTOR_R
- removed sheet TMC2209_L
- removed sheet TMC2209_R
- sheet STM32H743 ports: added none; removed DIAG_L, DIAG_R, DIR_L, DIR_R, INDEX_L, INDEX_R, RXD0, RXD1, STEP_L, STEP_R, TMC_EN_L, TMC_EN_R, TXD0, TXD1
