File: ELECTRONICS/MAINBOARD/MCT8316Z.kicad_sch (KiCad schematic)
At the start: 9 parts, among them U14 MCT8316ZR

Commit message: Add files via upload
Parts:
- added C74: 10u, symbol Device:C_Polarized
- added C76: 100n, symbol Device:C
- renumbered C45 to C75, C59 to C77, C48 to C78, C57 to C79, L1 to L2, R9 to R23, R23 to R24, R27 to R25, U14 to U20
Connections:
- net +24V: now also C74.1, C76.1
- net BLDC_CONNECTOR/HALL_A: no longer U20.27 (HPA)
- net BLDC_CONNECTOR/HALL_B: no longer U20.29 (HPB)
- net BLDC_CONNECTOR/HALL_C: no longer U20.31 (HPC)
- net GNDREF: now also C74.2, C76.2; no longer U20.28 (HNA), U20.30 (HNB), U20.32 (HNC)
- new net HALL_A/N: U20.28 (HNA)
- new net HALL_A/P: U20.27 (HPA)
- new net HALL_B/N: U20.30 (HNB)
- new net HALL_B/P: U20.29 (HPB)
- new net HALL_C/N: U20.32 (HNC)
- new net HALL_C/P: U20.31 (HPC)
Other:
- added sheet HALL_A (Hall_Sensor.kicad_sch)
- added sheet HALL_B (Hall_Sensor.kicad_sch)
- added sheet HALL_C (Hall_Sensor.kicad_sch)
- sheet BLDC_CONNECTOR ports: added 5V/3V3; removed none
- note added: "digital hall sensor config (single ended)"
- moved on the sheet: C77, C79, U20

Commit message: Add files via upload
Parts:
- added C97: 100n, Capacitor_SMD:C_0402_1005Metric, symbol Device:C
- added R47: r, Capacitor_SMD:C_0402_1005Metric, symbol Device:R
- C75: value C -> 22u; footprint (none) -> Capacitor_SMD:C_0402_1005Metric
- C76, C77, C78, C79, R23, R24: footprint (none) -> Capacitor_SMD:C_0402_1005Metric
- L2: value L -> 47u
- R25: value 10k -> r; footprint (none) -> Capacitor_SMD:C_0402_1005Metric
Connections:
- net +24V: now also C97.1
- net GNDREF: now also R25.2, C97.2
- net VDD: now also R47.1
- net at R25.1, U20.37 (ILIM): now also R47.2
Other:
- moved on the sheet: C74, R25

Commit message: Add files via upload
Parts:
- removed C75: 22u, Capacitor_SMD:C_0402_1005Metric, symbol Device:C
- C74: value 10u -> 100u; footprint (none) -> MyFootprintLibrary:CAP-SMD_BD6.3-L6.6-W6.6-LS7.3-FD
- C78: value C -> 1u
- L2: footprint (none) -> MyFootprintLibrary:IND-SMD_L4.0-W4.0
Connections:
- net GNDREF: now also C78.2, U20.2 (AGND), U20.26 (AGND), U20.41 (GNDPAD)
- net VDD: no longer C78.2, U20.2 (AGND), U20.26 (AGND)
Other:
- moved on the sheet: C74, C76, C97

Commit message: commit 1 commit 1 10/03/2026
Parts:
- added C81: 22u, Capacitor_SMD:C_0805_2012Metric, symbol Device:C
Connections:
- net GNDREF: now also C81.2
- net VDD: now also C81.1
Changed lines of the file:
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@@
+	)
+	(symbol
+		(lib_id "Device:C")
+		(at 93.98 52.07 0)
+		(unit 1)
+		(body_style 1)
+		(exclude_from_sim no)
+		(in_bom yes)
+		(on_board yes)
+		(in_pos_files yes)
+		(dnp no)
+		(property "Reference" "C81"
+			(at 94.742 50.038 0)
+			(show_name no)
+			(do_not_autoplace no)
+			(effects
+				(font
+					(size 1.27 1.27)
+				)
+				(justify left)
+			)
+		)
+		(property "Value" "22u"
+			(at 94.488 54.102 0)
+			(show_name no)
+			(do_not_autoplace no)
+			(effects
+				(font
+					(size 1.27 1.27)
+				)
+				(justify left)
+			)
+		)
+		(property "Footprint" "Capacitor_SMD:C_0805_2012Metric"
+			(at 94.9452 55.88 0)
+			(hide yes)
+			(show_name no)
+			(do_not_autoplace no)
+			(effects
+				(font
+					(size 1.27 1.27)
+				)
+			)
+		)
+		(property "Datasheet" ""
+			(at 93.98 52.07 0)
+			(hide yes)
+			(show_name no)
+			(do_not_autoplace no)
+			(effects
+				(font
+					(size 1.27 1.27)
+				)
+			)
+		)
+		(property "Description" "Unpolarized capacitor"
+			(at 93.98 52.07 0)
+			(hide yes)
+			(show_name no)
+			(do_not_autoplace no)
+			(effects
+				(font
+					(size 1.27 1.27)
+				)
+			)
+		)
+		(pin "2"
+		)
+		(pin "1"
+		)
+		(instances
+			(project "autobot_mainboard"
+				(path "/f053f1d0-b1f5-4f80-9758-8ee1a2d3659d/f3a82e5b-62e6-4c1f-9ee9-6ab064c88bd0/35b0743f-bfc0-4c80-81d1-a26461aee3a5"
+					(reference "C81")
+					(unit 1)
+				)
+				(path "/f053f1d0-b1f5-4f80-9758-8ee1a2d3659d/f3a82e5b-62e6-4c1f-9ee9-6ab064c88bd0/a979bc8f-363d-4880-b49b-89facb6aaa9b"
+					(reference "C99")
+					(unit 1)
+				)
+			)
+		)
 	)
 	(symbol
