File: ELECTRONICS/MAINBOARD/DW3220.kicad_sch (KiCad schematic)
At the start: 31 parts, among them IC1 DW3210, J7 Conn_01x03_Pin, J8 Conn_Coaxial, J9 Conn_Coaxial, Q1 DMG1012T, Q2 DMG1012T, Q3 DMG1012T, Y1 TXC 8Y38472012

Commit message: change tvs1400 to another tvs with higher clamping voltage. fix footprints and add nreset
Parts:
- IC1: footprint (none) -> MyFootprintLibrary:qfn_DW3220_QOR-M
Changed lines of the file:
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@@
 			)
 		)
-		(property "Footprint" ""
+		(property "Footprint" "MyFootprintLibrary:qfn_DW3220_QOR-M"
 			(at 92.71 182.55 0)
 			(hide yes)

Commit message: commit 1 commit 1 10/03/2026
Parts:
- IC1: footprint MyFootprintLibrary:qfn_DW3220_QOR-M -> QFN40P500X500X80-40N-D
Changed lines of the file:
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@@
 			)
 		)
-		(property "Footprint" "MyFootprintLibrary:qfn_DW3220_QOR-M"
+		(property "Footprint" "QFN40P500X500X80-40N-D"
 			(at 92.71 182.55 0)
 			(hide yes)

Commit message: driver board schematic
Parts:
- IC1: footprint QFN40P500X500X80-40N-D -> (none)
Changed lines of the file:
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@@
 			)
 		)
-		(property "Footprint" "QFN40P500X500X80-40N-D"
+		(property "Footprint" ""
 			(at 92.71 182.55 0)
 			(hide yes)
