File: ELECTRONICS/MAINBOARD/DW3220.kicad_sch (KiCad schematic)
At the start: 31 parts, among them IC1 DW3210, J7 Conn_Coaxial, J8 Conn_Coaxial, J9 Conn_01x03_Pin, Q1 DMG1012T, Q2 DMG1012T, Q3 DMG1012T, Y1 TXC 8Y38472012

Commit message: Add files via upload
Parts:
- renumbered C20 to C38, C31 to C39, C21 to C40, C4 to C41, C5 to C42, C24 to C43, C25 to C44, C2 to C45, C26 to C46, C27 to C47, C3 to C48, C28 to C49, C29 to C50, C32 to C51, C33 to C52, D3 to D2, D5 to D3, FB1 to FB2, J8 to J10, J9 to J8, J7 to J9, Q3 to Q2, Q2 to Q3, R15 to R17, R16 to R18, R17 to R19

Commit message: Add files via upload
Parts:
- renumbered J8 to J7, J9 to J8, J10 to J9
Changed lines of the file:
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@@
 		(dnp no)
 		(fields_autoplaced yes)
-		(property "Reference" "#PWR082"
+		(property "Reference" "#PWR081"
 			(at 162.56 121.92 0)
 			(hide yes)
@@
 			(project "autobot_mainboard"
 				(path "/f053f1d0-b1f5-4f80-9758-8ee1a2d3659d/b49e282a-c8ff-467d-bc65-06b02df06bd0"
-					(reference "#PWR082")
+					(reference "#PWR081")
 					(unit 1)
 				)
@@
 		(dnp no)
 		(fields_autoplaced yes)
-		(property "Reference" "#PWR075"
+		(property "Reference" "#PWR074"
 			(at 121.92 124.46 0)
 			(hide yes)
@@
 			(project "autobot_mainboard"
 				(path "/f053f1d0-b1f5-4f80-9758-8ee1a2d3659d/b49e282a-c8ff-467d-bc65-06b02df06bd0"
-					(reference "#PWR075")
+					(reference "#PWR074")
 					(unit 1)
 				)
@@
 		(dnp no)
 		(fields_autoplaced yes)
-		(property "Reference" "#PWR071"
+		(property "Reference" "#PWR070"
 			(at 114.3 100.33 0)
 			(hide yes)
@@
 			(project "autobot_mainboard"
 				(path "/f053f1d0-b1f5-4f80-9758-8ee1a2d3659d/b49e282a-c8ff-467d-bc65-06b02df06bd0"
-					(reference "#PWR071")
+					(reference "#PWR070")
 					(unit 1)
 				)
@@
 		(dnp no)
 		(fields_autoplaced yes)
-		(property "Reference" "#PWR078"
+		(property "Reference" "#PWR077"
 			(at 138.43 29.21 0)
 			(hide yes)
@@
 			(project "autobot_mainboard"
 				(path "/f053f1d0-b1f5-4f80-9758-8ee1a2d3659d/b49e282a-c8ff-467d-bc65-06b02df06bd0"
-					(reference "#PWR078")
+					(reference "#PWR077")
 					(unit 1)
 				)
@@
 		(in_pos_files yes)
 		(dnp no)
-		(property "Reference" "J10"
+		(property "Reference" "J9"
 			(at 166.37 108.2431 0)
 			(show_name no)
@@
 			(project "autobot_mainboard"
 				(path "/f053f1d0-b1f5-4f80-9758-8ee1a2d3659d/b49e282a-c8ff-467d-bc65-06b02df06bd0"
-					(reference "J10")
+					(reference "J9")
 					(unit 1)
 				)
@@
 		(dnp no)
 		(fields_autoplaced yes)
-		(property "Reference" "#PWR068"
+		(property "Reference" "#PWR067"
 			(at 110.49 153.67 0)
 			(hide yes)
@@
 			(project "autobot_mainboard"
 				(path "/f053f1d0-b1f5-4f80-9758-8ee1a2d3659d/b49e282a-c8ff-467d-bc65-06b02df06bd0"
-					(reference "#PWR068")
+					(reference "#PWR067")
 					(unit 1)
 				)
@@
 		(dnp no)
 		(fields_autoplaced yes)
-		(property "Reference" "#PWR080"
+		(property "Reference" "#PWR079"
 			(at 156.21 153.67 0)
 			(hide yes)
@@
 			(project "autobot_mainboard"
 				(path "/f053f1d0-b1f5-4f80-9758-8ee1a2d3659d/b49e282a-c8ff-467d-bc65-06b02df06bd0"
-					(reference "#PWR080")
+					(reference "#PWR079")
 					(unit 1)
 				)
@@
 		(in_pos_files yes)
 		(dnp no)
-		(property "Reference" "#PWR077"
+		(property "Reference" "#PWR076"
 			(at 128.27 85.09 0)
 			(hide yes)
@@
 			(project "autobot_mainboard"
 				(path "/f053f1d0-b1f5-4f80-9758-8ee1a2d3659d/b49e282a-c8ff-467d-bc65-06b02df06bd0"
-					(reference "#PWR077")
+					(reference "#PWR076")
 					(unit 1)
 				)
@@
 		(dnp no)
 		(fields_autoplaced yes)
-		(property "Reference" "#PWR081"
+		(property "Reference" "#PWR080"
 			(at 162.56 107.95 0)
 			(hide yes)
@@
 			(project "autobot_mainboard"
 				(path "/f053f1d0-b1f5-4f80-9758-8ee1a2d3659d/b49e282a-c8ff-467d-bc65-06b02df06bd0"
-					(reference "#PWR081")
+					(reference "#PWR080")
 					(unit 1)
 				)
@@
 		(dnp no)
 		(fields_autoplaced yes)
-		(property "Reference" "#PWR079"
+		(property "Reference" "#PWR078"
 			(at 138.43 62.23 0)
 			(hide yes)
@@
 			(project "autobot_mainboard"
 				(path "/f053f1d0-b1f5-4f80-9758-8ee1a2d3659d/b49e282a-c8ff-467d-bc65-06b02df06bd0"
-					(reference "#PWR079")
+					(reference "#PWR078")
 					(unit 1)
 				)
@@
 		(dnp no)
 		(fields_autoplaced yes)
-		(property "Reference" "#PWR067"
+		(property "Reference" "#PWR066"
 			(at 106.68 135.89 0)
 			(hide yes)
@@
 			(project "autobot_mainboard"
 				(path "/f053f1d0-b1f5-4f80-9758-8ee1a2d3659d/b49e282a-c8ff-467d-bc65-06b02df06bd0"
-					(reference "#PWR067")
+					(reference "#PWR066")
 					(unit 1)
 				)
@@
 		(dnp no)
 		(fields_autoplaced yes)
-		(property "Reference" "#PWR072"
+		(property "Reference" "#PWR071"
 			(at 114.3 124.46 0)
 			(hide yes)
@@
 			(project "autobot_mainboard"
 				(path "/f053f1d0-b1f5-4f80-9758-8ee1a2d3659d/b49e282a-c8ff-467d-bc65-06b02df06bd0"
-					(reference "#PWR072")
+					(reference "#PWR071")
 					(unit 1)
 				)
@@
 		(dnp no)
 		(fields_autoplaced yes)
-		(property "Reference" "#PWR084"
+		(property "Reference" "#PWR083"
 			(at 163.83 62.23 0)
 			(hide yes)
@@
 			(project "autobot_mainboard"
 				(path "/f053f1d0-b1f5-4f80-9758-8ee1a2d3659d/b49e282a-c8ff-467d-bc65-06b02df06bd0"
-					(reference "#PWR084")
+					(reference "#PWR083")
 					(unit 1)
 				)
@@
 		(dnp no)
 		(fields_autoplaced yes)
-		(property "Reference" "#PWR076"
+		(property "Reference" "#PWR075"
 			(at 121.92 135.89 0)
 			(hide yes)
@@
 			(project "autobot_mainboard"
 				(path "/f053f1d0-b1f5-4f80-9758-8ee1a2d3659d/b49e282a-c8ff-467d-bc65-06b02df06bd0"
-					(reference "#PWR076")
+					(reference "#PWR075")
 					(unit 1)
 				)
@@
 		(dnp no)
 		(fields_autoplaced yes)
-		(property "Reference" "#PWR069"
+		(property "Reference" "#PWR068"
 			(at 113.03 29.21 0)
 			(hide yes)
@@
 			(project "autobot_mainboard"
 				(path "/f053f1d0-b1f5-4f80-9758-8ee1a2d3659d/b49e282a-c8ff-467d-bc65-06b02df06bd0"
-					(reference "#PWR069")
+					(reference "#PWR068")
 					(unit 1)
 				)
@@
 		(dnp no)
 		(fields_autoplaced yes)
-		(property "Reference" "#PWR074"
+		(property "Reference" "#PWR073"
 			(at 121.92 100.33 0)
 			(hide yes)
@@
 			(project "autobot_mainboard"
 				(path "/f053f1d0-b1f5-4f80-9758-8ee1a2d3659d/b49e282a-c8ff-467d-bc65-06b02df06bd0"
-					(reference "#PWR074")
+					(reference "#PWR073")
 					(unit 1)
 				)
@@
 		(dnp no)
 		(fields_autoplaced yes)
-		(property "Reference" "#PWR062"
+		(property "Reference" "#PWR061"
 			(at 24.13 125.73 0)
 			(hide yes)
@@
 			(project "autobot_mainboard"
 				(path "/f053f1d0-b1f5-4f80-9758-8ee1a2d3659d/b49e282a-c8ff-467d-bc65-06b02df06bd0"
-					(reference "#PWR062")
+					(reference "#PWR061")
 					(unit 1)
 				)
@@
 		(dnp no)
 		(fields_autoplaced yes)
-		(property "Reference" "#PWR063"
+		(property "Reference" "#PWR062"
 			(at 67.31 160.02 0)
 			(hide yes)
@@
 			(project "autobot_mainboard"
 				(path "/f053f1d0-b1f5-4f80-9758-8ee1a2d3659d/b49e282a-c8ff-467d-bc65-06b02df06bd0"
-					(reference "#PWR063")
+					(reference "#PWR062")
 					(unit 1)
 				)
@@
 		(dnp no)
 		(fields_autoplaced yes)
-		(property "Reference" "#PWR065"
+		(property "Reference" "#PWR064"
 			(at 106.68 111.76 0)
 			(hide yes)
@@
 			(project "autobot_mainboard"
 				(path "/f053f1d0-b1f5-4f80-9758-8ee1a2d3659d/b49e282a-c8ff-467d-bc65-06b02df06bd0"
-					(reference "#PWR065")
+					(reference "#PWR064")
 					(unit 1)
 				)
@@
 		(dnp no)
 		(fields_autoplaced yes)
-		(property "Reference" "#PWR073"
+		(property "Reference" "#PWR072"
 			(at 114.3 135.89 0)
 			(hide yes)
@@
 			(project "autobot_mainboard"
 				(path "/f053f1d0-b1f5-4f80-9758-8ee1a2d3659d/b49e282a-c8ff-467d-bc65-06b02df06bd0"
-					(reference "#PWR073")
+					(reference "#PWR072")
 					(unit 1)
 				)
@@
 		(dnp no)
 		(fields_autoplaced yes)
-		(property "Reference" "#PWR064"
+		(property "Reference" "#PWR063"
 			(at 102.87 156.21 0)
 			(hide yes)
@@
 			(project "autobot_mainboard"
 				(path "/f053f1d0-b1f5-4f80-9758-8ee1a2d3659d/b49e282a-c8ff-467d-bc65-06b02df06bd0"
-					(reference "#PWR064")
+					(reference "#PWR063")
 					(unit 1)
 				)
@@
 		(dnp no)
 		(fields_autoplaced yes)
-		(property "Reference" "#PWR066"
+		(property "Reference" "#PWR065"
 			(at 106.68 124.46 0)
 			(hide yes)
@@
 			(project "autobot_mainboard"
 				(path "/f053f1d0-b1f5-4f80-9758-8ee1a2d3659d/b49e282a-c8ff-467d-bc65-06b02df06bd0"
-					(reference "#PWR066")
+					(reference "#PWR065")
 					(unit 1)
 				)
@@
 		(dnp no)
 		(fields_autoplaced yes)
-		(property "Reference" "#PWR070"
+		(property "Reference" "#PWR069"
 			(at 113.03 62.23 0)
 			(hide yes)
@@
 			(project "autobot_mainboard"
 				(path "/f053f1d0-b1f5-4f80-9758-8ee1a2d3659d/b49e282a-c8ff-467d-bc65-06b02df06bd0"
-					(reference "#PWR070")
+					(reference "#PWR069")
 					(unit 1)
 				)
@@
 		(in_pos_files yes)
 		(dnp no)
-		(property "Reference" "J9"
+		(property "Reference" "J8"
 			(at 166.37 94.2731 0)
 			(show_name no)
@@
 			(project "autobot_mainboard"
 				(path "/f053f1d0-b1f5-4f80-9758-8ee1a2d3659d/b49e282a-c8ff-467d-bc65-06b02df06bd0"
-					(reference "J9")
+					(reference "J8")
 					(unit 1)
 				)
@@
 		(dnp no)
 		(fields_autoplaced yes)
-		(property "Reference" "J8"
+		(property "Reference" "J7"
 			(at 156.845 69.85 0)
 			(show_name no)
@@
 			(project "autobot_mainboard"
 				(path "/f053f1d0-b1f5-4f80-9758-8ee1a2d3659d/b49e282a-c8ff-467d-bc65-06b02df06bd0"
-					(reference "J8")
+					(reference "J7")
 					(unit 1)
 				)
@@
 		(dnp no)
 		(fields_autoplaced yes)
-		(property "Reference" "#PWR083"
+		(property "Reference" "#PWR082"
 			(at 163.83 29.21 0)
 			(hide yes)
@@
 			(project "autobot_mainboard"
 				(path "/f053f1d0-b1f5-4f80-9758-8ee1a2d3659d/b49e282a-c8ff-467d-bc65-06b02df06bd0"
-					(reference "#PWR083")
+					(reference "#PWR082")
 					(unit 1)
 				)

Commit message: rollback
Parts:
- renumbered C38 to C33, C39 to C34, C40 to C35, C41 to C36, C42 to C37, C43 to C38, C44 to C39, C45 to C40, C46 to C41, C47 to C42, C48 to C43, C49 to C44, C50 to C45, C51 to C46, C52 to C47, D2 to D7, D3 to D8, D4 to D9, J7 to J10, J8 to J11, J9 to J12, Q1 to Q2, Q2 to Q3, Q3 to Q4
