File: ELECTRONICS/MAINBOARD/BMI270.kicad_sch (KiCad schematic)
At the start: 4 parts, among them U13 BMI270

Commit message: commit 1 commit 1 10/03/2026
Parts:
- U13: footprint MyFootprintLibrary:BMI270_BOS-M -> BMI270_BOS
Changed lines of the file:
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@@
 			)
 		)
-		(property "Footprint" "MyFootprintLibrary:BMI270_BOS-M"
+		(property "Footprint" "BMI270_BOS"
 			(at 91.44 55.88 0)
 			(hide yes)

Commit message: driver board schematic
Parts:
- U13: footprint BMI270_BOS -> (none)
Changed lines of the file:
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@@
 			)
 		)
-		(property "Footprint" "BMI270_BOS"
+		(property "Footprint" ""
 			(at 91.44 55.88 0)
 			(hide yes)

Commit message: change tvs1400 to another tvs with higher clamping voltage. fix footprints and add nreset
Parts:
- U13: footprint (none) -> MyFootprintLibrary:BMI270_BOS-M
Changed lines of the file:
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@@
 			)
 		)
-		(property "Footprint" ""
+		(property "Footprint" "MyFootprintLibrary:BMI270_BOS-M"
 			(at 91.44 55.88 0)
 			(hide yes)
