File: ELECTRONICS/MAINBOARD/STM32H743.kicad_sch (KiCad schematic)
At the start: 28 parts, among them J13 Conn_01x05_Socket, J6 Conn_01x05_Socket, SW1 RESET, SW2 BOOT, U16 STM32H743ZITx, Y3 25mhz placeholder

Commit message: 9/4
Connections:
- net AMT_A_L: now also U16.136 (PB6)
- net AMT_A_R: now also U16.60 (PE9)
- net AMT_B_L: now also U16.137 (PB7)
- net AMT_B_R: now also U16.64 (PE11)
- net AMT_X_L: now also U16.132 (PG15)
- net AMT_X_R: now also U16.65 (PE12)
- net DIAG_L: now also U16.2 (PE3)
- net DIAG_R: now also U16.76 (PB15)
- net DIR_L: now also U16.139 (PB8); no longer U16.140 (PB9)
- net DIR_R: now also U16.68 (PE15); no longer U16.77 (PD8)
- net INDEX_L: now also U16.1 (PE2)
- net INDEX_R: now also U16.75 (PB14)
- net IRQ_T: now also U16.36 (PA2)
- net MISO_T: now also U16.42 (PA6)
- net MOSI_T: now also U16.43 (PA7)
- net RESET_T: now also U16.37 (PA3)
- net RXD0: now also U16.142 (PE1)
- net RXD1: now also U16.73 (PB12)
- net SPICLK_T: now also U16.41 (PA5)
- net STEP_L: now also U16.140 (PB9); no longer U16.141 (PE0)
- net STEP_R: now also U16.69 (PB10); no longer U16.75 (PB14)
- net TMC_EN_L: now also U16.3 (PE4)
- net TXD0: now also U16.141 (PE0)
- net TXD1: now also U16.74 (PB13)
- net WAKEUP_T: now also U16.40 (PA4)

Commit message: Add files via upload
Parts:
- removed U16: STM32H743ZITx, Package_QFP:LQFP-144_20x20mm_P0.5mm, symbol MCU_ST_STM32H7:STM32H743ZITx
- added U10: STM32H743VITx, Package_QFP:LQFP-100_14x14mm_P0.5mm, symbol MCU_ST_STM32H7:STM32H743VITx
Connections:
- net +3V3: now also U10.100 (VDD), U10.11 (VDD), U10.27 (VDD), U10.50 (VDD), U10.6 (VBAT), U10.75 (VDD)
- net BOOT0: now also U10.94 (BOOT0)
- net D+: now also U10.71 (PA12)
- net D-: now also U10.70 (PA11)
- net DIAG_L: now also U10.2 (PE3)
- net DIR_L: now also U10.95 (PB8)
- net INDEX_L: now also U10.1 (PE2)
- net NRST: now also U10.14 (NRST)
- net PH0: now also U10.12 (PH0)
- net PH1: now also U10.13 (PH1)
- net RXD0: now also U10.97 (PE0)
- net STEP_L: now also U10.96 (PB9)
- net SWCLK: now also U10.76 (PA14)
- net SWDIO: now also U10.72 (PA13)
- net TXD0: now also U10.98 (PE1)
- net VREF: now also U10.20 (VREF+)
- net at C82.1, C83.1, FB5.2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: now also U10.21 (VDDA)
- net at C63.1: now also U10.73 (VCAP)
- net at C62.1: now also U10.48 (VCAP)
- new net: U10.10 (VSS), U10.26 (VSS), U10.49 (VSS), U10.74 (VSS), U10.99 (VSS)
Other:
- moved on the sheet: C61, C62, C63, C81, C82, C83, FB5, J13, J6, R25, R26, SW1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

Commit message: Add files via upload
Parts:
- renumbered C79 to C55, C80 to C56, C61 to C57, C62 to C58, C63 to C59, C81 to C60, C82 to C61, C83 to C62, C64 to C63, C65 to C64, C66 to C65, C67 to C66, C68 to C67, C69 to C68, C70 to C69, C71 to C70, C72 to C71, C73 to C72, C74 to C73, FB5 to FB3, J6 to J11, J13 to J12, R25 to R21, R26 to R22, U10 to U19, Y3 to Y2

Commit message: Add files via upload
Changed lines of the file:
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@@
-	(wire
-		(pts
-			(xy 132.08 132.08) (xy 139.7 132.08)
-		)
-		(stroke
-			(width 0)
-			(type default)
-		)
-	)
 	(wire
 		(pts
@@
 	(wire
 		(pts
-			(xy 132.08 140.97) (xy 135.89 140.97)
-		)
-		(stroke
-			(width 0)
-			(type default)
-		)
-	)
-	(wire
-		(pts
 			(xy 226.06 78.74) (xy 233.68 78.74)
 		)
@@
 	(wire
 		(pts
-			(xy 132.08 143.51) (xy 135.89 143.51)
-		)
-		(stroke
-			(width 0)
-			(type default)
-		)
-	)
-	(wire
-		(pts
 			(xy 317.5 41.91) (xy 317.5 43.18)
 		)
@@
 	(wire
 		(pts
-			(xy 132.08 129.54) (xy 139.7 129.54)
-		)
-		(stroke
-			(width 0)
-			(type default)
-		)
-	)
-	(wire
-		(pts
-			(xy 140.97 118.11) (xy 132.08 118.11)
-		)
-		(stroke
-			(width 0)
-			(type default)
-		)
-	)
-	(wire
-		(pts
 			(xy 140.97 90.17) (xy 140.97 92.71)
 		)
@@
 		(pts
 			(xy 287.02 43.18) (xy 294.64 43.18)
-		)
-		(stroke
-			(width 0)
-			(type default)
-		)
-	)
-	(wire
-		(pts
-			(xy 132.08 135.89) (xy 135.89 135.89)
 		)
 		(stroke
@@
 		)
 	)
-	(hierarchical_label "AMT_B_L"
-		(shape output)
-		(at 132.08 129.54 180)
-		(effects
-			(font
-				(size 1.27 1.27)
-			)
-			(justify right)
-		)
-	)
-	(hierarchical_label "AMT_B_R"
-		(shape output)
-		(at 132.08 140.97 180)
-		(effects
-			(font
-				(size 1.27 1.27)
-			)
-			(justify right)
-		)
-	)
 	(hierarchical_label "CSN_T"
 		(shape output)
@@
 		)
 	)
-	(hierarchical_label "AMT_A_L"
-		(shape output)
-		(at 132.08 132.08 180)
-		(effects
-			(font
-				(size 1.27 1.27)
-			)
-			(justify right)
-		)
-	)
 	(hierarchical_label "BMI_SCK_L"
 		(shape bidirectional)
@@
 		)
 	)
-	(hierarchical_label "AMT_X_R"
-		(shape output)
-		(at 132.08 143.51 180)
+	(hierarchical_label "BMI_CS_R"
+		(shape bidirectional)
+		(at -29.21 162.56 0)
+		(effects
+			(font
+				(size 1.27 1.27)
+			)
+			(justify left)
+		)
+	)
+	(hierarchical_label "BMI_INT_L"
+		(shape output)
+		(at -12.7 152.4 0)
+		(effects
+			(font
+				(size 1.27 1.27)
+			)
+			(justify left)
+		)
+	)
+	(hierarchical_label "SPICLK_T"
+		(shape output)
+		(at 233.68 81.28 0)
+		(effects
+			(font
+				(size 1.27 1.27)
+			)
+			(justify left)
+		)
+	)
+	(hierarchical_label "VL_SDA_0"
+		(shape bidirectional)
+		(at 50.8 186.69 0)
+		(effects
+			(font
+				(size 1.27 1.27)
+			)
+			(justify left)
+		)
+	)
+	(hierarchical_label "CSN_B"
+		(shape output)
+		(at 46.99 123.19 180)
 		(effects
 			(font
@@
 		)
 	)
-	(hierarchical_label "BMI_CS_R"
-		(shape bidirectional)
-		(at -29.21 162.56 0)
-		(effects
-			(font
-				(size 1.27 1.27)
-			)
-			(justify left)
-		)
-	)
-	(hierarchical_label "BMI_INT_L"
-		(shape output)
-		(at -12.7 152.4 0)
-		(effects
-			(font
-				(size 1.27 1.27)
-			)
-			(justify left)
-		)
-	)
-	(hierarchical_label "SPICLK_T"
-		(shape output)
-		(at 233.68 81.28 0)
-		(effects
-			(font
-				(size 1.27 1.27)
-			)
-			(justify left)
-		)
-	)
-	(hierarchical_label "VL_SDA_0"
-		(shape bidirectional)
-		(at 50.8 186.69 0)
-		(effects
-			(font
-				(size 1.27 1.27)
-			)
-			(justify left)
-		)
-	)
-	(hierarchical_label "CSN_B"
-		(shape output)
-		(at 46.99 123.19 180)
-		(effects
-			(font
-				(size 1.27 1.27)
-			)
-			(justify right)
-		)
-	)
-	(hierarchical_label "AMT_A_R"
-		(shape output)
-		(at 132.08 135.89 180)
-		(effects
-			(font
-				(size 1.27 1.27)
-			)
-			(justify right)
-		)
-	)
 	(hierarchical_label "VL_SCL_1"
 		(shape bidirectional)
@@
 		(shape bidirectional)
 		(at 50.8 184.15 0)
+		(effects
+			(font
+				(size 1.27 1.27)
+			)
+			(justify left)
+		)
+	)
+	(hierarchical_label "USART_TX"
+		(shape output)
+		(at 64.77 104.14 0)
 		(effects
 			(font
@@
 		)
 	)
-	(hierarchical_label "AMT_X_L"
-		(shape output)
-		(at 132.08 118.11 180)
-		(effects
-			(font
-				(size 1.27 1.27)
-			)
-			(justify right)
-		)
-	)
 	(hierarchical_label "DIR_L"
 		(shape output)
@@
 		(effects
 			(font
+				(size 1.27 1.27)
+			)
+			(justify left)
+		)
+	)
+	(hierarchical_label "USART_RX"
+		(shape input)
+		(at 64.77 106.68 0)
+		(effects
+			(font

Commit message: Add files via upload
Parts:
- removed J12: Conn_01x05_Socket, Connector_PinHeader_2.54mm:PinHeader_1x05_P2.54mm_Vertical, symbol Connector:Conn_01x05_Socket
- added J19: Conn_02x05_Odd_Even, symbol Connector_Generic:Conn_02x05_Odd_Even
- renumbered J11 to J10
Connections:
- net +3V3: now also J19.7 (Pin_7), J19.8 (Pin_8)
- net GNDREF: now also J19.5 (Pin_5), J19.6 (Pin_6)
- net NRESET: now also J19.1 (Pin_1)
- net SWCLK: now also J19.2 (Pin_2)
- net SWDIO: now also J19.4 (Pin_4)
- no-connect marks 3 -> 5
Other:
- moved on the sheet: J10

Commit message: Add files via upload
Parts:
- J19: footprint (none) -> Connector_PinSocket_2.54mm:PinSocket_2x05_P2.54mm_Vertical
Changed lines of the file:
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@@
 			)
 		)
-		(property "Footprint" ""
+		(property "Footprint" "Connector_PinSocket_2.54mm:PinSocket_2x05_P2.54mm_Vertical"
 			(at 255.27 102.87 0)
 			(hide yes)

Commit message: functionally finished driver board
Parts:
- SW1, SW2: footprint Button_Switch_THT:SW_PUSH_6mm -> MyFootprintLibrary:SW-SMD_L3.9-W3.0-P4.45
Changed lines of the file:
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@@
 			)
 		)
-		(property "Footprint" "Button_Switch_THT:SW_PUSH_6mm"
+		(property "Footprint" "MyFootprintLibrary:SW-SMD_L3.9-W3.0-P4.45"
 			(at 118.11 97.79 0)
 			(hide yes)
@@
 			)
 		)
-		(property "Footprint" "Button_Switch_THT:SW_PUSH_6mm"
+		(property "Footprint" "MyFootprintLibrary:SW-SMD_L3.9-W3.0-P4.45"
 			(at 135.89 85.09 0)
 			(hide yes)

Commit message: update
Connections:
- net GNDREF: now also U19.10 (VSS), U19.19 (VSSA), U19.26 (VSS), U19.49 (VSS), U19.74 (VSS), U19.99 (VSS)
- net DIR_L: no longer names the net of U19.95 (PB8)
- net STEP_L: no longer names the net of U19.96 (PB9)
