File: ELECTRONICS/MAINBOARD/STM32H743.kicad_sch (KiCad schematic)
At the start: 23 parts, among them J19 Conn_02x05_Odd_Even, SW1 RESET, SW2 BOOT, U19 STM32H743VITx, Y2 25mhz placeholder

Commit message: resize driver board to 60x55 mm^2, spread out bldc motor out pads
Parts:
- added J16: Conn_01x02_Pin, Connector_JST:JST_PH_S2B-PH-K_1x02_P2.00mm_Horizontal, symbol Connector:Conn_01x02_Pin
Connections:
- net BMI_CS_L: now also U19.41 (PE11)
- net BMI_CS_R: no longer U19.41 (PE11)
- net BMI_MISO_L: now also U19.43 (PE13)
- net BMI_MISO_R: no longer U19.43 (PE13)
- net BMI_MOSI_L: now also U19.44 (PE14)
- net BMI_MOSI_R: no longer U19.44 (PE14)
- net BMI_SCK_L: now also U19.42 (PE12)
- net BMI_SCK_R: no longer U19.42 (PE12)
- net USART_RX: now also U19.54 (PB15), J16.2 (Pin_2)
- net USART_TX: now also U19.53 (PB14), J16.1 (Pin_1)
Changed lines of the file:
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@@
 	(wire
 		(pts
+			(xy 247.65 168.91) (xy 261.62 168.91)
+		)
+		(stroke
+			(width 0)
+			(type default)
+		)
+	)
+	(wire
+		(pts
 			(xy 78.74 74.93) (xy 95.25 74.93)
 		)
@@
 	(wire
 		(pts
+			(xy 227.33 168.91) (xy 217.17 168.91)
+		)
+		(stroke
+			(width 0)
+			(type default)
+		)
+	)
+	(wire
+		(pts
 			(xy 196.85 50.8) (xy 201.93 50.8)
 		)
@@
 	(wire
 		(pts
-			(xy 224.79 151.13) (xy 217.17 151.13)
-		)
-		(stroke
-			(width 0)
-			(type default)
-		)
-	)
-	(wire
-		(pts
 			(xy 165.1 105.41) (xy 171.45 105.41)
 		)
@@
 	(wire
 		(pts
-			(xy 217.17 153.67) (xy 224.79 153.67)
-		)
-		(stroke
-			(width 0)
-			(type default)
-		)
-	)
-	(wire
-		(pts
 			(xy 165.1 92.71) (xy 171.45 92.71)
 		)
@@
 	(wire
 		(pts
+			(xy 227.33 166.37) (xy 217.17 166.37)
+		)
+		(stroke
+			(width 0)
+			(type default)
+		)
+	)
+	(wire
+		(pts
 			(xy 279.4 43.18) (xy 287.02 43.18)
 		)
@@
 	(wire
 		(pts
+			(xy 247.65 166.37) (xy 261.62 166.37)
+		)
+		(stroke
+			(width 0)
+			(type default)
+		)
+	)
+	(wire
+		(pts
 			(xy 317.5 52.07) (xy 317.5 50.8)
 		)
@@
 		)
 	)
+	(label "PB15"
+		(at 260.35 168.91 180)
+		(effects
+			(font
+				(size 1.27 1.27)
+			)
+			(justify right bottom)
+		)
+	)
 	(label "PH0"
 		(at 165.1 102.87 0)
@@
 		)
 	)
+	(label "PB14"
+		(at 260.35 166.37 180)
+		(effects
+			(font
+				(size 1.27 1.27)
+			)
+			(justify right bottom)
+		)
+	)
 	(label "SWDIO"
 		(at 224.79 120.65 180)
@@
 		)
 	)
+	(label "PB15"
+		(at 227.33 168.91 180)
+		(effects
+			(font
+				(size 1.27 1.27)
+			)
+			(justify right bottom)
+		)
+	)
 	(label "NRST"
 		(at 165.1 87.63 0)
@@
 		)
 	)
+	(label "PB14"
+		(at 227.33 166.37 180)
+		(effects
+			(font
+				(size 1.27 1.27)
+			)
+			(justify right bottom)
+		)
+	)
 	(hierarchical_label "VL_IO_1"
 		(shape bidirectional)
@@
 	(hierarchical_label "BMI_MOSI_L"
 		(shape output)
-		(at 119.38 151.13 0)
+		(at 171.45 146.05 180)
 		(effects
 			(font
 				(size 1.27 1.27)
 			)
-			(justify left)
+			(justify right)
 		)
 	)
@@
 	(hierarchical_label "BMI_SCK_R"
 		(shape bidirectional)
-		(at 171.45 140.97 180)
+		(at 119.38 153.67 0)
 		(effects
 			(font
 				(size 1.27 1.27)
 			)
-			(justify right)
+			(justify left)
 		)
 	)
@@
 	(hierarchical_label "BMI_SCK_L"
 		(shape bidirectional)
-		(at 119.38 153.67 0)
+		(at 171.45 140.97 180)
 		(effects
 			(font
 				(size 1.27 1.27)
 			)
-			(justify left)
+			(justify right)
 		)
 	)
@@
 	(hierarchical_label "BMI_MISO_R"
 		(shape input)
-		(at 171.45 143.51 180)
+		(at 119.38 160.02 0)
 		(effects
 			(font
 				(size 1.27 1.27)
 			)
-			(justify right)
+			(justify left)
 		)
 	)
 	(hierarchical_label "BMI_CS_R"
 		(shape bidirectional)
-		(at 171.45 138.43 180)
+		(at 119.38 156.21 0)
 		(effects
 			(font
 				(size 1.27 1.27)
 			)
-			(justify right)
+			(justify left)
 		)
 	)
@@
 	(hierarchical_label "USART_TX"
 		(shape output)
-		(at 92.71 120.65 0)
+		(at 261.62 166.37 0)
 		(effects
 			(font
@@
 	(hierarchical_label "BMI_MISO_L"
 		(shape input)
-		(at 119.38 160.02 0)
+		(at 171.45 143.51 180)
 		(effects
 			(font
 				(size 1.27 1.27)
 			)
-			(justify left)
+			(justify right)
 		)
 	)
 	(hierarchical_label "BMI_MOSI_R"
 		(shape output)
-		(at 171.45 146.05 180)
+		(at 119.38 151.13 0)
 		(effects
 			(font
 				(size 1.27 1.27)
 			)
-			(justify right)
+			(justify left)
 		)
 	)
@@
 	(hierarchical_label "BMI_CS_L"
 		(shape bidirectional)
-		(at 119.38 156.21 0)
+		(at 171.45 138.43 180)
 		(effects
 			(font
 				(size 1.27 1.27)
 			)
-			(justify left)
+			(justify right)
 		)
 	)
@@
 	(hierarchical_label "USART_RX"
 		(shape input)
-		(at 92.71 123.19 0)
+		(at 261.62 168.91 0)
 		(effects
 			(font
@@
 					(unit 1)
 				)
+			)
+		)
+	)
+	(symbol
+		(lib_id "Connector:Conn_01x02_Pin")
+		(at 242.57 166.37 0)
+		(unit 1)
+		(body_style 1)
+		(exclude_from_sim no)
+		(in_bom yes)
+		(on_board yes)
+		(in_pos_files yes)
+		(dnp no)
+		(fields_autoplaced yes)
+		(property "Reference" "J16"
+			(at 243.205 161.29 0)
+			(show_name no)
+			(do_not_autoplace no)
+			(effects
+				(font
+					(size 1.27 1.27)
+				)
+			)
+		)
+		(property "Value" "Conn_01x02_Pin"
+			(at 243.205 163.83 0)
+			(show_name no)
+			(do_not_autoplace no)
+			(effects
+				(font
+					(size 1.27 1.27)
+				)
+			)
+		)
+		(property "Footprint" "Connector_JST:JST_PH_S2B-PH-K_1x02_P2.00mm_Horizontal"
+			(at 242.57 166.37 0)
+			(hide yes)
+			(show_name no)
+			(do_not_autoplace no)
+			(effects
+				(font
+					(size 1.27 1.27)
+				)
+			)
+		)
+		(property "Datasheet" ""
+			(at 242.57 166.37 0)
+			(hide yes)
+			(show_name no)
+			(do_not_autoplace no)
+			(effects
+				(font
+					(size 1.27 1.27)
+				)
+			)
+		)
+		(property "Description" "Generic connector, single row, 01x02, script generated"
+			(at 242.57 166.37 0)
+			(hide yes)
+			(show_name no)
+			(do_not_autoplace no)
+			(effects
+				(font
+					(size 1.27 1.27)
+				)
+			)
+		)
+		(pin "2"
+		)
+		(pin "1"
+		)
+		(instances
+			(project "autobot_mainboard"
+				(path "/f053f1d0-b1f5-4f80-9758-8ee1a2d3659d/81f4ef01-6699-40d7-b94c-738d9569ae26"
+					(reference "J16")
+					(unit 1)
+				)

Commit message: rollback
Parts:
- renumbered C55 to C50, C56 to C51, C57 to C52, C58 to C53, C59 to C54, C60 to C55, C61 to C56, C62 to C57, C63 to C58, C64 to C59, C65 to C60, C66 to C61, C67 to C62, C68 to C63, C69 to C64, J16 to J13, J19 to J14, SW1 to SW2, SW2 to SW3, U19 to U11
