File: ELECTRONICS/MAINBOARD/autobot_mainboard.kicad_pcb (KiCad board)
At the start: 4 copper layers, 253 x 112 mm, 165 parts, among them IC1 DW3210, J1 USB_C_Receptacle_USB2.0_16P, J10 Conn_01x02_Pin, J11 Conn_01x01_Socket, J12 Conn_01x02_Pin, J13 Conn_01x01_Socket, J14 Conn_01x02_Pin, J15 Conn_01x02_Pin, J17 Conn_01x02_Pin, J18 Conn_01x02_Pin, J19 Conn_02x05_Odd_Even, J2 Conn_01x01_Socket, J20 Conn_02x05_Odd_Even, J3 Conn_01x01_Socket, J4 Conn_01x02_Socket, J5 Conn_01x01_Socket, J6 Conn_01x01_Socket, J7 Conn_01x03_Pin, J8 Conn_Coaxial, J9 Conn_Coaxial, Q1 DMG1012T, Q2 DMG1012T, Q3 DMG1012T, Q4 DMG1012T, Q5 DMG1012T, SW1 RESET, SW2 BOOT, SW3 SW_Push, U1 TVS1400DRV, U13 BMI270, U14 BMI270, U15 NCP1117-3.3_SOT223, U16 LP5907MFX-3.3, U18 LP5907MFX-3.3, U19 STM32H743VITx, U2 LMR51430XDDCR, U23 LP5907MFX-3.3, U4 TPD2EUSB30A, U7 STM32G031C_4-6-8_Tx, U9 VL53L1X, Y1 TXC 8Y38472012, Y2 25mhz placeholder

Commit message: resize driver board to 60x55 mm^2, spread out bldc motor out pads
Parts:
- added J16: Conn_01x02_Pin, Connector_JST:JST_PH_S2B-PH-K_1x02_P2.00mm_Horizontal, F.Cu at (256.8, 101.8)
- added REF**: MountingHole_3.2mm_M3_DIN965_Pad_TopBottom, MountingHole:MountingHole_3.2mm_M3_DIN965_Pad_TopBottom, F.Cu at (10.1, 61.7)
- added REF**: MountingHole_3.2mm_M3_DIN965_Pad_TopBottom, MountingHole:MountingHole_3.2mm_M3_DIN965_Pad_TopBottom, F.Cu at (10.1, 12.8)
- added REF**: MountingHole_3.2mm_M3_DIN965_Pad_TopBottom, MountingHole:MountingHole_3.2mm_M3_DIN965_Pad_TopBottom, F.Cu at (63.9, 12.8)
- added REF**: MountingHole_3.2mm_M3_DIN965_Pad_TopBottom, MountingHole:MountingHole_3.2mm_M3_DIN965_Pad_TopBottom, F.Cu at (63.9, 59.1)
- moved C2 40.0 mm to (290.3, 129.7)
- moved C4 40.0 mm to (296.9, 111.9)
- moved R1 40.0 mm to (293.7, 134.7)
- moved R2 40.0 mm to (292.0, 134.7)
- moved U1 40.0 mm to (285.2, 128.3)
- moved U2 40.0 mm to (293.8, 130.4)
- moved C1 40.0 mm to (288.8, 129.6)
- moved C3 40.0 mm to (297.5, 130.9)
- moved L1 40.0 mm to (293.9, 118.0)
- moved J17 8.30 mm to (56.6, 62.5)
- moved D13 8.20 mm to (30.1, 62.1)
- moved J4 8.20 mm to (17.9, 12.0)
- moved J18 8.20 mm to (38.0, 60.1)
- moved J20 8.12 mm to (27.0, 12.1)
- moved C88 6.34 mm to (10.3, 47.7)
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Connections:
- J20 pad 1: /STM32G0/NRESET -> /STM32G0/nRESET
- U19 pad 53: unconnected-(U19-PB14-Pad53) -> /STM32G0/USART_RX
- U19 pad 54: unconnected-(U19-PB15-Pad54) -> /STM32G0/USART_TX
Routing:
- net /STM32G0/nRESET: track 17.7 -> 46.6 mm
- net +24V: track 59.9 -> 71.0 mm
- net +5V: track 122.3 -> 133.2 mm
- net /STM32G0/USART_TX: track 30.2 -> 38.4 mm
- net /STM32G0/USART_RX: track 29.6 -> 37.8 mm
- net +3V3: track 128.0 -> 136.1 mm
- net /AMT102_L/AMT_X: track 36.6 -> 44.5 mm
- net /AMT102_L/AMT_A: track 28.9 -> 36.6 mm
- net /AMT102_L/AMT_B: track 30.9 -> 38.5 mm
- net /STM32G0/SWCLK: track 26.4 -> 33.7 mm
- net /STM32G0/SWDIO: track 24.8 -> 31.9 mm
- net /AMT102_R/AMT_A: track 24.7 -> 31.6 mm
- net Net-(C88-VIN): track 5.05 -> 11.8 mm
- net /AMT102_R/AMT_B: track 26.2 -> 33.0 mm
- net /AMT102_R/AMT_X: track 29.1 -> 35.8 mm
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Other:
- board size 253 x 112 mm -> 258 x 120.2 mm
