File: ELECTRONICS/MAINBOARD/LDO.kicad_sch (KiCad schematic)
At the start: 3 parts, among them U15 LP5907MFX-3.3

Commit message: Add files via upload
Parts:
- renumbered C22 to C5, C23 to C6, U15 to U3
Changed lines of the file:
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@@
 		(dnp no)
 		(fields_autoplaced yes)
-		(property "Reference" "#PWR040"
+		(property "Reference" "#PWR013"
 			(at 72.39 64.77 0)
 			(hide yes)
@@
 			(project "autobot_mainboard"
 				(path "/f053f1d0-b1f5-4f80-9758-8ee1a2d3659d/0fccf487-82ba-46aa-b4f9-fa30b5ecd66a"
-					(reference "#PWR048")
+					(reference "#PWR085")
 					(unit 1)
 				)
 				(path "/f053f1d0-b1f5-4f80-9758-8ee1a2d3659d/6f7d3baf-6e9d-45ae-a329-b78f8e18855d"
-					(reference "#PWR066")
+					(reference "#PWR051")
 					(unit 1)
 				)
 				(path "/f053f1d0-b1f5-4f80-9758-8ee1a2d3659d/d04181f1-3545-4903-8afb-41feb0a4a9a3"
-					(reference "#PWR040")
+					(reference "#PWR013")
 					(unit 1)
 				)
@@
 		(dnp no)
 		(fields_autoplaced yes)
-		(property "Reference" "#PWR043"
+		(property "Reference" "#PWR014"
 			(at 90.17 64.77 0)
 			(hide yes)
@@
 			(project "autobot_mainboard"
 				(path "/f053f1d0-b1f5-4f80-9758-8ee1a2d3659d/0fccf487-82ba-46aa-b4f9-fa30b5ecd66a"
-					(reference "#PWR050")
+					(reference "#PWR086")
 					(unit 1)
 				)
 				(path "/f053f1d0-b1f5-4f80-9758-8ee1a2d3659d/6f7d3baf-6e9d-45ae-a329-b78f8e18855d"
-					(reference "#PWR067")
+					(reference "#PWR052")
 					(unit 1)
 				)
 				(path "/f053f1d0-b1f5-4f80-9758-8ee1a2d3659d/d04181f1-3545-4903-8afb-41feb0a4a9a3"
-					(reference "#PWR043")
+					(reference "#PWR014")
 					(unit 1)
 				)
@@
 		(dnp no)
 		(fields_autoplaced yes)
-		(property "Reference" "#PWR044"
+		(property "Reference" "#PWR015"
 			(at 107.95 64.77 0)
 			(hide yes)
@@
 			(project "autobot_mainboard"
 				(path "/f053f1d0-b1f5-4f80-9758-8ee1a2d3659d/0fccf487-82ba-46aa-b4f9-fa30b5ecd66a"
-					(reference "#PWR051")
+					(reference "#PWR087")
 					(unit 1)
 				)
 				(path "/f053f1d0-b1f5-4f80-9758-8ee1a2d3659d/6f7d3baf-6e9d-45ae-a329-b78f8e18855d"
-					(reference "#PWR068")
+					(reference "#PWR053")
 					(unit 1)
 				)
 				(path "/f053f1d0-b1f5-4f80-9758-8ee1a2d3659d/d04181f1-3545-4903-8afb-41feb0a4a9a3"
-					(reference "#PWR044")
+					(reference "#PWR015")
 					(unit 1)
 				)
@@
 		(in_pos_files yes)
 		(dnp no)
-		(property "Reference" "C22"
+		(property "Reference" "C5"
 			(at 72.898 52.578 0)
 			(show_name no)
@@
 			(project "autobot_mainboard"
 				(path "/f053f1d0-b1f5-4f80-9758-8ee1a2d3659d/0fccf487-82ba-46aa-b4f9-fa30b5ecd66a"
-					(reference "C30")
+					(reference "C53")
 					(unit 1)
 				)
 				(path "/f053f1d0-b1f5-4f80-9758-8ee1a2d3659d/6f7d3baf-6e9d-45ae-a329-b78f8e18855d"
-					(reference "C38")
+					(reference "C34")
 					(unit 1)
 				)
 				(path "/f053f1d0-b1f5-4f80-9758-8ee1a2d3659d/d04181f1-3545-4903-8afb-41feb0a4a9a3"
-					(reference "C22")
+					(reference "C5")
 					(unit 1)
 				)
@@
 		(in_pos_files yes)
 		(dnp no)
-		(property "Reference" "C23"
+		(property "Reference" "C6"
 			(at 108.458 52.578 0)
 			(show_name no)
@@
 			(project "autobot_mainboard"
 				(path "/f053f1d0-b1f5-4f80-9758-8ee1a2d3659d/0fccf487-82ba-46aa-b4f9-fa30b5ecd66a"
-					(reference "C34")
+					(reference "C54")
 					(unit 1)
 				)
 				(path "/f053f1d0-b1f5-4f80-9758-8ee1a2d3659d/6f7d3baf-6e9d-45ae-a329-b78f8e18855d"
-					(reference "C39")
+					(reference "C35")
 					(unit 1)
 				)
 				(path "/f053f1d0-b1f5-4f80-9758-8ee1a2d3659d/d04181f1-3545-4903-8afb-41feb0a4a9a3"
-					(reference "C23")
+					(reference "C6")
 					(unit 1)
 				)
@@
 		(dnp no)
 		(fields_autoplaced yes)
-		(property "Reference" "U15"
+		(property "Reference" "U3"
 			(at 90.17 40.64 0)
 			(show_name no)
@@
 			(project "autobot_mainboard"
 				(path "/f053f1d0-b1f5-4f80-9758-8ee1a2d3659d/0fccf487-82ba-46aa-b4f9-fa30b5ecd66a"
-					(reference "U17")
+					(reference "U18")
 					(unit 1)
 				)
 				(path "/f053f1d0-b1f5-4f80-9758-8ee1a2d3659d/6f7d3baf-6e9d-45ae-a329-b78f8e18855d"
-					(reference "U19")
+					(reference "U16")
 					(unit 1)
 				)
 				(path "/f053f1d0-b1f5-4f80-9758-8ee1a2d3659d/d04181f1-3545-4903-8afb-41feb0a4a9a3"
-					(reference "U15")
-					(unit 1)
-				)
+					(reference "U3")
+					(unit 1)
+				)

Commit message: 10/24 save
Parts:
- renumbered C5 to C53, C6 to C54, U3 to U18
Changed lines of the file:
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@@
 		(dnp no)
 		(fields_autoplaced yes)
-		(property "Reference" "#PWR013"
+		(property "Reference" "#PWR084"
 			(at 72.39 64.77 0)
 			(hide yes)
@@
 				(path "/f053f1d0-b1f5-4f80-9758-8ee1a2d3659d/0fccf487-82ba-46aa-b4f9-fa30b5ecd66a"
 					(reference "#PWR084")
-					(unit 1)
-				)
-				(path "/f053f1d0-b1f5-4f80-9758-8ee1a2d3659d/6f7d3baf-6e9d-45ae-a329-b78f8e18855d"
-					(reference "#PWR051")
-					(unit 1)
-				)
-				(path "/f053f1d0-b1f5-4f80-9758-8ee1a2d3659d/d04181f1-3545-4903-8afb-41feb0a4a9a3"
-					(reference "#PWR013")
 					(unit 1)
 				)
@@
 		(dnp no)
 		(fields_autoplaced yes)
-		(property "Reference" "#PWR014"
+		(property "Reference" "#PWR085"
 			(at 90.17 64.77 0)
 			(hide yes)
@@
 				(path "/f053f1d0-b1f5-4f80-9758-8ee1a2d3659d/0fccf487-82ba-46aa-b4f9-fa30b5ecd66a"
 					(reference "#PWR085")
-					(unit 1)
-				)
-				(path "/f053f1d0-b1f5-4f80-9758-8ee1a2d3659d/6f7d3baf-6e9d-45ae-a329-b78f8e18855d"
-					(reference "#PWR052")
-					(unit 1)
-				)
-				(path "/f053f1d0-b1f5-4f80-9758-8ee1a2d3659d/d04181f1-3545-4903-8afb-41feb0a4a9a3"
-					(reference "#PWR014")
 					(unit 1)
 				)
@@
 		(dnp no)
 		(fields_autoplaced yes)
-		(property "Reference" "#PWR015"
+		(property "Reference" "#PWR086"
 			(at 107.95 64.77 0)
 			(hide yes)
@@
 				(path "/f053f1d0-b1f5-4f80-9758-8ee1a2d3659d/0fccf487-82ba-46aa-b4f9-fa30b5ecd66a"
 					(reference "#PWR086")
-					(unit 1)
-				)
-				(path "/f053f1d0-b1f5-4f80-9758-8ee1a2d3659d/6f7d3baf-6e9d-45ae-a329-b78f8e18855d"
-					(reference "#PWR053")
-					(unit 1)
-				)
-				(path "/f053f1d0-b1f5-4f80-9758-8ee1a2d3659d/d04181f1-3545-4903-8afb-41feb0a4a9a3"
-					(reference "#PWR015")
 					(unit 1)
 				)
@@
 		(in_pos_files yes)
 		(dnp no)
-		(property "Reference" "C5"
+		(property "Reference" "C53"
 			(at 72.898 52.578 0)
 			(show_name no)
@@
 				(path "/f053f1d0-b1f5-4f80-9758-8ee1a2d3659d/0fccf487-82ba-46aa-b4f9-fa30b5ecd66a"
 					(reference "C53")
-					(unit 1)
-				)
-				(path "/f053f1d0-b1f5-4f80-9758-8ee1a2d3659d/6f7d3baf-6e9d-45ae-a329-b78f8e18855d"
-					(reference "C34")
-					(unit 1)
-				)
-				(path "/f053f1d0-b1f5-4f80-9758-8ee1a2d3659d/d04181f1-3545-4903-8afb-41feb0a4a9a3"
-					(reference "C5")
 					(unit 1)
 				)
@@
 		(in_pos_files yes)
 		(dnp no)
-		(property "Reference" "C6"
+		(property "Reference" "C54"
 			(at 108.458 52.578 0)
 			(show_name no)
@@
 				(path "/f053f1d0-b1f5-4f80-9758-8ee1a2d3659d/0fccf487-82ba-46aa-b4f9-fa30b5ecd66a"
 					(reference "C54")
-					(unit 1)
-				)
-				(path "/f053f1d0-b1f5-4f80-9758-8ee1a2d3659d/6f7d3baf-6e9d-45ae-a329-b78f8e18855d"
-					(reference "C35")
-					(unit 1)
-				)
-				(path "/f053f1d0-b1f5-4f80-9758-8ee1a2d3659d/d04181f1-3545-4903-8afb-41feb0a4a9a3"
-					(reference "C6")
 					(unit 1)
 				)
@@
 		(dnp no)
 		(fields_autoplaced yes)
-		(property "Reference" "U3"
+		(property "Reference" "U18"
 			(at 90.17 40.64 0)
 			(show_name no)
@@
 					(unit 1)
 				)
-				(path "/f053f1d0-b1f5-4f80-9758-8ee1a2d3659d/6f7d3baf-6e9d-45ae-a329-b78f8e18855d"
-					(reference "U16")
-					(unit 1)
-				)
-				(path "/f053f1d0-b1f5-4f80-9758-8ee1a2d3659d/d04181f1-3545-4903-8afb-41feb0a4a9a3"
-					(reference "U3")
-					(unit 1)
-				)

Commit message: rollback
Parts:
- renumbered C53 to C48, C54 to C49, U18 to U10
Changed lines of the file:
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@@
 		(dnp no)
 		(fields_autoplaced yes)
-		(property "Reference" "#PWR084"
+		(property "Reference" "#PWR076"
 			(at 72.39 64.77 0)
 			(hide yes)
@@
 			(project "autobot_mainboard"
 				(path "/f053f1d0-b1f5-4f80-9758-8ee1a2d3659d/0fccf487-82ba-46aa-b4f9-fa30b5ecd66a"
-					(reference "#PWR084")
-					(unit 1)
-				)
-				(path "/f053f1d0-b1f5-4f80-9758-8ee1a2d3659d/f0fcce4b-6906-4d25-bb22-3fd6d8b4f8dc"
-					(reference "#PWR0153")
+					(reference "#PWR076")
+					(unit 1)
+				)
+				(path "/f053f1d0-b1f5-4f80-9758-8ee1a2d3659d/f0fcce4b-6906-4d25-bb22-3fd6d8b4f8dc"
+					(reference "#PWR0107")
 					(unit 1)
 				)
@@
 		(dnp no)
 		(fields_autoplaced yes)
-		(property "Reference" "#PWR085"
+		(property "Reference" "#PWR077"
 			(at 90.17 64.77 0)
 			(hide yes)
@@
 			(project "autobot_mainboard"
 				(path "/f053f1d0-b1f5-4f80-9758-8ee1a2d3659d/0fccf487-82ba-46aa-b4f9-fa30b5ecd66a"
-					(reference "#PWR085")
-					(unit 1)
-				)
-				(path "/f053f1d0-b1f5-4f80-9758-8ee1a2d3659d/f0fcce4b-6906-4d25-bb22-3fd6d8b4f8dc"
-					(reference "#PWR0154")
+					(reference "#PWR077")
+					(unit 1)
+				)
+				(path "/f053f1d0-b1f5-4f80-9758-8ee1a2d3659d/f0fcce4b-6906-4d25-bb22-3fd6d8b4f8dc"
+					(reference "#PWR0108")
 					(unit 1)
 				)
@@
 		(dnp no)
 		(fields_autoplaced yes)
-		(property "Reference" "#PWR086"
+		(property "Reference" "#PWR078"
 			(at 107.95 64.77 0)
 			(hide yes)
@@
 			(project "autobot_mainboard"
 				(path "/f053f1d0-b1f5-4f80-9758-8ee1a2d3659d/0fccf487-82ba-46aa-b4f9-fa30b5ecd66a"
-					(reference "#PWR086")
-					(unit 1)
-				)
-				(path "/f053f1d0-b1f5-4f80-9758-8ee1a2d3659d/f0fcce4b-6906-4d25-bb22-3fd6d8b4f8dc"
-					(reference "#PWR0155")
+					(reference "#PWR078")
+					(unit 1)
+				)
+				(path "/f053f1d0-b1f5-4f80-9758-8ee1a2d3659d/f0fcce4b-6906-4d25-bb22-3fd6d8b4f8dc"
+					(reference "#PWR0109")
 					(unit 1)
 				)
@@
 		(in_pos_files yes)
 		(dnp no)
-		(property "Reference" "C53"
+		(property "Reference" "C48"
 			(at 72.898 52.578 0)
 			(show_name no)
@@
 			(project "autobot_mainboard"
 				(path "/f053f1d0-b1f5-4f80-9758-8ee1a2d3659d/0fccf487-82ba-46aa-b4f9-fa30b5ecd66a"
-					(reference "C53")
-					(unit 1)
-				)
-				(path "/f053f1d0-b1f5-4f80-9758-8ee1a2d3659d/f0fcce4b-6906-4d25-bb22-3fd6d8b4f8dc"
-					(reference "C95")
+					(reference "C48")
+					(unit 1)
+				)
+				(path "/f053f1d0-b1f5-4f80-9758-8ee1a2d3659d/f0fcce4b-6906-4d25-bb22-3fd6d8b4f8dc"
+					(reference "C68")
 					(unit 1)
 				)
@@
 		(in_pos_files yes)
 		(dnp no)
-		(property "Reference" "C54"
+		(property "Reference" "C49"
 			(at 108.458 52.578 0)
 			(show_name no)
@@
 			(project "autobot_mainboard"
 				(path "/f053f1d0-b1f5-4f80-9758-8ee1a2d3659d/0fccf487-82ba-46aa-b4f9-fa30b5ecd66a"
-					(reference "C54")
-					(unit 1)
-				)
-				(path "/f053f1d0-b1f5-4f80-9758-8ee1a2d3659d/f0fcce4b-6906-4d25-bb22-3fd6d8b4f8dc"
-					(reference "C96")
+					(reference "C49")
+					(unit 1)
+				)
+				(path "/f053f1d0-b1f5-4f80-9758-8ee1a2d3659d/f0fcce4b-6906-4d25-bb22-3fd6d8b4f8dc"
+					(reference "C69")
 					(unit 1)
 				)
@@
 		(dnp no)
 		(fields_autoplaced yes)
-		(property "Reference" "U18"
+		(property "Reference" "U10"
 			(at 90.17 40.64 0)
 			(show_name no)
@@
 			(project "autobot_mainboard"
 				(path "/f053f1d0-b1f5-4f80-9758-8ee1a2d3659d/0fccf487-82ba-46aa-b4f9-fa30b5ecd66a"
-					(reference "U18")
-					(unit 1)
-				)
-				(path "/f053f1d0-b1f5-4f80-9758-8ee1a2d3659d/f0fcce4b-6906-4d25-bb22-3fd6d8b4f8dc"
-					(reference "U23")
-					(unit 1)
-				)
+					(reference "U10")
+					(unit 1)
+				)
+				(path "/f053f1d0-b1f5-4f80-9758-8ee1a2d3659d/f0fcce4b-6906-4d25-bb22-3fd6d8b4f8dc"
+					(reference "U12")
+					(unit 1)
+				)
