File: ELECTRONICS/MAINBOARD/MCT8316A1V.kicad_sch (KiCad schematic)
At the start: 17 parts, among them J11 Conn_01x01_Socket, J2 Conn_01x01_Socket, J5 Conn_01x01_Socket

Commit message: rollback
Parts:
- renumbered C11 to C10, C14 to C11, C13 to C12, C8 to C5, C7 to C6, C9 to C7, C10 to C8, C12 to C9, J5 to J3, J11 to J4, U5 to U4
