File: ELECTRONICS/MAINBOARD/POWER_CONNECTOR.kicad_sch (KiCad schematic)
At the start: 1 part, among them J5 Conn_01x03_Pin

Commit message: Add files via upload
Parts:
- removed J5: Conn_01x03_Pin, Connector_PinHeader_2.54mm:PinHeader_1x03_P2.54mm_Vertical, symbol Connector:Conn_01x03_Pin
- added J13: Conn_01x02_Pin, symbol Connector:Conn_01x02_Pin
Connections:
- net 12V: now also J13.1 (Pin_1)
- net GNDREF: now also J13.2 (Pin_2)
Changed lines of the file:
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@@
 	(wire
 		(pts
-			(xy 107.95 69.85) (xy 115.57 69.85)
+			(xy 116.84 55.88) (xy 109.22 55.88)
 		)
 		(stroke
@@
 	(wire
 		(pts
-			(xy 107.95 67.31) (xy 115.57 67.31)
+			(xy 109.22 53.34) (xy 116.84 53.34)
 		)
 		(stroke
@@
 		)
 	)
-	(wire
-		(pts
-			(xy 107.95 64.77) (xy 115.57 64.77)
-		)
-		(stroke
-			(width 0)
-			(type default)
-		)
-	)
-	(hierarchical_label "24V"
-		(shape output)
-		(at 115.57 67.31 0)
-		(effects
-			(font
-				(size 1.27 1.27)
-			)
-			(justify left)
-		)
-	)
 	(hierarchical_label "12V"
 		(shape output)
-		(at 115.57 64.77 0)
+		(at 116.84 53.34 0)
 		(effects
 			(font
@@
 	)
 	(symbol
-		(lib_id "Connector:Conn_01x03_Pin")
-		(at 102.87 67.31 0)
+		(lib_id "Connector:Conn_01x02_Pin")
+		(at 104.14 53.34 0)
 		(unit 1)
 		(body_style 1)
@@
 		(dnp no)
 		(fields_autoplaced yes)
-		(property "Reference" "J5"
-			(at 103.505 59.69 0)
+		(property "Reference" "J13"
+			(at 104.775 48.26 0)
 			(show_name no)
 			(do_not_autoplace no)
@@
 			)
 		)
-		(property "Value" "Conn_01x03_Pin"
-			(at 103.505 62.23 0)
+		(property "Value" "Conn_01x02_Pin"
+			(at 104.775 50.8 0)
 			(show_name no)
 			(do_not_autoplace no)
@@
 			)
 		)
-		(property "Footprint" "Connector_PinHeader_2.54mm:PinHeader_1x03_P2.54mm_Vertical"
-			(at 102.87 67.31 0)
+		(property "Footprint" ""
+			(at 104.14 53.34 0)
 			(hide yes)
 			(show_name no)
@@
 		)
 		(property "Datasheet" ""
-			(at 102.87 67.31 0)
+			(at 104.14 53.34 0)
 			(hide yes)
 			(show_name no)
@@
 			)
 		)
-		(property "Description" "Generic connector, single row, 01x03, script generated"
-			(at 102.87 67.31 0)
+		(property "Description" "Generic connector, single row, 01x02, script generated"
+			(at 104.14 53.34 0)
 			(hide yes)
 			(show_name no)
@@
 			)
 		)
+		(pin "2"
+		)
 		(pin "1"
-		)
-		(pin "3"
-		)
-		(pin "2"
 		)
 		(instances
 			(project "autobot_mainboard"
 				(path "/f053f1d0-b1f5-4f80-9758-8ee1a2d3659d/1c6d06e3-b0d2-4b47-a753-c45fb24fef2f"
-					(reference "J5")
+					(reference "J13")
 					(unit 1)
 				)
@@
 	(symbol
 		(lib_id "power:GNDREF")
-		(at 115.57 69.85 0)
+		(at 116.84 55.88 0)
 		(unit 1)
 		(body_style 1)
@@
 		(dnp no)
 		(fields_autoplaced yes)
-		(property "Reference" "#PWR0104"
-			(at 115.57 76.2 0)
+		(property "Reference" "#PWR0105"
+			(at 116.84 62.23 0)
 			(hide yes)
 			(show_name no)
@@
 		)
 		(property "Value" "GNDREF"
-			(at 115.57 74.93 0)
+			(at 116.84 60.96 0)
 			(hide yes)
 			(show_name no)
@@
 		)
 		(property "Footprint" ""
-			(at 115.57 69.85 0)
+			(at 116.84 55.88 0)
 			(hide yes)
 			(show_name no)
@@
 		)
 		(property "Datasheet" ""
-			(at 115.57 69.85 0)
+			(at 116.84 55.88 0)
 			(hide yes)
 			(show_name no)
@@
 		)
 		(property "Description" "Power symbol creates a global label with name \"GNDREF\" , reference supply ground"
-			(at 115.57 69.85 0)
+			(at 116.84 55.88 0)
 			(hide yes)
 			(show_name no)
@@
 			(project "autobot_mainboard"
 				(path "/f053f1d0-b1f5-4f80-9758-8ee1a2d3659d/1c6d06e3-b0d2-4b47-a753-c45fb24fef2f"
-					(reference "#PWR0104")
+					(reference "#PWR0105")
 					(unit 1)
 				)

Commit message: Add files via upload
Parts:
- renumbered J13 to J12
Changed lines of the file:
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@@
 		(dnp no)
 		(fields_autoplaced yes)
-		(property "Reference" "J13"
+		(property "Reference" "J12"
 			(at 104.775 48.26 0)
 			(show_name no)
@@
 			(project "autobot_mainboard"
 				(path "/f053f1d0-b1f5-4f80-9758-8ee1a2d3659d/1c6d06e3-b0d2-4b47-a753-c45fb24fef2f"
-					(reference "J13")
+					(reference "J12")
 					(unit 1)
 				)
@@
 		(dnp no)
 		(fields_autoplaced yes)
-		(property "Reference" "#PWR0105"
+		(property "Reference" "#PWR0104"
 			(at 116.84 62.23 0)
 			(hide yes)
@@
 			(project "autobot_mainboard"
 				(path "/f053f1d0-b1f5-4f80-9758-8ee1a2d3659d/1c6d06e3-b0d2-4b47-a753-c45fb24fef2f"
-					(reference "#PWR0105")
+					(reference "#PWR0104")
 					(unit 1)
 				)

Commit message: commit 1 commit 1 10/03/2026
Parts:
- J12: footprint (none) -> Connector_PinSocket_2.54mm:PinSocket_1x02_P2.54mm_Vertical
Changed lines of the file:
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@@
 			)
 		)
-		(property "Footprint" ""
+		(property "Footprint" "Connector_PinSocket_2.54mm:PinSocket_1x02_P2.54mm_Vertical"
 			(at 104.14 53.34 0)
 			(hide yes)

Commit message: rollback
Parts:
- renumbered J12 to J15
Changed lines of the file:
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@@
 		(dnp no)
 		(fields_autoplaced yes)
-		(property "Reference" "J12"
+		(property "Reference" "J15"
 			(at 104.775 48.26 0)
 			(show_name no)
@@
 			(project "autobot_mainboard"
 				(path "/f053f1d0-b1f5-4f80-9758-8ee1a2d3659d/1c6d06e3-b0d2-4b47-a753-c45fb24fef2f"
-					(reference "J12")
+					(reference "J15")
 					(unit 1)
 				)
@@
 		(dnp no)
 		(fields_autoplaced yes)
-		(property "Reference" "#PWR0104"
+		(property "Reference" "#PWR096"
 			(at 116.84 62.23 0)
 			(hide yes)
@@
 			(project "autobot_mainboard"
 				(path "/f053f1d0-b1f5-4f80-9758-8ee1a2d3659d/1c6d06e3-b0d2-4b47-a753-c45fb24fef2f"
-					(reference "#PWR0104")
+					(reference "#PWR096")
 					(unit 1)
 				)
