File: ELECTRONICS/MAINBOARD/Power.sch.kicad_sch (KiCad schematic)
At the start: 9 parts, among them U21 TVS1400DRV, U22 LMR51430XDDCR

Commit message: Add files via upload
Parts:
- renumbered C75 to C1, C76 to C2, C77 to C3, C78 to C4, L2 to L1, R18 to R1, R19 to R2, U21 to U1, U22 to U2
Changed lines of the file:
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@@
 		(dnp no)
 		(fields_autoplaced yes)
-		(property "Reference" "#PWR0114"
+		(property "Reference" "#PWR011"
 			(at 144.78 148.59 0)
 			(hide yes)
@@
 			(project "autobot_mainboard"
 				(path "/f053f1d0-b1f5-4f80-9758-8ee1a2d3659d/3bfa3ac1-569b-4dcd-933b-7ef1c6ac8888"
-					(reference "#PWR0114")
+					(reference "#PWR011")
 					(unit 1)
 				)
@@
 		(dnp no)
 		(fields_autoplaced yes)
-		(property "Reference" "C78"
+		(property "Reference" "C4"
 			(at 162.56 128.2699 0)
 			(show_name no)
@@
 			(project "autobot_mainboard"
 				(path "/f053f1d0-b1f5-4f80-9758-8ee1a2d3659d/3bfa3ac1-569b-4dcd-933b-7ef1c6ac8888"
-					(reference "C78")
+					(reference "C4")
 					(unit 1)
 				)
@@
 		(dnp no)
 		(fields_autoplaced yes)
-		(property "Reference" "#PWR0110"
+		(property "Reference" "#PWR07"
 			(at 53.34 119.38 0)
 			(hide yes)
@@
 			(project "autobot_mainboard"
 				(path "/f053f1d0-b1f5-4f80-9758-8ee1a2d3659d/3bfa3ac1-569b-4dcd-933b-7ef1c6ac8888"
-					(reference "#PWR0110")
+					(reference "#PWR07")
 					(unit 1)
 				)
@@
 		(dnp no)
 		(fields_autoplaced yes)
-		(property "Reference" "#PWR0113"
+		(property "Reference" "#PWR010"
 			(at 105.41 148.59 0)
 			(hide yes)
@@
 			(project "autobot_mainboard"
 				(path "/f053f1d0-b1f5-4f80-9758-8ee1a2d3659d/3bfa3ac1-569b-4dcd-933b-7ef1c6ac8888"
-					(reference "#PWR0113")
+					(reference "#PWR010")
 					(unit 1)
 				)
@@
 		(dnp no)
 		(fields_autoplaced yes)
-		(property "Reference" "R18"
+		(property "Reference" "R1"
 			(at 147.32 123.1899 0)
 			(show_name no)
@@
 			(project "autobot_mainboard"
 				(path "/f053f1d0-b1f5-4f80-9758-8ee1a2d3659d/3bfa3ac1-569b-4dcd-933b-7ef1c6ac8888"
-					(reference "R18")
+					(reference "R1")
 					(unit 1)
 				)
@@
 		(in_pos_files yes)
 		(dnp no)
-		(property "Reference" "C75"
+		(property "Reference" "C1"
 			(at 71.374 105.918 0)
 			(show_name no)
@@
 			(project "autobot_mainboard"
 				(path "/f053f1d0-b1f5-4f80-9758-8ee1a2d3659d/3bfa3ac1-569b-4dcd-933b-7ef1c6ac8888"
-					(reference "C75")
+					(reference "C1")
 					(unit 1)
 				)
@@
 		(dnp no)
 		(fields_autoplaced yes)
-		(property "Reference" "#PWR0112"
+		(property "Reference" "#PWR09"
 			(at 81.28 118.11 0)
 			(hide yes)
@@
 			(project "autobot_mainboard"
 				(path "/f053f1d0-b1f5-4f80-9758-8ee1a2d3659d/3bfa3ac1-569b-4dcd-933b-7ef1c6ac8888"
-					(reference "#PWR0112")
+					(reference "#PWR09")
 					(unit 1)
 				)
@@
 		(dnp no)
 		(fields_autoplaced yes)
-		(property "Reference" "U21"
+		(property "Reference" "U1"
 			(at 57.15 104.1399 0)
 			(show_name no)
@@
 			(project "autobot_mainboard"
 				(path "/f053f1d0-b1f5-4f80-9758-8ee1a2d3659d/3bfa3ac1-569b-4dcd-933b-7ef1c6ac8888"
-					(reference "U21")
+					(reference "U1")
 					(unit 1)
 				)
@@
 		(dnp no)
 		(fields_autoplaced yes)
-		(property "Reference" "C77"
+		(property "Reference" "C3"
 			(at 132.08 113.0299 0)
 			(show_name no)
@@
 			(project "autobot_mainboard"
 				(path "/f053f1d0-b1f5-4f80-9758-8ee1a2d3659d/3bfa3ac1-569b-4dcd-933b-7ef1c6ac8888"
-					(reference "C77")
+					(reference "C3")
 					(unit 1)
 				)
@@
 		(dnp no)
 		(fields_autoplaced yes)
-		(property "Reference" "#PWR0115"
+		(property "Reference" "#PWR012"
 			(at 158.75 148.59 0)
 			(hide yes)
@@
 			(project "autobot_mainboard"
 				(path "/f053f1d0-b1f5-4f80-9758-8ee1a2d3659d/3bfa3ac1-569b-4dcd-933b-7ef1c6ac8888"
-					(reference "#PWR0115")
+					(reference "#PWR012")
 					(unit 1)
 				)
@@
 		(dnp no)
 		(fields_autoplaced yes)
-		(property "Reference" "L2"
+		(property "Reference" "L1"
 			(at 140.97 114.3 90)
 			(show_name no)
@@
 			(project "autobot_mainboard"
 				(path "/f053f1d0-b1f5-4f80-9758-8ee1a2d3659d/3bfa3ac1-569b-4dcd-933b-7ef1c6ac8888"
-					(reference "L2")
+					(reference "L1")
 					(unit 1)
 				)
@@
 		(in_pos_files yes)
 		(dnp no)
-		(property "Reference" "C76"
+		(property "Reference" "C2"
 			(at 81.788 106.172 0)
 			(show_name no)
@@
 			(project "autobot_mainboard"
 				(path "/f053f1d0-b1f5-4f80-9758-8ee1a2d3659d/3bfa3ac1-569b-4dcd-933b-7ef1c6ac8888"
-					(reference "C76")
+					(reference "C2")
 					(unit 1)
 				)
@@
 		(dnp no)
 		(fields_autoplaced yes)
-		(property "Reference" "U22"
+		(property "Reference" "U2"
 			(at 107.5533 100.33 0)
 			(show_name no)
@@
 			(project "autobot_mainboard"
 				(path "/f053f1d0-b1f5-4f80-9758-8ee1a2d3659d/3bfa3ac1-569b-4dcd-933b-7ef1c6ac8888"
-					(reference "U22")
+					(reference "U2")
 					(unit 1)
 				)
@@
 		(dnp no)
 		(fields_autoplaced yes)
-		(property "Reference" "R19"
+		(property "Reference" "R2"
 			(at 147.32 133.3499 0)
 			(show_name no)
@@
 			(project "autobot_mainboard"
 				(path "/f053f1d0-b1f5-4f80-9758-8ee1a2d3659d/3bfa3ac1-569b-4dcd-933b-7ef1c6ac8888"
-					(reference "R19")
+					(reference "R2")
 					(unit 1)
 				)
@@
 		(dnp no)
 		(fields_autoplaced yes)
-		(property "Reference" "#PWR0111"
+		(property "Reference" "#PWR08"
 			(at 71.12 118.11 0)
 			(hide yes)
@@
 			(project "autobot_mainboard"
 				(path "/f053f1d0-b1f5-4f80-9758-8ee1a2d3659d/3bfa3ac1-569b-4dcd-933b-7ef1c6ac8888"
-					(reference "#PWR0111")
-					(unit 1)
-				)
+					(reference "#PWR08")
+					(unit 1)
+				)
