File: ELECTRONICS/MAINBOARD/Power_connector_g0.kicad_sch (KiCad schematic)
At the start: 2 parts, among them J18 Conn_01x02_Pin, J19 Conn_01x02_Pin

Commit message: Add files via upload
Parts:
- J17: renamed from J18; footprint (none) -> Connector_AMASS:AMASS_XT60-F_1x02_P7.20mm_Vertical
- J18: renamed from J19; footprint (none) -> Connector_AMASS:AMASS_XT60-F_1x02_P7.20mm_Vertical
Changed lines of the file:
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@@
 		(dnp no)
 		(fields_autoplaced yes)
-		(property "Reference" "J18"
+		(property "Reference" "J17"
 			(at 59.055 46.99 0)
 			(show_name no)
@@
 			)
 		)
-		(property "Footprint" ""
+		(property "Footprint" "Connector_AMASS:AMASS_XT60-F_1x02_P7.20mm_Vertical"
 			(at 58.42 52.07 0)
 			(hide yes)
@@
 			(project "autobot_mainboard"
 				(path "/f053f1d0-b1f5-4f80-9758-8ee1a2d3659d/333584c5-5177-4b5f-b371-6c9cddbf8d2e"
-					(reference "J18")
+					(reference "J17")
 					(unit 1)
 				)
@@
 		(dnp no)
 		(fields_autoplaced yes)
-		(property "Reference" "#PWR0152"
+		(property "Reference" "#PWR0151"
 			(at 71.12 60.96 0)
 			(hide yes)
@@
 			(project "autobot_mainboard"
 				(path "/f053f1d0-b1f5-4f80-9758-8ee1a2d3659d/333584c5-5177-4b5f-b371-6c9cddbf8d2e"
-					(reference "#PWR0152")
+					(reference "#PWR0151")
 					(unit 1)
 				)
@@
 		(dnp no)
 		(fields_autoplaced yes)
-		(property "Reference" "J19"
+		(property "Reference" "J18"
 			(at 59.055 57.15 0)
 			(show_name no)
@@
 			)
 		)
-		(property "Footprint" ""
+		(property "Footprint" "Connector_AMASS:AMASS_XT60-F_1x02_P7.20mm_Vertical"
 			(at 58.42 62.23 0)
 			(hide yes)
@@
 			(project "autobot_mainboard"
 				(path "/f053f1d0-b1f5-4f80-9758-8ee1a2d3659d/333584c5-5177-4b5f-b371-6c9cddbf8d2e"
-					(reference "J19")
+					(reference "J18")
 					(unit 1)
 				)
@@
 		(dnp no)
 		(fields_autoplaced yes)
-		(property "Reference" "#PWR0153"
+		(property "Reference" "#PWR0152"
 			(at 71.12 71.12 0)
 			(hide yes)
@@
 			(project "autobot_mainboard"
 				(path "/f053f1d0-b1f5-4f80-9758-8ee1a2d3659d/333584c5-5177-4b5f-b371-6c9cddbf8d2e"
-					(reference "#PWR0153")
-					(unit 1)
-				)
+					(reference "#PWR0152")
+					(unit 1)
+				)

Commit message: commit 1 commit 1 10/03/2026
Parts:
- J17: footprint Connector_AMASS:AMASS_XT60-F_1x02_P7.20mm_Vertical -> Connector_PinHeader_2.54mm:PinHeader_1x02_P2.54mm_Vertical
Changed lines of the file:
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@@
 			)
 		)
-		(property "Footprint" "Connector_AMASS:AMASS_XT60-F_1x02_P7.20mm_Vertical"
+		(property "Footprint" "Connector_PinHeader_2.54mm:PinHeader_1x02_P2.54mm_Vertical"
 			(at 58.42 52.07 0)
 			(hide yes)

Commit message: almost done
Parts:
- J17: footprint Connector_PinHeader_2.54mm:PinHeader_1x02_P2.54mm_Vertical -> Connector_JST:JST_PH_B2B-PH-K_1x02_P2.00mm_Vertical
Changed lines of the file:
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@@
 			)
 		)
-		(property "Footprint" "Connector_PinHeader_2.54mm:PinHeader_1x02_P2.54mm_Vertical"
+		(property "Footprint" "Connector_JST:JST_PH_B2B-PH-K_1x02_P2.00mm_Vertical"
 			(at 58.42 52.07 0)
 			(hide yes)

Commit message: rollback
Parts:
- renumbered J17 to J16, J18 to J17
Changed lines of the file:
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@@
 		(dnp no)
 		(fields_autoplaced yes)
-		(property "Reference" "J17"
+		(property "Reference" "J16"
 			(at 59.055 46.99 0)
 			(show_name no)
@@
 			(project "autobot_mainboard"
 				(path "/f053f1d0-b1f5-4f80-9758-8ee1a2d3659d/333584c5-5177-4b5f-b371-6c9cddbf8d2e"
-					(reference "J17")
+					(reference "J16")
 					(unit 1)
 				)
@@
 		(dnp no)
 		(fields_autoplaced yes)
-		(property "Reference" "#PWR0151"
+		(property "Reference" "#PWR0105"
 			(at 71.12 60.96 0)
 			(hide yes)
@@
 			(project "autobot_mainboard"
 				(path "/f053f1d0-b1f5-4f80-9758-8ee1a2d3659d/333584c5-5177-4b5f-b371-6c9cddbf8d2e"
-					(reference "#PWR0151")
+					(reference "#PWR0105")
 					(unit 1)
 				)
@@
 		(dnp no)
 		(fields_autoplaced yes)
-		(property "Reference" "J18"
+		(property "Reference" "J17"
 			(at 59.055 57.15 0)
 			(show_name no)
@@
 			(project "autobot_mainboard"
 				(path "/f053f1d0-b1f5-4f80-9758-8ee1a2d3659d/333584c5-5177-4b5f-b371-6c9cddbf8d2e"
-					(reference "J18")
+					(reference "J17")
 					(unit 1)
 				)
@@
 		(dnp no)
 		(fields_autoplaced yes)
-		(property "Reference" "#PWR0152"
+		(property "Reference" "#PWR0106"
 			(at 71.12 71.12 0)
 			(hide yes)
@@
 			(project "autobot_mainboard"
 				(path "/f053f1d0-b1f5-4f80-9758-8ee1a2d3659d/333584c5-5177-4b5f-b371-6c9cddbf8d2e"
-					(reference "#PWR0152")
-					(unit 1)
-				)
+					(reference "#PWR0106")
+					(unit 1)
+				)
