File: ELECTRONICS/MAINBOARD/USB.kicad_sch (KiCad schematic)
At the start: 7 parts, among them J2 USB_C_Receptacle_USB2.0_16P, U5 TPD2EUSB30A

Commit message: Add files via upload
Parts:
- renumbered J2 to J1, R1 to R3, R2 to R4, R3 to R5, R4 to R6, U5 to U4
Changed lines of the file:
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@@
 		(dnp no)
 		(fields_autoplaced yes)
-		(property "Reference" "#PWR013"
+		(property "Reference" "#PWR018"
 			(at 106.68 80.01 0)
 			(hide yes)
@@
 			(project "autobot_mainboard"
 				(path "/f053f1d0-b1f5-4f80-9758-8ee1a2d3659d/784d5709-397e-4ddf-a25c-7a5778089f9e"
-					(reference "#PWR013")
+					(reference "#PWR018")
 					(unit 1)
 				)
@@
 		(dnp no)
 		(fields_autoplaced yes)
-		(property "Reference" "#PWR021"
+		(property "Reference" "#PWR020"
 			(at 143.51 78.74 0)
 			(hide yes)
@@
 			(project "autobot_mainboard"
 				(path "/f053f1d0-b1f5-4f80-9758-8ee1a2d3659d/784d5709-397e-4ddf-a25c-7a5778089f9e"
-					(reference "#PWR021")
+					(reference "#PWR020")
 					(unit 1)
 				)
@@
 		(in_pos_files yes)
 		(dnp no)
-		(property "Reference" "R3"
+		(property "Reference" "R5"
 			(at 140.716 60.198 90)
 			(show_name no)
@@
 			(project "autobot_mainboard"
 				(path "/f053f1d0-b1f5-4f80-9758-8ee1a2d3659d/784d5709-397e-4ddf-a25c-7a5778089f9e"
-					(reference "R3")
+					(reference "R5")
 					(unit 1)
 				)
@@
 		(dnp no)
 		(fields_autoplaced yes)
-		(property "Reference" "J2"
+		(property "Reference" "J1"
 			(at 76.2 41.91 0)
 			(show_name no)
@@
 			(project "autobot_mainboard"
 				(path "/f053f1d0-b1f5-4f80-9758-8ee1a2d3659d/784d5709-397e-4ddf-a25c-7a5778089f9e"
-					(reference "J2")
+					(reference "J1")
 					(unit 1)
 				)
@@
 		(dnp no)
 		(fields_autoplaced yes)
-		(property "Reference" "#PWR03"
+		(property "Reference" "#PWR017"
 			(at 76.2 93.98 0)
 			(hide yes)
@@
 			(project "autobot_mainboard"
 				(path "/f053f1d0-b1f5-4f80-9758-8ee1a2d3659d/784d5709-397e-4ddf-a25c-7a5778089f9e"
-					(reference "#PWR03")
+					(reference "#PWR017")
 					(unit 1)
 				)
@@
 		(in_pos_files yes)
 		(dnp no)
-		(property "Reference" "R1"
+		(property "Reference" "R3"
 			(at 104.648 69.85 90)
 			(show_name no)
@@
 			(project "autobot_mainboard"
 				(path "/f053f1d0-b1f5-4f80-9758-8ee1a2d3659d/784d5709-397e-4ddf-a25c-7a5778089f9e"
-					(reference "R1")
+					(reference "R3")
 					(unit 1)
 				)
@@
 		(in_pos_files yes)
 		(dnp no)
-		(property "Reference" "U5"
+		(property "Reference" "U4"
 			(at 123.19 71.1199 90)
 			(show_name no)
@@
 			(project "autobot_mainboard"
 				(path "/f053f1d0-b1f5-4f80-9758-8ee1a2d3659d/784d5709-397e-4ddf-a25c-7a5778089f9e"
-					(reference "U5")
+					(reference "U4")
 					(unit 1)
 				)
@@
 		(dnp no)
 		(fields_autoplaced yes)
-		(property "Reference" "#PWR014"
+		(property "Reference" "#PWR019"
 			(at 110.49 72.39 0)
 			(hide yes)
@@
 			(project "autobot_mainboard"
 				(path "/f053f1d0-b1f5-4f80-9758-8ee1a2d3659d/784d5709-397e-4ddf-a25c-7a5778089f9e"
-					(reference "#PWR014")
+					(reference "#PWR019")
 					(unit 1)
 				)
@@
 		(in_pos_files yes)
 		(dnp no)
-		(property "Reference" "R2"
+		(property "Reference" "R4"
 			(at 108.458 62.23 90)
 			(show_name no)
@@
 			(project "autobot_mainboard"
 				(path "/f053f1d0-b1f5-4f80-9758-8ee1a2d3659d/784d5709-397e-4ddf-a25c-7a5778089f9e"
-					(reference "R2")
+					(reference "R4")
 					(unit 1)
 				)
@@
 		(in_pos_files yes)
 		(dnp no)
-		(property "Reference" "R4"
+		(property "Reference" "R6"
 			(at 140.716 80.518 90)
 			(show_name no)
@@
 			(project "autobot_mainboard"
 				(path "/f053f1d0-b1f5-4f80-9758-8ee1a2d3659d/784d5709-397e-4ddf-a25c-7a5778089f9e"
-					(reference "R4")
+					(reference "R6")
 					(unit 1)
 				)
@@
 		(dnp no)
 		(fields_autoplaced yes)
-		(property "Reference" "#PWR01"
+		(property "Reference" "#PWR016"
 			(at 68.58 93.98 0)
 			(hide yes)
@@
 			(project "autobot_mainboard"
 				(path "/f053f1d0-b1f5-4f80-9758-8ee1a2d3659d/784d5709-397e-4ddf-a25c-7a5778089f9e"
-					(reference "#PWR01")
-					(unit 1)
-				)
+					(reference "#PWR016")
+					(unit 1)
+				)

Commit message: power zone
Connections:
- net D+: now also R5.2; no longer R6.2
- net D-: now also R6.2; no longer R5.2
Changed lines of the file:
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@@
 	(hierarchical_label "D+"
 		(shape output)
-		(at 147.32 82.55 0)
+		(at 147.32 62.23 0)
 		(effects
 			(font
@@
 	(hierarchical_label "D-"
 		(shape output)
-		(at 147.32 62.23 0)
+		(at 147.32 82.55 0)
 		(effects
 			(font

Commit message: rollback
Parts:
- renumbered U4 to U3
Changed lines of the file:
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@@
 		(dnp no)
 		(fields_autoplaced yes)
-		(property "Reference" "#PWR018"
+		(property "Reference" "#PWR013"
 			(at 106.68 80.01 0)
 			(hide yes)
@@
 			(project "autobot_mainboard"
 				(path "/f053f1d0-b1f5-4f80-9758-8ee1a2d3659d/784d5709-397e-4ddf-a25c-7a5778089f9e"
-					(reference "#PWR018")
+					(reference "#PWR013")
 					(unit 1)
 				)
@@
 		(dnp no)
 		(fields_autoplaced yes)
-		(property "Reference" "#PWR020"
+		(property "Reference" "#PWR015"
 			(at 143.51 78.74 0)
 			(hide yes)
@@
 			(project "autobot_mainboard"
 				(path "/f053f1d0-b1f5-4f80-9758-8ee1a2d3659d/784d5709-397e-4ddf-a25c-7a5778089f9e"
-					(reference "#PWR020")
+					(reference "#PWR015")
 					(unit 1)
 				)
@@
 		(dnp no)
 		(fields_autoplaced yes)
-		(property "Reference" "#PWR017"
+		(property "Reference" "#PWR012"
 			(at 76.2 93.98 0)
 			(hide yes)
@@
 			(project "autobot_mainboard"
 				(path "/f053f1d0-b1f5-4f80-9758-8ee1a2d3659d/784d5709-397e-4ddf-a25c-7a5778089f9e"
-					(reference "#PWR017")
+					(reference "#PWR012")
 					(unit 1)
 				)
@@
 		(in_pos_files yes)
 		(dnp no)
-		(property "Reference" "U4"
+		(property "Reference" "U3"
 			(at 123.19 71.1199 90)
 			(show_name no)
@@
 			(project "autobot_mainboard"
 				(path "/f053f1d0-b1f5-4f80-9758-8ee1a2d3659d/784d5709-397e-4ddf-a25c-7a5778089f9e"
-					(reference "U4")
+					(reference "U3")
 					(unit 1)
 				)
@@
 		(dnp no)
 		(fields_autoplaced yes)
-		(property "Reference" "#PWR019"
+		(property "Reference" "#PWR014"
 			(at 110.49 72.39 0)
 			(hide yes)
@@
 			(project "autobot_mainboard"
 				(path "/f053f1d0-b1f5-4f80-9758-8ee1a2d3659d/784d5709-397e-4ddf-a25c-7a5778089f9e"
-					(reference "#PWR019")
+					(reference "#PWR014")
 					(unit 1)
 				)
@@
 		(dnp no)
 		(fields_autoplaced yes)
-		(property "Reference" "#PWR016"
+		(property "Reference" "#PWR011"
 			(at 68.58 93.98 0)
 			(hide yes)
@@
 			(project "autobot_mainboard"
 				(path "/f053f1d0-b1f5-4f80-9758-8ee1a2d3659d/784d5709-397e-4ddf-a25c-7a5778089f9e"
-					(reference "#PWR016")
-					(unit 1)
-				)
+					(reference "#PWR011")
+					(unit 1)
+				)
