File: ELECTRONICS/MAINBOARD/VL53L1X.kicad_sch (KiCad schematic)
At the start: 3 parts, among them U1 VL53L1X

Commit message: Add files via upload
Parts:
- renumbered C1 to C19, C52 to C20, U1 to U9
Changed lines of the file:
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@@
 		(dnp no)
 		(fields_autoplaced yes)
-		(property "Reference" "#PWR011"
+		(property "Reference" "#PWR032"
 			(at 114.3 93.98 0)
 			(hide yes)
@@
 			(project "autobot_mainboard"
 				(path "/f053f1d0-b1f5-4f80-9758-8ee1a2d3659d/037a1145-d2fa-427f-912d-11744b2ed89a"
-					(reference "#PWR036")
+					(reference "#PWR035")
 					(unit 1)
 				)
 				(path "/f053f1d0-b1f5-4f80-9758-8ee1a2d3659d/18a50009-3afb-45d9-96a2-f4fbe8f24a2b"
-					(reference "#PWR011")
+					(reference "#PWR032")
 					(unit 1)
 				)
 				(path "/f053f1d0-b1f5-4f80-9758-8ee1a2d3659d/bbe9edfa-2cce-4350-82ca-a6538778d251"
-					(reference "#PWR059")
+					(reference "#PWR041")
 					(unit 1)
 				)
 				(path "/f053f1d0-b1f5-4f80-9758-8ee1a2d3659d/ea0baaba-f154-47d1-ba71-cf9d27cdfb48"
-					(reference "#PWR058")
+					(reference "#PWR038")
 					(unit 1)
 				)
@@
 		(dnp no)
 		(fields_autoplaced yes)
-		(property "Reference" "#PWR05"
+		(property "Reference" "#PWR031"
 			(at 88.9 105.41 0)
 			(hide yes)
@@
 			(project "autobot_mainboard"
 				(path "/f053f1d0-b1f5-4f80-9758-8ee1a2d3659d/037a1145-d2fa-427f-912d-11744b2ed89a"
-					(reference "#PWR06")
+					(reference "#PWR034")
 					(unit 1)
 				)
 				(path "/f053f1d0-b1f5-4f80-9758-8ee1a2d3659d/18a50009-3afb-45d9-96a2-f4fbe8f24a2b"
-					(reference "#PWR05")
+					(reference "#PWR031")
 					(unit 1)
 				)
 				(path "/f053f1d0-b1f5-4f80-9758-8ee1a2d3659d/bbe9edfa-2cce-4350-82ca-a6538778d251"
-					(reference "#PWR010")
+					(reference "#PWR040")
 					(unit 1)
 				)
 				(path "/f053f1d0-b1f5-4f80-9758-8ee1a2d3659d/ea0baaba-f154-47d1-ba71-cf9d27cdfb48"
-					(reference "#PWR07")
+					(reference "#PWR037")
 					(unit 1)
 				)
@@
 		(in_pos_files yes)
 		(dnp no)
-		(property "Reference" "U1"
+		(property "Reference" "U9"
 			(at 82.55 83.8199 0)
 			(show_name no)
@@
 			(project "autobot_mainboard"
 				(path "/f053f1d0-b1f5-4f80-9758-8ee1a2d3659d/037a1145-d2fa-427f-912d-11744b2ed89a"
-					(reference "U2")
+					(reference "U10")
 					(unit 1)
 				)
 				(path "/f053f1d0-b1f5-4f80-9758-8ee1a2d3659d/18a50009-3afb-45d9-96a2-f4fbe8f24a2b"
-					(reference "U1")
+					(reference "U9")
 					(unit 1)
 				)
 				(path "/f053f1d0-b1f5-4f80-9758-8ee1a2d3659d/bbe9edfa-2cce-4350-82ca-a6538778d251"
-					(reference "U7")
+					(reference "U12")
 					(unit 1)
 				)
 				(path "/f053f1d0-b1f5-4f80-9758-8ee1a2d3659d/ea0baaba-f154-47d1-ba71-cf9d27cdfb48"
-					(reference "U6")
+					(reference "U11")
 					(unit 1)
 				)
@@
 		(dnp no)
 		(fields_autoplaced yes)
-		(property "Reference" "#PWR087"
+		(property "Reference" "#PWR033"
 			(at 121.92 93.98 0)
 			(hide yes)
@@
 			(project "autobot_mainboard"
 				(path "/f053f1d0-b1f5-4f80-9758-8ee1a2d3659d/037a1145-d2fa-427f-912d-11744b2ed89a"
-					(reference "#PWR088")
+					(reference "#PWR036")
 					(unit 1)
 				)
 				(path "/f053f1d0-b1f5-4f80-9758-8ee1a2d3659d/18a50009-3afb-45d9-96a2-f4fbe8f24a2b"
-					(reference "#PWR087")
+					(reference "#PWR033")
 					(unit 1)
 				)
 				(path "/f053f1d0-b1f5-4f80-9758-8ee1a2d3659d/bbe9edfa-2cce-4350-82ca-a6538778d251"
-					(reference "#PWR090")
+					(reference "#PWR042")
 					(unit 1)
 				)
 				(path "/f053f1d0-b1f5-4f80-9758-8ee1a2d3659d/ea0baaba-f154-47d1-ba71-cf9d27cdfb48"
-					(reference "#PWR089")
+					(reference "#PWR039")
 					(unit 1)
 				)
@@
 		(in_pos_files yes)
 		(dnp no)
-		(property "Reference" "C52"
+		(property "Reference" "C20"
 			(at 122.428 82.042 0)
 			(show_name no)
@@
 			(project "autobot_mainboard"
 				(path "/f053f1d0-b1f5-4f80-9758-8ee1a2d3659d/037a1145-d2fa-427f-912d-11744b2ed89a"
-					(reference "C54")
+					(reference "C22")
 					(unit 1)
 				)
 				(path "/f053f1d0-b1f5-4f80-9758-8ee1a2d3659d/18a50009-3afb-45d9-96a2-f4fbe8f24a2b"
-					(reference "C52")
+					(reference "C20")
 					(unit 1)
 				)
 				(path "/f053f1d0-b1f5-4f80-9758-8ee1a2d3659d/bbe9edfa-2cce-4350-82ca-a6538778d251"
-					(reference "C56")
+					(reference "C26")
 					(unit 1)
 				)
 				(path "/f053f1d0-b1f5-4f80-9758-8ee1a2d3659d/ea0baaba-f154-47d1-ba71-cf9d27cdfb48"
-					(reference "C55")
+					(reference "C24")
 					(unit 1)
 				)
@@
 		(in_pos_files yes)
 		(dnp no)
-		(property "Reference" "C1"
+		(property "Reference" "C19"
 			(at 114.554 82.042 0)
 			(show_name no)
@@
 			(project "autobot_mainboard"
 				(path "/f053f1d0-b1f5-4f80-9758-8ee1a2d3659d/037a1145-d2fa-427f-912d-11744b2ed89a"
-					(reference "C10")
+					(reference "C21")
 					(unit 1)
 				)
 				(path "/f053f1d0-b1f5-4f80-9758-8ee1a2d3659d/18a50009-3afb-45d9-96a2-f4fbe8f24a2b"
-					(reference "C1")
+					(reference "C19")
 					(unit 1)
 				)
 				(path "/f053f1d0-b1f5-4f80-9758-8ee1a2d3659d/bbe9edfa-2cce-4350-82ca-a6538778d251"
-					(reference "C37")
+					(reference "C25")
 					(unit 1)
 				)
 				(path "/f053f1d0-b1f5-4f80-9758-8ee1a2d3659d/ea0baaba-f154-47d1-ba71-cf9d27cdfb48"
-					(reference "C15")
-					(unit 1)
-				)
+					(reference "C23")
+					(unit 1)
+				)

Commit message: change ToF module connection to use just one bus
Connections:
- net VL_IO: no longer names the net of U9.5 (GPIO)
- net VL_XSHUT: no longer names the net of U9.6 (XSHUT)
- no-connect marks 0 -> 2
Changed lines of the file:
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@@
 		(color 0 0 0 0)
 	)
+	(no_connect
+		(at 96.52 82.55)
+	)
+	(no_connect
+		(at 96.52 85.09)
+	)
 	(wire
 		(pts
@@
 	(wire
 		(pts
-			(xy 96.52 85.09) (xy 99.06 85.09)
-		)
-		(stroke
-			(width 0)
-			(type default)
-		)
-	)
-	(wire
-		(pts
 			(xy 114.3 68.58) (xy 114.3 80.01)
-		)
-		(stroke
-			(width 0)
-			(type default)
-		)
-	)
-	(wire
-		(pts
-			(xy 96.52 82.55) (xy 99.06 82.55)
 		)
 		(stroke
@@
 		(shape bidirectional)
 		(at 99.06 77.47 0)
-		(effects
-			(font
-				(size 1.27 1.27)
-			)
-			(justify left)
-		)
-	)
-	(hierarchical_label "VL_XSHUT"
-		(shape input)
-		(at 99.06 85.09 0)
-		(effects
-			(font
-				(size 1.27 1.27)
-			)
-			(justify left)
-		)
-	)
-	(hierarchical_label "VL_IO"
-		(shape bidirectional)
-		(at 99.06 82.55 0)
 		(effects
 			(font
@@
 		(instances
 			(project "autobot_mainboard"
-				(path "/f053f1d0-b1f5-4f80-9758-8ee1a2d3659d/037a1145-d2fa-427f-912d-11744b2ed89a"
-					(reference "#PWR035")
-					(unit 1)
-				)
 				(path "/f053f1d0-b1f5-4f80-9758-8ee1a2d3659d/18a50009-3afb-45d9-96a2-f4fbe8f24a2b"
 					(reference "#PWR032")
-					(unit 1)
-				)
-				(path "/f053f1d0-b1f5-4f80-9758-8ee1a2d3659d/bbe9edfa-2cce-4350-82ca-a6538778d251"
-					(reference "#PWR041")
-					(unit 1)
-				)
-				(path "/f053f1d0-b1f5-4f80-9758-8ee1a2d3659d/ea0baaba-f154-47d1-ba71-cf9d27cdfb48"
-					(reference "#PWR038")
 					(unit 1)
 				)
@@
 		(instances
 			(project "autobot_mainboard"
-				(path "/f053f1d0-b1f5-4f80-9758-8ee1a2d3659d/037a1145-d2fa-427f-912d-11744b2ed89a"
-					(reference "#PWR034")
-					(unit 1)
-				)
 				(path "/f053f1d0-b1f5-4f80-9758-8ee1a2d3659d/18a50009-3afb-45d9-96a2-f4fbe8f24a2b"
 					(reference "#PWR031")
-					(unit 1)
-				)
-				(path "/f053f1d0-b1f5-4f80-9758-8ee1a2d3659d/bbe9edfa-2cce-4350-82ca-a6538778d251"
-					(reference "#PWR040")
-					(unit 1)
-				)
-				(path "/f053f1d0-b1f5-4f80-9758-8ee1a2d3659d/ea0baaba-f154-47d1-ba71-cf9d27cdfb48"
-					(reference "#PWR037")
 					(unit 1)
 				)
@@
 		(instances
 			(project "autobot_mainboard"
-				(path "/f053f1d0-b1f5-4f80-9758-8ee1a2d3659d/037a1145-d2fa-427f-912d-11744b2ed89a"
-					(reference "U10")
-					(unit 1)
-				)
 				(path "/f053f1d0-b1f5-4f80-9758-8ee1a2d3659d/18a50009-3afb-45d9-96a2-f4fbe8f24a2b"
 					(reference "U9")
-					(unit 1)
-				)
-				(path "/f053f1d0-b1f5-4f80-9758-8ee1a2d3659d/bbe9edfa-2cce-4350-82ca-a6538778d251"
-					(reference "U12")
-					(unit 1)
-				)
-				(path "/f053f1d0-b1f5-4f80-9758-8ee1a2d3659d/ea0baaba-f154-47d1-ba71-cf9d27cdfb48"
-					(reference "U11")
 					(unit 1)
 				)
@@
 		(instances
 			(project "autobot_mainboard"
-				(path "/f053f1d0-b1f5-4f80-9758-8ee1a2d3659d/037a1145-d2fa-427f-912d-11744b2ed89a"
-					(reference "#PWR036")
-					(unit 1)
-				)
 				(path "/f053f1d0-b1f5-4f80-9758-8ee1a2d3659d/18a50009-3afb-45d9-96a2-f4fbe8f24a2b"
 					(reference "#PWR033")
-					(unit 1)
-				)
-				(path "/f053f1d0-b1f5-4f80-9758-8ee1a2d3659d/bbe9edfa-2cce-4350-82ca-a6538778d251"
-					(reference "#PWR042")
-					(unit 1)
-				)
-				(path "/f053f1d0-b1f5-4f80-9758-8ee1a2d3659d/ea0baaba-f154-47d1-ba71-cf9d27cdfb48"
-					(reference "#PWR039")
 					(unit 1)
 				)
@@
 		(instances
 			(project "autobot_mainboard"
-				(path "/f053f1d0-b1f5-4f80-9758-8ee1a2d3659d/037a1145-d2fa-427f-912d-11744b2ed89a"
-					(reference "C22")
-					(unit 1)
-				)
 				(path "/f053f1d0-b1f5-4f80-9758-8ee1a2d3659d/18a50009-3afb-45d9-96a2-f4fbe8f24a2b"
 					(reference "C20")
-					(unit 1)
-				)
-				(path "/f053f1d0-b1f5-4f80-9758-8ee1a2d3659d/bbe9edfa-2cce-4350-82ca-a6538778d251"
-					(reference "C26")
-					(unit 1)
-				)
-				(path "/f053f1d0-b1f5-4f80-9758-8ee1a2d3659d/ea0baaba-f154-47d1-ba71-cf9d27cdfb48"
-					(reference "C24")
 					(unit 1)
 				)
@@
 		(instances
 			(project "autobot_mainboard"
-				(path "/f053f1d0-b1f5-4f80-9758-8ee1a2d3659d/037a1145-d2fa-427f-912d-11744b2ed89a"
-					(reference "C21")
-					(unit 1)
-				)
 				(path "/f053f1d0-b1f5-4f80-9758-8ee1a2d3659d/18a50009-3afb-45d9-96a2-f4fbe8f24a2b"
 					(reference "C19")
 					(unit 1)
 				)
-				(path "/f053f1d0-b1f5-4f80-9758-8ee1a2d3659d/bbe9edfa-2cce-4350-82ca-a6538778d251"
-					(reference "C25")
-					(unit 1)
-				)
-				(path "/f053f1d0-b1f5-4f80-9758-8ee1a2d3659d/ea0baaba-f154-47d1-ba71-cf9d27cdfb48"
-					(reference "C23")
-					(unit 1)
-				)

Commit message: rollback
Parts:
- renumbered C19 to C21, C20 to C22, U9 to U6
Changed lines of the file:
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@@
 		(dnp no)
 		(fields_autoplaced yes)
-		(property "Reference" "#PWR032"
+		(property "Reference" "#PWR031"
 			(at 114.3 93.98 0)
 			(hide yes)
@@
 			(project "autobot_mainboard"
 				(path "/f053f1d0-b1f5-4f80-9758-8ee1a2d3659d/18a50009-3afb-45d9-96a2-f4fbe8f24a2b"
-					(reference "#PWR032")
+					(reference "#PWR031")
 					(unit 1)
 				)
@@
 		(dnp no)
 		(fields_autoplaced yes)
-		(property "Reference" "#PWR031"
+		(property "Reference" "#PWR030"
 			(at 88.9 105.41 0)
 			(hide yes)
@@
 			(project "autobot_mainboard"
 				(path "/f053f1d0-b1f5-4f80-9758-8ee1a2d3659d/18a50009-3afb-45d9-96a2-f4fbe8f24a2b"
-					(reference "#PWR031")
+					(reference "#PWR030")
 					(unit 1)
 				)
@@
 		(in_pos_files yes)
 		(dnp no)
-		(property "Reference" "U9"
+		(property "Reference" "U6"
 			(at 82.55 83.8199 0)
 			(show_name no)
@@
 			(project "autobot_mainboard"
 				(path "/f053f1d0-b1f5-4f80-9758-8ee1a2d3659d/18a50009-3afb-45d9-96a2-f4fbe8f24a2b"
-					(reference "U9")
+					(reference "U6")
 					(unit 1)
 				)
@@
 		(dnp no)
 		(fields_autoplaced yes)
-		(property "Reference" "#PWR033"
+		(property "Reference" "#PWR032"
 			(at 121.92 93.98 0)
 			(hide yes)
@@
 			(project "autobot_mainboard"
 				(path "/f053f1d0-b1f5-4f80-9758-8ee1a2d3659d/18a50009-3afb-45d9-96a2-f4fbe8f24a2b"
-					(reference "#PWR033")
+					(reference "#PWR032")
 					(unit 1)
 				)
@@
 		(in_pos_files yes)
 		(dnp no)
-		(property "Reference" "C20"
+		(property "Reference" "C22"
 			(at 122.428 82.042 0)
 			(show_name no)
@@
 			(project "autobot_mainboard"
 				(path "/f053f1d0-b1f5-4f80-9758-8ee1a2d3659d/18a50009-3afb-45d9-96a2-f4fbe8f24a2b"
-					(reference "C20")
+					(reference "C22")
 					(unit 1)
 				)
@@
 		(in_pos_files yes)
 		(dnp no)
-		(property "Reference" "C19"
+		(property "Reference" "C21"
 			(at 114.554 82.042 0)
 			(show_name no)
@@
 			(project "autobot_mainboard"
 				(path "/f053f1d0-b1f5-4f80-9758-8ee1a2d3659d/18a50009-3afb-45d9-96a2-f4fbe8f24a2b"
-					(reference "C19")
-					(unit 1)
-				)
+					(reference "C21")
+					(unit 1)
+				)
