File: ELECTRONICS/Anchor_stable/Anchor.kicad_sch (KiCad schematic)
At the start: 85 parts, among them IC1 DW3210, J1 USB_C_Receptacle_USB2.0_16P, J2 Conn_01x05_Pin, J3 Conn_01x04_Pin, J4 Conn_01x05_Pin, J5 Conn_01x02_Pin, J6 Conn_01x04_Pin, J7 Conn_Coaxial, J8 Conn_Coaxial, Q1 DMG1012T, Q2 DMG1012T, Q3 DMG1012T, SW1 reset, SW3 SW_DIP_x05, U1 BQ24075RGT, U2 NRF52840-QFAA-R7, U3 AP7370-33FDC, Y1 TXC 8Y38472012, Y2 ECS-320-8-37B-CKY-TR, Y3 ECS-.327-6-1210B-N-TR

Commit message: Add files via upload
Parts:
- removed J2: Conn_01x05_Pin, Connector_PinHeader_2.54mm:PinHeader_1x05_P2.54mm_Vertical, symbol Connector:Conn_01x05_Pin
- added J9: Conn_01x03_Pin, Connector_PinHeader_2.54mm:PinHeader_1x03_P2.54mm_Vertical, symbol Connector:Conn_01x03_Pin
Connections:
- net DW_GPIO5 is gone; now on net GNDREF: IC1.5 (GPIO5_/_EXTTXE_/_SPIPOL)
- net DW_GPIO6 is gone; now on net GNDREF: IC1.2 (GPIO6_/_EXTRXE_/_SPIPHA)
- net DW_GPIO0: now also J9.1 (Pin_1)
- net DW_GPIO4: now also J9.2 (Pin_2)
- net DW_GPIO7: now also J9.3 (Pin_3)

Commit message: add reset button to anchor, polish later
Parts:
- SW1: footprint Button_Switch_THT:SW_PUSH_6mm -> MyFootprintLibrary:SW-SMD_L3.9-W3.0-P4.45
Changed lines of the file:
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@@
 			)
 		)
-		(property "Footprint" "Button_Switch_THT:SW_PUSH_6mm"
+		(property "Footprint" "MyFootprintLibrary:SW-SMD_L3.9-W3.0-P4.45"
 			(at 78.74 39.37 0)
 			(hide yes)
